Commit message: updates

File: lekiwi_description/urdf/base.urdf.xacro (robot description, xacro)
@@ -53,4 +53,6 @@
     </inertial>
   </link>
+  <!-- Laser frame -->
+  <link name="laser_frame"/>
   <!-- Camera link -->
   <link name="camera_link">
@@ -73,4 +75,6 @@
     </inertial>
   </link>
+  <!-- Camera frame-->
+  <link name="camera_frame"/>
   <!-- Left wheel link -->
   <link name="left_wheel_link">
@@ -146,4 +150,10 @@
     <origin xyz="${laser_base_offset_x} 0 ${laser_base_offset_z}" rpy="0 0 0"/>
   </joint>
+  <!-- laser_frame fixed joint -->
+  <joint name="laser_frame_joint" type="fixed">
+    <parent link="laser_link"/>
+    <child link="laser_frame"/>
+    <origin xyz="0 0 ${laser_frame_offset_z}" rpy="0 0 0"/>
+  </joint>
   <!-- camera fixed joint -->
   <joint name="camera_joint" type="fixed">
@@ -151,4 +161,10 @@
     <child link="camera_link"/>
     <origin xyz="${camera_base_offset_x} 0 ${camera_base_offset_z}" rpy="0 ${camera_offset_ry} 0"/>
+  </joint>
+  <!-- camera_frame fixed joint -->
+  <joint name="camera_frame_joint" type="fixed">
+    <parent link="camera_link"/>
+    <child link="camera_frame"/>
+    <origin xyz="0 0 0" rpy="0 0 0"/>
   </joint>
   <!-- left wheel joint: 60 degrees anti-clockwise from +X at radius wheel_base_radius -->

File: lekiwi_description/urdf/base_properties.xacro (robot description, xacro)
@@ -18,4 +18,6 @@
   <xacro:property name="camera_base_offset_z" value="0.026"/>
   <xacro:property name="camera_offset_ry" value="${pi/2}"/> <!-- Camera mesh/joint rotation about Y (rad) -->
+  <!-- LDLidar frame offsets from laser_link -->
+  <xacro:property name="laser_frame_offset_z" value="0.027"/>
   <!-- Wheel geometry for omnidirectional control -->
   <xacro:property name="wheel_radius" value="0.051"/>  <!-- meters -->

Commit message: update lekiwi_base_control, add command limits

File: lekiwi_description/urdf/base.urdf.xacro (robot description, xacro)
@@ -174,4 +174,5 @@
     <origin xyz="${wheel_base_radius * cos(offset)} ${wheel_base_radius * sin(offset)} ${wheel_base_offset_z}" rpy="0 ${pi/2} ${offset}"/>
     <axis xyz="0 0 1"/>
+    <limit effort="${max_torque_nm}" velocity="${max_velocity_rads}"/>
   </joint>
   <!-- back wheel joint: 180 degrees anti-clockwise from +X at radius base_radius -->
@@ -181,4 +182,5 @@
     <origin xyz="${wheel_base_radius * cos(offset + theta)} ${wheel_base_radius * sin(offset + theta)} ${wheel_base_offset_z}" rpy="0 ${pi/2} ${offset + theta}"/>
     <axis xyz="0 0 1"/>
+    <limit effort="${max_torque_nm}" velocity="${max_velocity_rads}"/>
   </joint>
   <!-- right wheel joint: 300 degrees (or -60 degrees) anti-clockwise from +X at radius base_radius -->
@@ -188,4 +190,5 @@
     <origin xyz="${wheel_base_radius * cos(offset - theta)} ${wheel_base_radius * sin(offset - theta)} ${wheel_base_offset_z}" rpy="0 ${pi/2} ${offset - theta}"/>
     <axis xyz="0 0 1"/>
+    <limit effort="${max_torque_nm}" velocity="${max_velocity_rads}"/>
   </joint>
   <!-- ROS 2 CONTROL -->
@@ -205,10 +208,9 @@
       <param name="motor_id">${left_motor_id}</param>
       <param name="operating_mode">${operating_mode}</param>
-      <param name="max_velocity">${max_velocity_rads}</param>
       <command_interface name="velocity"/>
       <command_interface name="acceleration"/>
       <state_interface name="position"/>
       <state_interface name="velocity"/>
-      <state_interface name="load"/>
+      <state_interface name="effort"/>
       <state_interface name="voltage"/>
       <state_interface name="temperature"/>
@@ -220,10 +222,9 @@
       <param name="motor_id">${back_motor_id}</param>
       <param name="operating_mode">${operating_mode}</param>
-      <param name="max_velocity">${max_velocity_rads}</param>
       <command_interface name="velocity"/>
       <command_interface name="acceleration"/>
       <state_interface name="position"/>
       <state_interface name="velocity"/>
-      <state_interface name="load"/>
+      <state_interface name="effort"/>
       <state_interface name="voltage"/>
       <state_interface name="temperature"/>
@@ -235,10 +236,9 @@
       <param name="motor_id">${right_motor_id}</param>
       <param name="operating_mode">${operating_mode}</param>
-      <param name="max_velocity">${max_velocity_rads}</param>
       <command_interface name="velocity"/>
       <command_interface name="acceleration"/>
       <state_interface name="position"/>
       <state_interface name="velocity"/>
-      <state_interface name="load"/>
+      <state_interface name="effort"/>
       <state_interface name="voltage"/>
       <state_interface name="temperature"/>

File: lekiwi_description/urdf/base_properties.xacro (robot description, xacro)
@@ -34,9 +34,10 @@
   <xacro:property name="serial_port" value="/dev/ttySERVO"/>
   <xacro:property name="baud_rate" value="1000000"/>
-  <!-- Maximum allowable speed/acceleration for each motor -->
+  <!-- Maximum allowable speed/acceleration/torque for each motor -->
   <xacro:property name="max_velocity_steps" value="2720"/> <!-- steps/second (80% of 3400 hardware max) -->
   <xacro:property name="max_velocity_rads" value="${max_velocity_steps*2*pi/4096}"/> <!-- rad/s -->
   <xacro:property name="max_acceleration_steps" value="${254*100}"/> <!-- steps/second² (100% hardware max) -->
   <xacro:property name="max_acceleration_rads" value="${max_acceleration_steps*2*pi/4096}"/> <!-- rad/s² -->
+  <xacro:property name="max_torque_nm" value="2.942"/> <!-- N⋅m (30 kgf⋅cm for STS3215) -->
   <!-- Omnidirectional Kinematics Calculations -->
   <!-- For 3-wheel omni drive: ω_i = (-sin(θ_i)·v_x + cos(θ_i)·v_y + R·ω_z) / r -->

Commit message: update wheel stl orientation

File: lekiwi_description/urdf/base.urdf.xacro (robot description, xacro)
@@ -80,12 +80,12 @@
   <link name="left_wheel_link">
     <visual>
-      <origin xyz="0 0 0" rpy="${wheel_offset_rx} 0 0"/>
-      <geometry>
-        <mesh filename="package://lekiwi_description/meshes/omni_wheel.stl"/>
-      </geometry>
-      <material name="charcoal"/>
-    </visual>
-    <collision>
-      <origin xyz="0 0 0" rpy="${wheel_offset_rx} 0 0"/>
+      <origin xyz="0 0 0" rpy="${wheel_offset_rx} 0 ${wheel_offset_rz}"/>
+      <geometry>
+        <mesh filename="package://lekiwi_description/meshes/omni_wheel.stl"/>
+      </geometry>
+      <material name="charcoal"/>
+    </visual>
+    <collision>
+      <origin xyz="0 0 0" rpy="${wheel_offset_rx} 0 ${wheel_offset_rz}"/>
       <geometry>
         <mesh filename="package://lekiwi_description/meshes/omni_wheel.stl"/>
@@ -100,12 +100,12 @@
   <link name="back_wheel_link">
     <visual>
-      <origin xyz="0 0 0" rpy="${wheel_offset_rx} 0 0"/>
-      <geometry>
-        <mesh filename="package://lekiwi_description/meshes/omni_wheel.stl"/>
-      </geometry>
-      <material name="charcoal"/>
-    </visual>
-    <collision>
-      <origin xyz="0 0 0" rpy="${wheel_offset_rx} 0 0"/>
+      <origin xyz="0 0 0" rpy="${wheel_offset_rx} 0 ${wheel_offset_rz}"/>
+      <geometry>
+        <mesh filename="package://lekiwi_description/meshes/omni_wheel.stl"/>
+      </geometry>
+      <material name="charcoal"/>
+    </visual>
+    <collision>
+      <origin xyz="0 0 0" rpy="${wheel_offset_rx} 0 ${wheel_offset_rz}"/>
       <geometry>
         <mesh filename="package://lekiwi_description/meshes/omni_wheel.stl"/>
@@ -120,12 +120,12 @@
   <link name="right_wheel_link">
     <visual>
-      <origin xyz="0 0 0" rpy="${wheel_offset_rx} 0 0"/>
-      <geometry>
-        <mesh filename="package://lekiwi_description/meshes/omni_wheel.stl"/>
-      </geometry>
-      <material name="charcoal"/>
-    </visual>
-    <collision>
-      <origin xyz="0 0 0" rpy="${wheel_offset_rx} 0 0"/>
+      <origin xyz="0 0 0" rpy="${wheel_offset_rx} 0 ${wheel_offset_rz}"/>
+      <geometry>
+        <mesh filename="package://lekiwi_description/meshes/omni_wheel.stl"/>
+      </geometry>
+      <material name="charcoal"/>
+    </visual>
+    <collision>
+      <origin xyz="0 0 0" rpy="${wheel_offset_rx} 0 ${wheel_offset_rz}"/>
       <geometry>
         <mesh filename="package://lekiwi_description/meshes/omni_wheel.stl"/>

File: lekiwi_description/urdf/base_properties.xacro (robot description, xacro)
@@ -10,4 +10,5 @@
   <xacro:property name="wheel_base_offset_z" value="0.01036"/>
   <xacro:property name="wheel_offset_rx" value="${pi}"/> <!-- Wheel mesh rotation about X (rad) -->
+  <xacro:property name="wheel_offset_rz" value="${pi}"/> <!-- Wheel mesh rotation about Z (rad) -->
   <!-- LD06 laser offsets from base_link -->
   <xacro:property name="laser_base_offset_x" value="-0.045042"/>

Commit message: update orientation offsets

File: lekiwi_description/urdf/base.urdf.xacro (robot description, xacro)
@@ -80,12 +80,12 @@
   <link name="left_wheel_link">
     <visual>
-      <origin xyz="0 0 0" rpy="${wheel_offset_rx} 0 ${wheel_offset_rz}"/>
-      <geometry>
-        <mesh filename="package://lekiwi_description/meshes/omni_wheel.stl"/>
-      </geometry>
-      <material name="charcoal"/>
-    </visual>
-    <collision>
-      <origin xyz="0 0 0" rpy="${wheel_offset_rx} 0 ${wheel_offset_rz}"/>
+      <origin xyz="0 0 0" rpy="0 0 0"/>
+      <geometry>
+        <mesh filename="package://lekiwi_description/meshes/omni_wheel.stl"/>
+      </geometry>
+      <material name="charcoal"/>
+    </visual>
+    <collision>
+      <origin xyz="0 0 0" rpy="0 0 0"/>
       <geometry>
         <mesh filename="package://lekiwi_description/meshes/omni_wheel.stl"/>
@@ -100,12 +100,12 @@
   <link name="back_wheel_link">
     <visual>
-      <origin xyz="0 0 0" rpy="${wheel_offset_rx} 0 ${wheel_offset_rz}"/>
-      <geometry>
-        <mesh filename="package://lekiwi_description/meshes/omni_wheel.stl"/>
-      </geometry>
-      <material name="charcoal"/>
-    </visual>
-    <collision>
-      <origin xyz="0 0 0" rpy="${wheel_offset_rx} 0 ${wheel_offset_rz}"/>
+      <origin xyz="0 0 0" rpy="0 0 0"/>
+      <geometry>
+        <mesh filename="package://lekiwi_description/meshes/omni_wheel.stl"/>
+      </geometry>
+      <material name="charcoal"/>
+    </visual>
+    <collision>
+      <origin xyz="0 0 0" rpy="0 0 0"/>
       <geometry>
         <mesh filename="package://lekiwi_description/meshes/omni_wheel.stl"/>
@@ -120,12 +120,12 @@
   <link name="right_wheel_link">
     <visual>
-      <origin xyz="0 0 0" rpy="${wheel_offset_rx} 0 ${wheel_offset_rz}"/>
-      <geometry>
-        <mesh filename="package://lekiwi_description/meshes/omni_wheel.stl"/>
-      </geometry>
-      <material name="charcoal"/>
-    </visual>
-    <collision>
-      <origin xyz="0 0 0" rpy="${wheel_offset_rx} 0 ${wheel_offset_rz}"/>
+      <origin xyz="0 0 0" rpy="0 0 0"/>
+      <geometry>
+        <mesh filename="package://lekiwi_description/meshes/omni_wheel.stl"/>
+      </geometry>
+      <material name="charcoal"/>
+    </visual>
+    <collision>
+      <origin xyz="0 0 0" rpy="0 0 0"/>
       <geometry>
         <mesh filename="package://lekiwi_description/meshes/omni_wheel.stl"/>

File: lekiwi_description/urdf/base_properties.xacro (robot description, xacro)
@@ -9,6 +9,4 @@
   <xacro:property name="wheel_base_radius" value="0.132239"/>
   <xacro:property name="wheel_base_offset_z" value="0.01036"/>
-  <xacro:property name="wheel_offset_rx" value="${pi}"/> <!-- Wheel mesh rotation about X (rad) -->
-  <xacro:property name="wheel_offset_rz" value="${pi}"/> <!-- Wheel mesh rotation about Z (rad) -->
   <!-- LD06 laser offsets from base_link -->
   <xacro:property name="laser_base_offset_x" value="-0.045042"/>

Commit message: Merge lekiwi_description and lekiwi_teleop updates from main branch

File: lekiwi_description/urdf/base.urdf.xacro (robot description, xacro)
@@ -80,12 +80,12 @@
   <link name="left_wheel_link">
     <visual>
-      <origin xyz="0 0 0" rpy="${wheel_offset_rx} 0 0"/>
-      <geometry>
-        <mesh filename="package://lekiwi_description/meshes/omni_wheel.stl"/>
-      </geometry>
-      <material name="charcoal"/>
-    </visual>
-    <collision>
-      <origin xyz="0 0 0" rpy="${wheel_offset_rx} 0 0"/>
+      <origin xyz="0 0 0" rpy="0 0 0"/>
+      <geometry>
+        <mesh filename="package://lekiwi_description/meshes/omni_wheel.stl"/>
+      </geometry>
+      <material name="charcoal"/>
+    </visual>
+    <collision>
+      <origin xyz="0 0 0" rpy="0 0 0"/>
       <geometry>
         <mesh filename="package://lekiwi_description/meshes/omni_wheel.stl"/>
@@ -100,12 +100,12 @@
   <link name="back_wheel_link">
     <visual>
-      <origin xyz="0 0 0" rpy="${wheel_offset_rx} 0 0"/>
-      <geometry>
-        <mesh filename="package://lekiwi_description/meshes/omni_wheel.stl"/>
-      </geometry>
-      <material name="charcoal"/>
-    </visual>
-    <collision>
-      <origin xyz="0 0 0" rpy="${wheel_offset_rx} 0 0"/>
+      <origin xyz="0 0 0" rpy="0 0 0"/>
+      <geometry>
+        <mesh filename="package://lekiwi_description/meshes/omni_wheel.stl"/>
+      </geometry>
+      <material name="charcoal"/>
+    </visual>
+    <collision>
+      <origin xyz="0 0 0" rpy="0 0 0"/>
       <geometry>
         <mesh filename="package://lekiwi_description/meshes/omni_wheel.stl"/>
@@ -120,12 +120,12 @@
   <link name="right_wheel_link">
     <visual>
-      <origin xyz="0 0 0" rpy="${wheel_offset_rx} 0 0"/>
-      <geometry>
-        <mesh filename="package://lekiwi_description/meshes/omni_wheel.stl"/>
-      </geometry>
-      <material name="charcoal"/>
-    </visual>
-    <collision>
-      <origin xyz="0 0 0" rpy="${wheel_offset_rx} 0 0"/>
+      <origin xyz="0 0 0" rpy="0 0 0"/>
+      <geometry>
+        <mesh filename="package://lekiwi_description/meshes/omni_wheel.stl"/>
+      </geometry>
+      <material name="charcoal"/>
+    </visual>
+    <collision>
+      <origin xyz="0 0 0" rpy="0 0 0"/>
       <geometry>
         <mesh filename="package://lekiwi_description/meshes/omni_wheel.stl"/>

File: lekiwi_description/urdf/base_properties.xacro (robot description, xacro)
@@ -9,5 +9,4 @@
   <xacro:property name="wheel_base_radius" value="0.132239"/>
   <xacro:property name="wheel_base_offset_z" value="0.01036"/>
-  <xacro:property name="wheel_offset_rx" value="${pi}"/> <!-- Wheel mesh rotation about X (rad) -->
   <!-- LD06 laser offsets from base_link -->
   <xacro:property name="laser_base_offset_x" value="-0.045042"/>

Commit message: updated urdf with mock mode argument

File: lekiwi_description/urdf/base.urdf.xacro (robot description, xacro)
@@ -2,5 +2,9 @@
 <robot xmlns:xacro="http://www.ros.org/wiki/xacro" name="lekiwi">
   <!-- Include robot properties -->
-  <xacro:include filename="$(find lekiwi_description)/urdf/base_properties.xacro"/>
+  <xacro:include filename="$(find lekiwi_description)/urdf/base.common.xacro"/>
+  <xacro:include filename="$(find lekiwi_description)/urdf/base.control.xacro"/>
+  <!-- Arguments -->
+  <xacro:arg name="serial_port" default="${serial_port}"/>
+  <xacro:arg name="use_mock" default="${use_mock}"/>
   <!-- Define custom materials for base and wheels using color properties -->
   <material name="light_grey">
@@ -142,5 +146,5 @@
     <parent link="base_footprint"/>
     <child link="base_link"/>
-    <origin xyz="0 0 ${base_footprint_offset_z}" rpy="0 0 0"/>
+    <origin xyz="0 0 ${wheel_radius - wheel_base_offset_z}" rpy="0 0 0"/>
   </joint>
   <!-- laser fixed joint -->
@@ -198,9 +202,8 @@
       <plugin>sts_hardware_interface/STSHardwareInterface</plugin>
       <!-- Serial communication parameters -->
-      <param name="serial_port">${serial_port}</param>
+      <param name="serial_port">$(arg serial_port)</param>
       <param name="baud_rate">${baud_rate}</param>
-      <param name="use_sync_write">true</param>
-      <param name="enable_multi_turn">true</param>
-      <param name="enable_mock_mode">false</param>
+      <param name="use_sync_write">${use_sync_write}</param>
+      <param name="enable_mock_mode">$(arg use_mock)</param>
     </hardware>
     <!-- Left wheel joint (Motor ID 7) -->
