Commit message: replace package:// with github paths

File: lekiwi_description/urdf/base.urdf (robot description, URDF)
Before this commit: robot lekiwi, 9 links, 8 joints
Links:
- link back_wheel_link: geometry collision mesh filename=https://raw.githubusercontent.com/adityakamath/lekiwi_ros2/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; visual mesh filename=https://raw.githubusercontent.com/adityakamath/lekiwi_ros2/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
- link base_link: geometry collision mesh filename=https://raw.githubusercontent.com/adityakamath/lekiwi_ros2/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; visual mesh filename=https://raw.githubusercontent.com/adityakamath/lekiwi_ros2/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
- link camera_link: geometry collision mesh filename=https://raw.githubusercontent.com/adityakamath/lekiwi_ros2/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; visual mesh filename=https://raw.githubusercontent.com/adityakamath/lekiwi_ros2/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
- link laser_link: geometry collision mesh filename=https://raw.githubusercontent.com/adityakamath/lekiwi_ros2/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; visual mesh filename=https://raw.githubusercontent.com/adityakamath/lekiwi_ros2/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
- link left_wheel_link: geometry collision mesh filename=https://raw.githubusercontent.com/adityakamath/lekiwi_ros2/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; visual mesh filename=https://raw.githubusercontent.com/adityakamath/lekiwi_ros2/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
- link right_wheel_link: geometry collision mesh filename=https://raw.githubusercontent.com/adityakamath/lekiwi_ros2/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; visual mesh filename=https://raw.githubusercontent.com/adityakamath/lekiwi_ros2/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

Commit message: revert to using package://

File: lekiwi_description/urdf/base.urdf (robot description, URDF)
Before this commit: robot lekiwi, 9 links, 8 joints
Links:
- link back_wheel_link: geometry collision mesh filename=package://lekiwi_description/meshes/omni_wheel.stl; visual mesh filename=package://lekiwi_description/meshes/omni_wheel.stl
- link base_link: geometry collision mesh filename=package://lekiwi_description/meshes/lekiwi_base.stl; visual mesh filename=package://lekiwi_description/meshes/lekiwi_base.stl
- link camera_link: geometry collision mesh filename=package://lekiwi_description/meshes/hd_webcam.stl; visual mesh filename=package://lekiwi_description/meshes/hd_webcam.stl
- link laser_link: geometry collision mesh filename=package://lekiwi_description/meshes/ld06_lidar.stl; visual mesh filename=package://lekiwi_description/meshes/ld06_lidar.stl
- link left_wheel_link: geometry collision mesh filename=package://lekiwi_description/meshes/omni_wheel.stl; visual mesh filename=package://lekiwi_description/meshes/omni_wheel.stl
- link right_wheel_link: geometry collision mesh filename=package://lekiwi_description/meshes/omni_wheel.stl; visual mesh filename=package://lekiwi_description/meshes/omni_wheel.stl

Commit message: add correct urdf

File: lekiwi_description/urdf/base.urdf (robot description, URDF)
Before this commit: robot lekiwi, 9 links, 8 joints
Joints:
- joint back_wheel_joint: limit effort=2.942 velocity=4.17167481696419 -> effort=2.942 velocity=4.218447166685513; origin xyz=-0.132239 0.00000000000000016 0.01036 rpy=0 1.57079632679490 3.14159265358979 -> xyz=-0.132239 1.6194606807244685e-17 0.01036 rpy=0 1.5707963267948966 3.141592653589793
- joint base_footprint_joint: origin xyz=0 0 0.04064 rpy=0 0 0 -> xyz=0 0 0.040639999999999996 rpy=0 0 0
- joint camera_joint: origin xyz=0.114 0 0.026 rpy=0 1.57079632679490 0 -> xyz=0.114 0 0.026 rpy=0 1.5707963267948966 0
- joint left_wheel_joint: limit effort=2.942 velocity=4.17167481696419 -> effort=2.942 velocity=4.218447166685513; origin xyz=0.06611950000000000 0.11449673600000000 0.01036 rpy=0 1.57079632679490 1.04719755119660 -> xyz=0.06611950000000001 0.11452233337105037 0.01036 rpy=0 1.5707963267948966 1.0471975511965976
- joint right_wheel_joint: limit effort=2.942 velocity=4.17167481696419 -> effort=2.942 velocity=4.218447166685513; origin xyz=0.06611950000000000 -0.11449673600000000 0.01036 rpy=0 1.57079632679490 -1.04719755119660 -> xyz=0.06611950000000001 -0.11452233337105037 0.01036 rpy=0 1.5707963267948966 -1.0471975511965976

Commit message: update urdf: rename camera_frame to camera

File: lekiwi_description/urdf/base.urdf (robot description, URDF)
Before this commit: robot lekiwi, 9 links, 8 joints
Links:
- removed link camera_frame
- added link camera
Joints:
- joint camera_frame_joint: child camera_frame -> camera

File: lekiwi_description/urdf/base.urdf.xacro (robot description, xacro)
@@ -80,5 +80,5 @@
   </link>
   <!-- Camera frame-->
-  <link name="camera_frame"/>
+  <link name="camera"/>
   <!-- Left wheel link -->
   <link name="left_wheel_link">
@@ -169,6 +169,6 @@
   <joint name="camera_frame_joint" type="fixed">
     <parent link="camera_link"/>
-    <child link="camera_frame"/>
-    <origin xyz="0 0 0" rpy="0 0 0"/>
+    <child link="camera"/>
+    <origin xyz="0 0 0" rpy="0 0 ${3*pi/2}"/>
   </joint>
   <!-- left wheel joint: 60 degrees anti-clockwise from +X at radius wheel_base_radius -->
