Commit message: tune: lower proportional_acc_max and restore physics-derived limits
Reduce proportional_acc_max from 100 → 25 so hardware ramps span
~100ms rather than <5ms. At 100 the scaled ACC values still complete
within a single 20ms control cycle, making proportional synchronisation
irrelevant and leaving the back wheel (2× velocity for pure-Y strafe)
lagging the front wheels on start/stop, causing chassis rotation.

At ACC=25 the ramp is slow enough that proportional scaling meaningfully
synchronises all three wheels, fixing the drift-and-twitch observed
during lateral strafing.

Also restores software acceleration limits to their physics-derived
values (2.61 / 2.26 / 17.1) and updates the comment to document the
>2 m/s² per-cycle-step requirement for hardware ACC to engage.

Co-Authored-By: Claude Sonnet 4.6 <noreply@anthropic.com>

File: lekiwi_description/urdf/base.control.xacro (robot description, xacro)
@@ -13,5 +13,5 @@
   <!-- All others scaled proportionally so every wheel finishes ramping in equal time. -->
   <!-- Set proportional_acc_max to 0 to disable (ACC=0 for all wheels). -->
-  <xacro:property name="proportional_acc_max" value="100"/>       <!-- [0-254] -->
+  <xacro:property name="proportional_acc_max" value="25"/>        <!-- [0-254] -->
   <xacro:property name="proportional_acc_deadband" value="0.05"/> <!-- rad/s, below this max-delta ACC=0 (steady-state cruise) -->
   <!-- Motor IDs and mode -->

Commit message: feat: wire proportional per-wheel ACC and restore physics-derived limits
Add proportional_acc_max and proportional_acc_deadband xacro properties
to base.control.xacro and pass them through to the sts_hardware_interface
<hardware> block in base.urdf.xacro.

sts_hardware_interface already implements the proportional ACC algorithm
(back wheel gets acc_max, others scale so all wheels finish ramping in
equal wall-clock time), but the parameters were never wired from the
lekiwi_ros2 side — the hardware was silently falling back to defaults.
This change makes the configuration explicit and tunable.

With proportional ACC now active, software acceleration limits are
restored to their physics-derived values (2.61 / 2.26 / 17.1) and the
stale "hardware receives 0" comment is replaced with an accurate
description of the proportional ACC behaviour.

Co-Authored-By: Claude Sonnet 4.6 <noreply@anthropic.com>

File: lekiwi_description/urdf/base.control.xacro (robot description, xacro)
@@ -9,4 +9,10 @@
   <!-- Adjust for other motor models: STS3032 max=2900, STS3235 max=3400 -->
   <xacro:property name="sts_max_velocity_steps" value="3400"/>  <!-- Max hardware velocity in steps/s (absolute motor limit, do not exceed) -->
+  <!-- Proportional ACC parameters (SyncWriteSpe velocity path only) -->
+  <!-- ACC given to the wheel with the largest |target - current| velocity delta. -->
+  <!-- All others scaled proportionally so every wheel finishes ramping in equal time. -->
+  <!-- Set proportional_acc_max to 0 to disable (ACC=0 for all wheels). -->
+  <xacro:property name="proportional_acc_max" value="100"/>        <!-- [0-254] -->
+  <xacro:property name="proportional_acc_deadband" value="0.05"/>  <!-- rad/s, below this max-delta ACC=0 (steady-state cruise) -->
   <!-- Motor IDs and mode -->
   <xacro:property name="left_motor_id" value="7"/>

File: lekiwi_description/urdf/base.urdf.xacro (robot description, xacro)
@@ -208,4 +208,7 @@
       <!-- Motor-specific parameter (adjust for different STS motor models) -->
       <param name="max_velocity_steps">${sts_max_velocity_steps}</param>
+      <!-- Proportional per-wheel ACC: back wheel gets acc_max, others scale proportionally -->
+      <param name="proportional_acc_max">${proportional_acc_max}</param>
+      <param name="proportional_acc_deadband">${proportional_acc_deadband}</param>
     </hardware>
     <!-- Left wheel joint (Motor ID 7) -->

Commit message: tune: increase proportional_acc_max from 100 to 150
Higher ACC value improves hardware tracking of the software velocity ramp
per 20ms cycle (~0.46 rad/s vs ~0.31 rad/s for the back wheel), reducing
the lag between commanded and actual wheel velocities during acceleration.
The proportional relationship across wheels is preserved, so synchronisation
is maintained.

Co-Authored-By: Claude Sonnet 4.6 <noreply@anthropic.com>

File: lekiwi_description/urdf/base.control.xacro (robot description, xacro)
@@ -13,5 +13,5 @@
   <!-- All others scaled proportionally so every wheel finishes ramping in equal time. -->
   <!-- Set proportional_acc_max to 0 to disable (ACC=0 for all wheels). -->
-  <xacro:property name="proportional_acc_max" value="100"/>        <!-- [0-254] -->
+  <xacro:property name="proportional_acc_max" value="150"/>        <!-- [0-254] -->
   <xacro:property name="proportional_acc_deadband" value="0.05"/>  <!-- rad/s, below this max-delta ACC=0 (steady-state cruise) -->
   <!-- Motor IDs and mode -->
