Commit message: update config files

File: lekiwi_description/urdf/base.control.xacro (robot description, xacro)
@@ -6,4 +6,7 @@
   <xacro:property name="use_mock" default="false"/>
   <xacro:property name="use_sync_write" default="true"/>
+  <!-- Motor-specific parameter (STS3215 default) -->
+  <!-- Adjust for other motor models: STS3032 max=2900, STS3235 max=3400 -->
+  <xacro:property name="sts_max_velocity_steps" value="3400"/>  <!-- Max hardware velocity in steps/s -->
   <!-- Motor IDs and mode -->
   <xacro:property name="left_motor_id" value="7"/>

File: lekiwi_description/urdf/base.urdf.xacro (robot description, xacro)
@@ -206,4 +206,6 @@
       <param name="use_sync_write">${use_sync_write}</param>
       <param name="enable_mock_mode">$(arg use_mock)</param>
+      <!-- Motor-specific parameter (adjust for different STS motor models) -->
+      <param name="max_velocity_steps">${sts_max_velocity_steps}</param>
     </hardware>
     <!-- Left wheel joint (Motor ID 7) -->

Commit message: Tune velocity and acceleration limits for lekiwi base
- Increase max_velocity_steps from 2750 to 2890 (85% of 3400 hardware max)
- Enable enforce_command_limits via JointSaturationLimiter
- Update cascaded velocity limits in base_controllers.yaml and teleop_config.yaml
- Set max_acceleration to ~100ms ramp-to-full-speed on all axes
- Add comments explaining software vs hardware acceleration semantics

File: lekiwi_description/urdf/base.control.xacro (robot description, xacro)
@@ -8,5 +8,5 @@
   <!-- Motor-specific parameter (STS3215 default) -->
   <!-- Adjust for other motor models: STS3032 max=2900, STS3235 max=3400 -->
-  <xacro:property name="sts_max_velocity_steps" value="3400"/>  <!-- Max hardware velocity in steps/s -->
+  <xacro:property name="sts_max_velocity_steps" value="3400"/>  <!-- Max hardware velocity in steps/s (absolute motor limit, do not exceed) -->
   <!-- Motor IDs and mode -->
   <xacro:property name="left_motor_id" value="7"/>
@@ -19,5 +19,5 @@
   <xacro:property name="theta" value="${2*pi/3}"/>  <!-- 120° between wheels -->
   <!-- Maximum allowable speed/acceleration/torque for each motor -->
-  <xacro:property name="max_velocity_steps" value="2750"/> <!-- steps/second (81% of 3400 hardware max, +1% margin) -->
+  <xacro:property name="max_velocity_steps" value="2890"/> <!-- steps/second (85% of 3400 hardware max, 15% safety margin) -->
   <xacro:property name="max_velocity_rads" value="${max_velocity_steps*2*pi/4096}"/> <!-- rad/s -->
   <xacro:property name="max_torque_nm" value="2.942"/> <!-- N⋅m (30 kgf⋅cm for STS3215) -->

Commit message: feat: expose proportional ACC params in URDF, reduce controller max_acceleration
- Add proportional_acc_max (default 100) and proportional_acc_deadband (default 0.05 rad/s)
  as xacro properties in base.control.xacro and param entries in base.urdf.xacro
- Reduce base_controllers.yaml max_acceleration: x 2.61->1.0, y 2.26->1.0, z 17.1->10.0
  (softer twist_mux ramp; proportional hw ACC handles per-wheel sync)

File: lekiwi_description/urdf/base.control.xacro (robot description, xacro)
@@ -9,4 +9,10 @@
   <!-- Adjust for other motor models: STS3032 max=2900, STS3235 max=3400 -->
   <xacro:property name="sts_max_velocity_steps" value="3400"/>  <!-- Max hardware velocity in steps/s (absolute motor limit, do not exceed) -->
+  <!-- Proportional ACC parameters (SyncWriteSpe velocity path only) -->
+  <!-- ACC given to the wheel with the largest |target - current| velocity delta. -->
+  <!-- All others scaled proportionally so every wheel finishes ramping in equal time. -->
+  <!-- Set proportional_acc_max to 0 to disable (ACC=0 for all wheels). -->
+  <xacro:property name="proportional_acc_max" value="100"/>       <!-- [0-254] -->
+  <xacro:property name="proportional_acc_deadband" value="0.05"/> <!-- rad/s, below this max-delta ACC=0 (steady-state cruise) -->
   <!-- Motor IDs and mode -->
   <xacro:property name="left_motor_id" value="7"/>

File: lekiwi_description/urdf/base.urdf.xacro (robot description, xacro)
@@ -208,4 +208,7 @@
       <!-- Motor-specific parameter (adjust for different STS motor models) -->
       <param name="max_velocity_steps">${sts_max_velocity_steps}</param>
+      <!-- Proportional ACC: scale per-wheel acceleration so all wheels finish ramping in equal time -->
+      <param name="proportional_acc_max">${proportional_acc_max}</param>
+      <param name="proportional_acc_deadband">${proportional_acc_deadband}</param>
     </hardware>
     <!-- Left wheel joint (Motor ID 7) -->

Commit message: minor updates - control values

File: lekiwi_description/urdf/base.control.xacro (robot description, xacro)
@@ -25,5 +25,5 @@
   <xacro:property name="theta" value="${2*pi/3}"/>  <!-- 120° between wheels -->
   <!-- Maximum allowable speed/acceleration/torque for each motor -->
-  <xacro:property name="max_velocity_steps" value="2890"/> <!-- steps/second (85% of 3400 hardware max, 15% safety margin) -->
+  <xacro:property name="max_velocity_steps" value="${int(sts_max_velocity_steps * 0.85)}"/> <!-- steps/second (85% of hardware max, 15% safety margin) -->
   <xacro:property name="max_velocity_rads" value="${max_velocity_steps*2*pi/4096}"/> <!-- rad/s -->
   <xacro:property name="max_torque_nm" value="2.942"/> <!-- N⋅m (30 kgf⋅cm for STS3215) -->

Commit message: urdf: remove acceleration command interface and proportional_acc_deadband property
- acceleration command interface removed from all 3 wheel joints in
  base.urdf.xacro; OmniWheelDriveController never writes it and the
  sts_hardware_interface now treats it as optional for MODE_VELOCITY
- proportional_acc_deadband removed from base.control.xacro; it is now
  a hardware-level parameter with a hardcoded default in sts_hardware_interface

File: lekiwi_description/urdf/base.control.xacro (robot description, xacro)
@@ -14,5 +14,4 @@
   <!-- Set proportional_acc_max to 0 to disable (ACC=0 for all wheels). -->
   <xacro:property name="proportional_acc_max" value="25"/>        <!-- [0-254] -->
-  <xacro:property name="proportional_acc_deadband" value="0.05"/> <!-- rad/s, below this max-delta ACC=0 (steady-state cruise) -->
   <!-- Motor IDs and mode -->
   <xacro:property name="left_motor_id" value="7"/>

File: lekiwi_description/urdf/base.urdf.xacro (robot description, xacro)
@@ -210,5 +210,4 @@
       <!-- Proportional ACC: scale per-wheel acceleration so all wheels finish ramping in equal time -->
       <param name="proportional_acc_max">${proportional_acc_max}</param>
-      <param name="proportional_acc_deadband">${proportional_acc_deadband}</param>
     </hardware>
     <!-- Left wheel joint (Motor ID 7) -->
@@ -217,5 +216,4 @@
       <param name="operating_mode">${operating_mode}</param>
       <command_interface name="velocity"/>
-      <command_interface name="acceleration"/>
       <state_interface name="position"/>
       <state_interface name="velocity"/>
@@ -231,5 +229,4 @@
       <param name="operating_mode">${operating_mode}</param>
       <command_interface name="velocity"/>
-      <command_interface name="acceleration"/>
       <state_interface name="position"/>
       <state_interface name="velocity"/>
@@ -245,5 +242,4 @@
       <param name="operating_mode">${operating_mode}</param>
       <command_interface name="velocity"/>
-      <command_interface name="acceleration"/>
       <state_interface name="position"/>
       <state_interface name="velocity"/>
