Commit message: added BNO055 IMU

File: lekiwi_description/urdf/base.common.xacro (robot description, xacro)
@@ -19,3 +19,6 @@
   <!-- LDLidar frame offsets from laser_link -->
   <xacro:property name="laser_frame_offset_z" value="0.027"/>
+  <!-- BNO055 IMU offsets from base_link -->
+  <xacro:property name="imu_base_offset_x" value="-0.044"/>
+  <xacro:property name="imu_base_offset_z" value="0.08"/>
 </robot>

File: lekiwi_description/urdf/base.control.xacro (robot description, xacro)
@@ -14,4 +14,9 @@
   <!-- Set proportional_acc_max to 0 to disable (ACC=0 for all wheels). -->
   <xacro:property name="proportional_acc_max" value="25"/>        <!-- [0-254] -->
+  <!-- BNO055 IMU parameters -->
+  <xacro:property name="imu_i2c_bus"    value="1"/>       <!-- I2C bus number (/dev/i2c-1) -->
+  <xacro:property name="imu_i2c_addr"   value="28"/>      <!-- I2C address: 28 = 0x28 (ADR pin low) -->
+  <xacro:property name="imu_axis_remap" value="P1"/>      <!-- Mounting orientation P0-P7, see BNO055 datasheet Table 3-4 -->
+  <xacro:property name="imu_sensor_mode" value="NDOF"/>   <!-- Fusion mode: NDOF, NDOF_FMC_OFF, IMUPLUS -->
   <!-- Motor IDs and mode -->
   <xacro:property name="left_motor_id" value="7"/>

File: lekiwi_description/urdf/base.urdf (robot description, URDF)
Before this commit: robot lekiwi, 9 links, 8 joints
Links:
- added link imu_frame
- added link imu_link, mass 0.01; collision mesh filename=../meshes/bno055_imu.stl; visual mesh filename=../meshes/bno055_imu.stl
Joints:
- added joint imu_frame_joint: type fixed, parent imu_link, child imu_frame, origin xyz=0 0 0 rpy=0 0 0
- added joint imu_joint: type fixed, parent base_link, child imu_link, origin xyz=-0.044 0 0.08 rpy=0 0 0
- joint back_wheel_joint: limit effort=2.942 velocity=4.218447166685513 -> effort=2.942 velocity=4.433204476989503
- joint camera_frame_joint: origin xyz=0 0 0 rpy=0 0 0 -> xyz=0 0 0 rpy=0 0 4.71238898038469
- joint left_wheel_joint: limit effort=2.942 velocity=4.218447166685513 -> effort=2.942 velocity=4.433204476989503
- joint right_wheel_joint: limit effort=2.942 velocity=4.218447166685513 -> effort=2.942 velocity=4.433204476989503

File: lekiwi_description/urdf/base.urdf.xacro (robot description, xacro)
@@ -5,6 +5,10 @@
   <xacro:include filename="$(find lekiwi_description)/urdf/base.control.xacro"/>
   <!-- Arguments -->
-  <xacro:arg name="serial_port" default="${serial_port}"/>
-  <xacro:arg name="use_mock" default="${use_mock}"/>
+  <xacro:arg name="serial_port"  default="${serial_port}"/>
+  <xacro:arg name="use_mock"     default="${use_mock}"/>
+  <xacro:arg name="i2c_bus"     default="${imu_i2c_bus}"/>
+  <xacro:arg name="i2c_addr"    default="${imu_i2c_addr}"/>
+  <xacro:arg name="axis_remap"  default="${imu_axis_remap}"/>
+  <xacro:arg name="sensor_mode" default="${imu_sensor_mode}"/>
   <!-- Define custom materials for base and wheels using color properties -->
   <material name="light_grey">
@@ -59,4 +63,26 @@
   <!-- Laser frame -->
   <link name="laser_frame"/>
+  <!-- BNO055 IMU link -->
+  <link name="imu_link">
+    <visual>
+      <origin xyz="0 0 0" rpy="0 0 0"/>
+      <geometry>
+        <mesh filename="package://lekiwi_description/meshes/bno055_imu.stl"/>
+      </geometry>
+      <material name="charcoal"/>
+    </visual>
+    <collision>
+      <origin xyz="0 0 0" rpy="0 0 0"/>
+      <geometry>
+        <mesh filename="package://lekiwi_description/meshes/bno055_imu.stl"/>
+      </geometry>
+    </collision>
+    <inertial>
+      <mass value="0.01"/>
+      <inertia ixx="0.00001" ixy="0.0" ixz="0.0" iyy="0.00001" iyz="0.0" izz="0.00001"/>
+    </inertial>
+  </link>
+  <!-- IMU frame -->
+  <link name="imu_frame"/>
   <!-- Camera link -->
   <link name="camera_link">
@@ -159,4 +185,16 @@
     <child link="laser_frame"/>
     <origin xyz="0 0 ${laser_frame_offset_z}" rpy="0 0 0"/>
+  </joint>
+  <!-- IMU fixed joint -->
+  <joint name="imu_joint" type="fixed">
+    <parent link="base_link"/>
+    <child link="imu_link"/>
+    <origin xyz="${imu_base_offset_x} 0 ${imu_base_offset_z}" rpy="0 0 0"/>
+  </joint>
+  <!-- imu_frame fixed joint -->
+  <joint name="imu_frame_joint" type="fixed">
+    <parent link="imu_link"/>
+    <child link="imu_frame"/>
+    <origin xyz="0 0 0" rpy="0 0 0"/>
   </joint>
   <!-- camera fixed joint -->
@@ -251,3 +289,30 @@
     </joint>
   </ros2_control>
+  <!-- ROS 2 CONTROL -->
+  <!-- Sensor interface (BNO055 IMU) -->
+  <ros2_control name="lekiwi_imu" type="sensor">
+    <hardware>
+      <plugin>bno055_hardware_interface/BNO055HardwareInterface</plugin>
+      <param name="i2c_bus">$(arg i2c_bus)</param>       <!-- I2C bus number (default: 1 → /dev/i2c-1) -->
+      <param name="i2c_addr">$(arg i2c_addr)</param>     <!-- I2C address in hex, no 0x prefix (default: 28 = 0x28) -->
+      <param name="axis_remap">$(arg axis_remap)</param> <!-- Axis placement config: P0-P7 (default: P1) -->
+      <param name="sensor_mode">$(arg sensor_mode)</param> <!-- Fusion mode: NDOF, NDOF_FMC_OFF, IMUPLUS (default: NDOF) -->
+      <param name="enable_mock">$(arg use_mock)</param>  <!-- Reuse the system-level mock flag -->
+    </hardware>
+    <sensor name="bno055">
+      <!-- Orientation (quaternion, unit norm) -->
+      <state_interface name="orientation.x"/>
+      <state_interface name="orientation.y"/>
+      <state_interface name="orientation.z"/>
+      <state_interface name="orientation.w"/>
+      <!-- Angular velocity (rad/s) -->
+      <state_interface name="angular_velocity.x"/>
+      <state_interface name="angular_velocity.y"/>
+      <state_interface name="angular_velocity.z"/>
+      <!-- Linear acceleration (m/s²), gravity-compensated -->
+      <state_interface name="linear_acceleration.x"/>
+      <state_interface name="linear_acceleration.y"/>
+      <state_interface name="linear_acceleration.z"/>
+    </sensor>
+  </ros2_control>
 </robot>

Commit message: update URDF

File: lekiwi_description/urdf/base.common.xacro (robot description, xacro)
@@ -1,10 +1,10 @@
 <?xml version="1.0"?>
 <robot xmlns:xacro="http://www.ros.org/wiki/xacro">
-  <!-- Color properties for base and wheels (RGBA) -->
+  <!-- Color properties (RGBA) -->
   <xacro:property name="light_grey_rgba" value="0.8 0.8 0.8 1.0"/>
   <xacro:property name="charcoal_rgba" value="0.15 0.15 0.15 1.0"/>
-  <!-- Base offsets -->
-  <xacro:property name="base_offset_rz" value="${3*pi/2}"/> <!-- Base mesh rotation about Z (rad) -->
-  <!-- Wheel offsets -->
+  <!-- Base mesh rotation about Z (rad) -->
+  <xacro:property name="base_offset_rz" value="${3*pi/2}"/>
+  <!-- Wheel mount offsets -->
   <xacro:property name="wheel_base_radius" value="0.132239"/>
   <xacro:property name="wheel_base_offset_z" value="0.01036"/>
@@ -12,9 +12,10 @@
   <xacro:property name="laser_base_offset_x" value="-0.045042"/>
   <xacro:property name="laser_base_offset_z" value="0.0915"/>
-  <xacro:property name="laser_offset_rx" value="${pi/2}"/> <!-- LIDAR mesh rotation about X (rad) -->
+  <xacro:property name="laser_offset_rx" value="${pi/2}"/>
   <!-- HD camera offsets from base_link -->
   <xacro:property name="camera_base_offset_x" value="0.114"/>
   <xacro:property name="camera_base_offset_z" value="0.026"/>
-  <xacro:property name="camera_offset_ry" value="${pi/2}"/> <!-- Camera mesh/joint rotation about Y (rad) -->
+  <xacro:property name="camera_offset_ry" value="${pi/2}"/>
+  <xacro:property name="camera_frame_offset_rz" value="${3*pi/2}"/>
   <!-- LDLidar frame offsets from laser_link -->
   <xacro:property name="laser_frame_offset_z" value="0.027"/>

File: lekiwi_description/urdf/base.control.xacro (robot description, xacro)
@@ -1,9 +1,14 @@
 <?xml version="1.0"?>
 <robot xmlns:xacro="http://www.ros.org/wiki/xacro">
-  <!-- Hardware interface parameters -->
+  <!-- Shared hardware interface parameters (single STS servo bus) -->
   <xacro:property name="serial_port" default="/dev/ttySERVO"/>
   <xacro:property name="baud_rate" default="1000000"/>
   <xacro:property name="use_mock" default="false"/>
   <xacro:property name="use_sync_write" default="true"/>
+  <!-- Base motor IDs and mode -->
+  <xacro:property name="left_motor_id" value="7"/>
+  <xacro:property name="back_motor_id" value="8"/>
+  <xacro:property name="right_motor_id" value="9"/>
+  <xacro:property name="base_operating_mode" value="1"/>  <!-- Velocity mode -->
   <!-- Motor-specific parameter (STS3215 default) -->
   <!-- Adjust for other motor models: STS3032 max=2900, STS3235 max=3400 -->
@@ -19,9 +24,4 @@
   <xacro:property name="imu_axis_remap" value="P1"/>      <!-- Mounting orientation P0-P7, see BNO055 datasheet Table 3-4 -->
   <xacro:property name="imu_sensor_mode" value="NDOF"/>   <!-- Fusion mode: NDOF, NDOF_FMC_OFF, IMUPLUS -->
-  <!-- Motor IDs and mode -->
-  <xacro:property name="left_motor_id" value="7"/>
-  <xacro:property name="back_motor_id" value="8"/>
-  <xacro:property name="right_motor_id" value="9"/>
-  <xacro:property name="operating_mode" value="1"/>  <!-- Velocity mode -->
   <!-- Wheel geometry for omnidirectional control -->
   <xacro:property name="wheel_radius" value="0.051"/>  <!-- meters -->
@@ -37,4 +37,4 @@
   <xacro:property name="max_linear_velocity_x" value="${wheel_radius * max_velocity_rads / (sqrt(3)/2)}"/>
   <xacro:property name="max_linear_velocity_y" value="${wheel_radius * max_velocity_rads / 1.0}"/>
-  <xacro:property name="max_angular_velocity_z" value="${wheel_radius * max_velocity_rads / wheel_base_offset}"/>
+  <xacro:property name="max_angular_velocity_z" value="${wheel_radius * max_velocity_rads / wheel_base_radius}"/>
 </robot>

File: lekiwi_description/urdf/base.urdf (robot description, URDF)
Before this commit: robot lekiwi, 11 links, 10 joints
Links:
- link back_wheel_link: geometry collision mesh filename=../meshes/base/omni_wheel.stl; visual mesh filename=../meshes/base/omni_wheel.stl
- link base_link: geometry collision mesh filename=../meshes/base/lekiwi_base.stl; visual mesh filename=../meshes/base/lekiwi_base.stl
- link camera_link: geometry collision mesh filename=../meshes/base/hd_webcam.stl; visual mesh filename=../meshes/base/hd_webcam.stl
- link imu_link: geometry collision mesh filename=../meshes/base/bno055_imu.stl; visual mesh filename=../meshes/base/bno055_imu.stl
- link laser_link: geometry collision mesh filename=../meshes/base/ld06_lidar.stl; visual mesh filename=../meshes/base/ld06_lidar.stl
- link left_wheel_link: geometry collision mesh filename=../meshes/base/omni_wheel.stl; visual mesh filename=../meshes/base/omni_wheel.stl
- link right_wheel_link: geometry collision mesh filename=../meshes/base/omni_wheel.stl; visual mesh filename=../meshes/base/omni_wheel.stl
Joints:
- joint back_wheel_joint: limit effort=2.942 velocity=4.433204476989503 -> effort=2.942 velocity=4.433204; origin xyz=-0.132239 1.6194606807244685e-17 0.01036 rpy=0 1.5707963267948966 3.141592653589793 -> xyz=-0.132239 0.000000 0.01036 rpy=0 1.5708 3.1416
- joint base_footprint_joint: origin xyz=0 0 0.040639999999999996 rpy=0 0 0 -> xyz=0 0 0.04064 rpy=0 0 0
- joint camera_frame_joint: origin xyz=0 0 0 rpy=0 0 4.71238898038469 -> xyz=0 0 0 rpy=0 0 4.7124
- joint camera_joint: origin xyz=0.114 0 0.026 rpy=0 1.5707963267948966 0 -> xyz=0.114 0 0.026 rpy=0 1.5708 0
- joint left_wheel_joint: limit effort=2.942 velocity=4.433204476989503 -> effort=2.942 velocity=4.433204; origin xyz=0.06611950000000001 0.11452233337105037 0.01036 rpy=0 1.5707963267948966 1.0471975511965976 -> xyz=0.066120 0.114522 0.01036 rpy=0 1.5708 1.0472
- joint right_wheel_joint: limit effort=2.942 velocity=4.433204476989503 -> effort=2.942 velocity=4.433204; origin xyz=0.06611950000000001 -0.11452233337105037 0.01036 rpy=0 1.5707963267948966 -1.0471975511965976 -> xyz=0.066120 -0.114522 0.01036 rpy=0 1.5708 -1.0472

File: lekiwi_description/urdf/base.urdf.xacro (robot description, xacro)
@@ -1,5 +1,5 @@
 <?xml version="1.0"?>
 <robot xmlns:xacro="http://www.ros.org/wiki/xacro" name="lekiwi">
-  <!-- Include robot properties -->
+  <!-- Include properties -->
   <xacro:include filename="$(find lekiwi_description)/urdf/base.common.xacro"/>
   <xacro:include filename="$(find lekiwi_description)/urdf/base.control.xacro"/>
@@ -11,5 +11,5 @@
   <xacro:arg name="axis_remap"  default="${imu_axis_remap}"/>
   <xacro:arg name="sensor_mode" default="${imu_sensor_mode}"/>
-  <!-- Define custom materials for base and wheels using color properties -->
+  <!-- Define custom materials for lekiwi color properties -->
   <material name="light_grey">
     <color rgba="${light_grey_rgba}"/>
@@ -26,5 +26,5 @@
       <origin xyz="0 0 0" rpy="0 0 ${base_offset_rz}"/>
       <geometry>
-        <mesh filename="package://lekiwi_description/meshes/lekiwi_base.stl"/>
+        <mesh filename="package://lekiwi_description/meshes/base/lekiwi_base.stl"/>
       </geometry>
       <material name="light_grey"/>
@@ -33,5 +33,5 @@
       <origin xyz="0 0 0" rpy="0 0 ${base_offset_rz}"/>
       <geometry>
-        <mesh filename="package://lekiwi_description/meshes/lekiwi_base.stl"/>
+        <mesh filename="package://lekiwi_description/meshes/base/lekiwi_base.stl"/>
       </geometry>
     </collision>
@@ -46,5 +46,5 @@
       <origin xyz="0 0 0" rpy="${laser_offset_rx} 0 0"/>
       <geometry>
-        <mesh filename="package://lekiwi_description/meshes/ld06_lidar.stl"/>
+        <mesh filename="package://lekiwi_description/meshes/base/ld06_lidar.stl"/>
       </geometry>
       <material name="charcoal"/>
@@ -53,5 +53,5 @@
       <origin xyz="0 0 0" rpy="${laser_offset_rx} 0 0"/>
       <geometry>
-        <mesh filename="package://lekiwi_description/meshes/ld06_lidar.stl"/>
+        <mesh filename="package://lekiwi_description/meshes/base/ld06_lidar.stl"/>
       </geometry>
     </collision>
@@ -68,12 +68,12 @@
       <origin xyz="0 0 0" rpy="0 0 0"/>
       <geometry>
-        <mesh filename="package://lekiwi_description/meshes/bno055_imu.stl"/>
-      </geometry>
-      <material name="charcoal"/>
-    </visual>
-    <collision>
-      <origin xyz="0 0 0" rpy="0 0 0"/>
-      <geometry>
-        <mesh filename="package://lekiwi_description/meshes/bno055_imu.stl"/>
+        <mesh filename="package://lekiwi_description/meshes/base/bno055_imu.stl"/>
+      </geometry>
+      <material name="charcoal"/>
+    </visual>
+    <collision>
+      <origin xyz="0 0 0" rpy="0 0 0"/>
+      <geometry>
+        <mesh filename="package://lekiwi_description/meshes/base/bno055_imu.stl"/>
       </geometry>
     </collision>
@@ -90,12 +90,12 @@
       <origin xyz="0 0 0" rpy="0 0 0"/>
       <geometry>
-        <mesh filename="package://lekiwi_description/meshes/hd_webcam.stl"/>
-      </geometry>
-      <material name="charcoal"/>
-    </visual>
-    <collision>
-      <origin xyz="0 0 0" rpy="0 0 0"/>
-      <geometry>
-        <mesh filename="package://lekiwi_description/meshes/hd_webcam.stl"/>
+        <mesh filename="package://lekiwi_description/meshes/base/hd_webcam.stl"/>
+      </geometry>
+      <material name="charcoal"/>
+    </visual>
+    <collision>
+      <origin xyz="0 0 0" rpy="0 0 0"/>
+      <geometry>
+        <mesh filename="package://lekiwi_description/meshes/base/hd_webcam.stl"/>
       </geometry>
     </collision>
@@ -112,12 +112,12 @@
       <origin xyz="0 0 0" rpy="0 0 0"/>
       <geometry>
-        <mesh filename="package://lekiwi_description/meshes/omni_wheel.stl"/>
-      </geometry>
-      <material name="charcoal"/>
-    </visual>
-    <collision>
-      <origin xyz="0 0 0" rpy="0 0 0"/>
-      <geometry>
-        <mesh filename="package://lekiwi_description/meshes/omni_wheel.stl"/>
+        <mesh filename="package://lekiwi_description/meshes/base/omni_wheel.stl"/>
+      </geometry>
+      <material name="charcoal"/>
+    </visual>
+    <collision>
+      <origin xyz="0 0 0" rpy="0 0 0"/>
+      <geometry>
+        <mesh filename="package://lekiwi_description/meshes/base/omni_wheel.stl"/>
       </geometry>
     </collision>
@@ -132,12 +132,12 @@
       <origin xyz="0 0 0" rpy="0 0 0"/>
       <geometry>
-        <mesh filename="package://lekiwi_description/meshes/omni_wheel.stl"/>
-      </geometry>
-      <material name="charcoal"/>
-    </visual>
-    <collision>
-      <origin xyz="0 0 0" rpy="0 0 0"/>
-      <geometry>
-        <mesh filename="package://lekiwi_description/meshes/omni_wheel.stl"/>
+        <mesh filename="package://lekiwi_description/meshes/base/omni_wheel.stl"/>
+      </geometry>
+      <material name="charcoal"/>
+    </visual>
+    <collision>
+      <origin xyz="0 0 0" rpy="0 0 0"/>
+      <geometry>
+        <mesh filename="package://lekiwi_description/meshes/base/omni_wheel.stl"/>
       </geometry>
     </collision>
@@ -152,12 +152,12 @@
       <origin xyz="0 0 0" rpy="0 0 0"/>
       <geometry>
-        <mesh filename="package://lekiwi_description/meshes/omni_wheel.stl"/>
-      </geometry>
-      <material name="charcoal"/>
-    </visual>
-    <collision>
-      <origin xyz="0 0 0" rpy="0 0 0"/>
-      <geometry>
-        <mesh filename="package://lekiwi_description/meshes/omni_wheel.stl"/>
+        <mesh filename="package://lekiwi_description/meshes/base/omni_wheel.stl"/>
+      </geometry>
+      <material name="charcoal"/>
+    </visual>
+    <collision>
+      <origin xyz="0 0 0" rpy="0 0 0"/>
+      <geometry>
+        <mesh filename="package://lekiwi_description/meshes/base/omni_wheel.stl"/>
       </geometry>
     </collision>
@@ -208,5 +208,5 @@
     <parent link="camera_link"/>
     <child link="camera"/>
-    <origin xyz="0 0 0" rpy="0 0 ${3*pi/2}"/>
+    <origin xyz="0 0 0" rpy="0 0 ${camera_frame_offset_rz}"/>
   </joint>
   <!-- left wheel joint: 60 degrees anti-clockwise from +X at radius wheel_base_radius -->
@@ -252,5 +252,5 @@
     <joint name="left_wheel_joint">
       <param name="motor_id">${left_motor_id}</param>
-      <param name="operating_mode">${operating_mode}</param>
+      <param name="operating_mode">${base_operating_mode}</param>
       <command_interface name="velocity"/>
       <state_interface name="position"/>
@@ -265,5 +265,5 @@
     <joint name="back_wheel_joint">
       <param name="motor_id">${back_motor_id}</param>
-      <param name="operating_mode">${operating_mode}</param>
+      <param name="operating_mode">${base_operating_mode}</param>
       <command_interface name="velocity"/>
       <state_interface name="position"/>
@@ -278,5 +278,5 @@
     <joint name="right_wheel_joint">
       <param name="motor_id">${right_motor_id}</param>
-      <param name="operating_mode">${operating_mode}</param>
+      <param name="operating_mode">${base_operating_mode}</param>
       <command_interface name="velocity"/>
       <state_interface name="position"/>
