Commit message: add pantilt urdf

File: lekiwi_description/urdf/base.common.xacro (robot description, xacro)
@@ -23,3 +23,6 @@
   <xacro:property name="imu_base_offset_x" value="-0.044"/>
   <xacro:property name="imu_base_offset_z" value="0.08"/>
+  <!-- Pan-tilt mount point on base_link (front-center, ~5.25cm high) -->
+  <xacro:property name="pantilt_base_offset_x" value="0.032725"/>
+  <xacro:property name="pantilt_base_offset_z" value="0.0525"/>
 </robot>

File: lekiwi_description/urdf/base.control.xacro (robot description, xacro)
@@ -1,9 +1,13 @@
 <?xml version="1.0"?>
 <robot xmlns:xacro="http://www.ros.org/wiki/xacro">
-  <!-- Shared hardware interface parameters (single STS servo bus) -->
-  <xacro:property name="serial_port" default="/dev/ttySERVO"/>
-  <xacro:property name="baud_rate" default="1000000"/>
-  <xacro:property name="use_mock" default="false"/>
-  <xacro:property name="use_sync_write" default="true"/>
+  <!-- Arguments (externally settable via command line) -->
+  <xacro:arg name="serial_port"  default="/dev/ttySERVO"/>
+  <xacro:arg name="baud_rate"    default="1000000"/>
+  <xacro:arg name="use_mock"     default="false"/>
+  <xacro:arg name="use_sync_write" default="true"/>
+  <xacro:arg name="i2c_bus"      default="1"/>
+  <xacro:arg name="i2c_addr"     default="28"/>
+  <xacro:arg name="axis_remap"   default="P1"/>
+  <xacro:arg name="sensor_mode"  default="NDOF"/>
   <!-- Base motor IDs and mode -->
   <xacro:property name="left_motor_id" value="7"/>
@@ -11,4 +15,13 @@
   <xacro:property name="right_motor_id" value="9"/>
   <xacro:property name="base_operating_mode" value="1"/>  <!-- Velocity mode -->
+  <!-- Pan-tilt motor IDs and mode (when use_pantilt:=true) -->
+  <xacro:property name="pan_motor_id" value="1"/>
+  <xacro:property name="tilt_motor_id" value="2"/>
+  <xacro:property name="pantilt_operating_mode" value="0"/>  <!-- Position mode -->
+  <!-- Pan and tilt joint limits -->
+  <xacro:property name="pan_joint_lower" value="-2"/>
+  <xacro:property name="pan_joint_upper" value="2"/>
+  <xacro:property name="tilt_joint_lower" value="${-pi/2}"/>
+  <xacro:property name="tilt_joint_upper" value="${pi/2}"/>
   <!-- Motor-specific parameter (STS3215 default) -->
   <!-- Adjust for other motor models: STS3032 max=2900, STS3235 max=3400 -->
@@ -19,9 +32,4 @@
   <!-- Set proportional_acc_max to 0 to disable (ACC=0 for all wheels). -->
   <xacro:property name="proportional_acc_max" value="25"/>        <!-- [0-254] -->
-  <!-- BNO055 IMU parameters -->
-  <xacro:property name="imu_i2c_bus"    value="1"/>       <!-- I2C bus number (/dev/i2c-1) -->
-  <xacro:property name="imu_i2c_addr"   value="28"/>      <!-- I2C address: 28 = 0x28 (ADR pin low) -->
-  <xacro:property name="imu_axis_remap" value="P1"/>      <!-- Mounting orientation P0-P7, see BNO055 datasheet Table 3-4 -->
-  <xacro:property name="imu_sensor_mode" value="NDOF"/>   <!-- Fusion mode: NDOF, NDOF_FMC_OFF, IMUPLUS -->
   <!-- Wheel geometry for omnidirectional control -->
   <xacro:property name="wheel_radius" value="0.051"/>  <!-- meters -->
@@ -37,4 +45,122 @@
   <xacro:property name="max_linear_velocity_x" value="${wheel_radius * max_velocity_rads / (sqrt(3)/2)}"/>
   <xacro:property name="max_linear_velocity_y" value="${wheel_radius * max_velocity_rads / 1.0}"/>
-  <xacro:property name="max_angular_velocity_z" value="${wheel_radius * max_velocity_rads / wheel_base_radius}"/>
+  <!-- ROS 2 CONTROL -->
+  <!-- System interface (STS motors) -->
+  <ros2_control name="lekiwi_base" type="system">
+    <hardware>
+      <plugin>sts_hardware_interface/STSHardwareInterface</plugin>
+      <!-- Serial communication parameters -->
+      <param name="serial_port">$(arg serial_port)</param>
+      <param name="baud_rate">$(arg baud_rate)</param>
+      <param name="use_sync_write">$(arg use_sync_write)</param>
+      <param name="enable_mock_mode">$(arg use_mock)</param>
+      <!-- Motor-specific parameter (adjust for different STS motor models) -->
+      <param name="max_velocity_steps">${sts_max_velocity_steps}</param>
+      <!-- Proportional ACC: scale per-wheel acceleration so all wheels finish ramping in equal time -->
+      <param name="proportional_acc_max">${proportional_acc_max}</param>
+    </hardware>
+    <!-- Left wheel joint (Motor ID 7) -->
+    <joint name="left_wheel_joint">
+      <param name="motor_id">${left_motor_id}</param>
+      <param name="operating_mode">${base_operating_mode}</param>
+      <command_interface name="velocity"/>
+      <state_interface name="position"/>
+      <state_interface name="velocity"/>
+      <state_interface name="effort"/>
+      <state_interface name="voltage"/>
+      <state_interface name="temperature"/>
+      <state_interface name="current"/>
+      <state_interface name="is_moving"/>
+    </joint>
+    <!-- Back wheel joint (Motor ID 8) -->
+    <joint name="back_wheel_joint">
+      <param name="motor_id">${back_motor_id}</param>
+      <param name="operating_mode">${base_operating_mode}</param>
+      <command_interface name="velocity"/>
+      <state_interface name="position"/>
+      <state_interface name="velocity"/>
+      <state_interface name="effort"/>
+      <state_interface name="voltage"/>
+      <state_interface name="temperature"/>
+      <state_interface name="current"/>
+      <state_interface name="is_moving"/>
+    </joint>
+    <!-- Right wheel joint (Motor ID 9) -->
+    <joint name="right_wheel_joint">
+      <param name="motor_id">${right_motor_id}</param>
+      <param name="operating_mode">${base_operating_mode}</param>
+      <command_interface name="velocity"/>
+      <state_interface name="position"/>
+      <state_interface name="velocity"/>
+      <state_interface name="effort"/>
+      <state_interface name="voltage"/>
+      <state_interface name="temperature"/>
+      <state_interface name="current"/>
+      <state_interface name="is_moving"/>
+    </joint>
+    <!-- Pan and tilt joints (when use_pantilt:=true, shares same hardware interface) -->
+    <xacro:if value="$(arg use_pantilt)">
+      <!-- Pan axis: rotates the payload around Z (Motor ID 1) -->
+      <joint name="pan_joint">
+        <param name="motor_id">${pan_motor_id}</param>
+        <param name="operating_mode">${pantilt_operating_mode}</param>
+        <param name="min_position">${pan_joint_lower}</param>
+        <param name="max_position">${pan_joint_upper}</param>
+        <param name="max_velocity">${max_velocity_rads}</param>
+        <param name="position_center_steps">2048</param>
+        <command_interface name="position"/>
+        <state_interface name="position"/>
+        <state_interface name="velocity"/>
+        <state_interface name="effort"/>
+        <state_interface name="voltage"/>
+        <state_interface name="temperature"/>
+        <state_interface name="current"/>
+        <state_interface name="is_moving"/>
+      </joint>
+      <!-- Tilt axis: rotates the payload around Y (Motor ID 2) -->
+      <joint name="tilt_joint">
+        <param name="motor_id">${tilt_motor_id}</param>
+        <param name="operating_mode">${pantilt_operating_mode}</param>
+        <param name="min_position">${tilt_joint_lower}</param>
+        <param name="max_position">${tilt_joint_upper}</param>
+        <param name="max_velocity">${max_velocity_rads}</param>
+        <param name="position_center_steps">2048</param>
+        <command_interface name="position"/>
+        <state_interface name="position"/>
+        <state_interface name="velocity"/>
+        <state_interface name="effort"/>
+        <state_interface name="voltage"/>
+        <state_interface name="temperature"/>
+        <state_interface name="current"/>
+        <state_interface name="is_moving"/>
+      </joint>
+    </xacro:if>
+  </ros2_control>
+  <!-- ROS 2 CONTROL -->
+  <!-- Sensor interface (BNO055 IMU) -->
+  <ros2_control name="lekiwi_imu" type="sensor">
+    <hardware>
+      <plugin>bno055_hardware_interface/BNO055HardwareInterface</plugin>
+      <param name="i2c_bus">$(arg i2c_bus)</param>       <!-- I2C bus number (default: 1 → /dev/i2c-1) -->
+      <param name="i2c_addr">$(arg i2c_addr)</param>     <!-- I2C address in hex, no 0x prefix (default: 28 = 0x28) -->
+      <param name="axis_remap">$(arg axis_remap)</param> <!-- Axis placement config: P0-P7 (default: P1) -->
+      <param name="sensor_mode">$(arg sensor_mode)</param> <!-- Fusion mode: NDOF, NDOF_FMC_OFF, IMUPLUS (default: NDOF) -->
+      <param name="enable_mock_mode">$(arg use_mock)</param>  <!-- Reuse the system-level mock flag -->
+    </hardware>
+    <sensor name="bno055">
+      <!-- Orientation (quaternion, unit norm) -->
+      <state_interface name="orientation.x"/>
+      <state_interface name="orientation.y"/>
+      <state_interface name="orientation.z"/>
+      <state_interface name="orientation.w"/>
+      <!-- Angular velocity (rad/s) -->
+      <state_interface name="angular_velocity.x"/>
+      <state_interface name="angular_velocity.y"/>
+      <state_interface name="angular_velocity.z"/>
+      <!-- Linear acceleration (m/s²), gravity-compensated -->
+      <state_interface name="linear_acceleration.x"/>
+      <state_interface name="linear_acceleration.y"/>
+      <state_interface name="linear_acceleration.z"/>
+    </sensor>
+  </ros2_control>
 </robot>

File: lekiwi_description/urdf/base.urdf.xacro (robot description, xacro)
@@ -4,11 +4,7 @@
   <xacro:include filename="$(find lekiwi_description)/urdf/base.common.xacro"/>
   <xacro:include filename="$(find lekiwi_description)/urdf/base.control.xacro"/>
-  <!-- Arguments -->
-  <xacro:arg name="serial_port"  default="${serial_port}"/>
-  <xacro:arg name="use_mock"     default="${use_mock}"/>
-  <xacro:arg name="i2c_bus"     default="${imu_i2c_bus}"/>
-  <xacro:arg name="i2c_addr"    default="${imu_i2c_addr}"/>
-  <xacro:arg name="axis_remap"  default="${imu_axis_remap}"/>
-  <xacro:arg name="sensor_mode" default="${imu_sensor_mode}"/>
+  <!-- Optional pan-tilt module -->
+  <xacro:arg name="use_pantilt" default="false"/>
+  <xacro:include filename="$(find lepantilt_description)/urdf/pantilt.module.xacro"/>
   <!-- Define custom materials for lekiwi color properties -->
   <material name="light_grey">
@@ -234,85 +230,10 @@
     <limit effort="${max_torque_nm}" velocity="${max_velocity_rads}"/>
   </joint>
-  <!-- ROS 2 CONTROL -->
-  <!-- System interface -->
-  <ros2_control name="lekiwi_base" type="system">
-    <hardware>
-      <plugin>sts_hardware_interface/STSHardwareInterface</plugin>
-      <!-- Serial communication parameters -->
-      <param name="serial_port">$(arg serial_port)</param>
-      <param name="baud_rate">${baud_rate}</param>
-      <param name="use_sync_write">${use_sync_write}</param>
-      <param name="enable_mock_mode">$(arg use_mock)</param>
-      <!-- Motor-specific parameter (adjust for different STS motor models) -->
-      <param name="max_velocity_steps">${sts_max_velocity_steps}</param>
-      <!-- Proportional ACC: scale per-wheel acceleration so all wheels finish ramping in equal time -->
-      <param name="proportional_acc_max">${proportional_acc_max}</param>
-    </hardware>
-    <!-- Left wheel joint (Motor ID 7) -->
-    <joint name="left_wheel_joint">
-      <param name="motor_id">${left_motor_id}</param>
-      <param name="operating_mode">${base_operating_mode}</param>
-      <command_interface name="velocity"/>
-      <state_interface name="position"/>
-      <state_interface name="velocity"/>
-      <state_interface name="effort"/>
-      <state_interface name="voltage"/>
-      <state_interface name="temperature"/>
-      <state_interface name="current"/>
-      <state_interface name="is_moving"/>
-    </joint>
-    <!-- Back wheel joint (Motor ID 8) -->
-    <joint name="back_wheel_joint">
-      <param name="motor_id">${back_motor_id}</param>
-      <param name="operating_mode">${base_operating_mode}</param>
-      <command_interface name="velocity"/>
-      <state_interface name="position"/>
-      <state_interface name="velocity"/>
-      <state_interface name="effort"/>
-      <state_interface name="voltage"/>
-      <state_interface name="temperature"/>
-      <state_interface name="current"/>
-      <state_interface name="is_moving"/>
-    </joint>
-    <!-- Right wheel joint (Motor ID 9) -->
-    <joint name="right_wheel_joint">
-      <param name="motor_id">${right_motor_id}</param>
-      <param name="operating_mode">${base_operating_mode}</param>
-      <command_interface name="velocity"/>
-      <state_interface name="position"/>
-      <state_interface name="velocity"/>
-      <state_interface name="effort"/>
-      <state_interface name="voltage"/>
-      <state_interface name="temperature"/>
-      <state_interface name="current"/>
-      <state_interface name="is_moving"/>
-    </joint>
-  </ros2_control>
-  <!-- ROS 2 CONTROL -->
-  <!-- Sensor interface (BNO055 IMU) -->
-  <ros2_control name="lekiwi_imu" type="sensor">
-    <hardware>
-      <plugin>bno055_hardware_interface/BNO055HardwareInterface</plugin>
-      <param name="i2c_bus">$(arg i2c_bus)</param>       <!-- I2C bus number (default: 1 → /dev/i2c-1) -->
-      <param name="i2c_addr">$(arg i2c_addr)</param>     <!-- I2C address in hex, no 0x prefix (default: 28 = 0x28) -->
-      <param name="axis_remap">$(arg axis_remap)</param> <!-- Axis placement config: P0-P7 (default: P1) -->
-      <param name="sensor_mode">$(arg sensor_mode)</param> <!-- Fusion mode: NDOF, NDOF_FMC_OFF, IMUPLUS (default: NDOF) -->
-      <param name="enable_mock_mode">$(arg use_mock)</param>  <!-- Reuse the system-level mock flag -->
-    </hardware>
-    <sensor name="bno055">
-      <!-- Orientation (quaternion, unit norm) -->
-      <state_interface name="orientation.x"/>
-      <state_interface name="orientation.y"/>
-      <state_interface name="orientation.z"/>
-      <state_interface name="orientation.w"/>
-      <!-- Angular velocity (rad/s) -->
-      <state_interface name="angular_velocity.x"/>
-      <state_interface name="angular_velocity.y"/>
-      <state_interface name="angular_velocity.z"/>
-      <!-- Linear acceleration (m/s²), gravity-compensated -->
-      <state_interface name="linear_acceleration.x"/>
-      <state_interface name="linear_acceleration.y"/>
-      <state_interface name="linear_acceleration.z"/>
-    </sensor>
-  </ros2_control>
+  <!-- Optional pan-tilt module (mounted on front-center of base) -->
+  <xacro:if value="$(arg use_pantilt)">
+    <xacro:lepantilt_module parent="base_link">
+      <origin xyz="${pantilt_base_offset_x} 0 ${pantilt_base_offset_z}" rpy="0 0 0"/>
+      <!-- OAK-D mesh color enforced as charcoal (0.15 0.15 0.15 1.0) in pantilt.module.xacro and base_pantilt.urdf -->
+    </xacro:lepantilt_module>
+  </xacro:if>
 </robot>

File: lekiwi_description/urdf/base_pantilt.urdf (robot description, URDF)
Before this commit: robot lekiwi, 11 links, 10 joints
Links:
- added link oak_imu_frame
- added link oak_link
- added link oak_link_left_camera_frame
- added link oak_link_left_camera_optical_frame
- added link oak_link_model_origin; visual mesh filename=../meshes/pantilt/oakd_s2.stl
- added link oak_link_rgb_camera_frame
- added link oak_link_rgb_camera_optical_frame
- added link oak_link_right_camera_frame
- added link oak_link_right_camera_optical_frame
- added link pan_link, mass 0.119226; collision mesh filename=../meshes/pantilt/pan_joint.stl; visual mesh filename=../meshes/pantilt/pan_joint.stl
- added link pantilt_base_link, mass 1.0; collision mesh filename=../meshes/pantilt/pantilt_base.stl; visual mesh filename=../meshes/pantilt/pan_motor.stl
- added link tilt_link, mass 0.1; collision mesh filename=../meshes/pantilt/tilt_joint.stl; visual mesh filename=../meshes/pantilt/tilt_joint.stl
Joints:
- added joint oak_imu_joint: type fixed, parent oak_link, child oak_imu_frame, origin xyz=-0.008 -0.037945 -0.00079 rpy=3.141592653589793 1.5707963267948966 0
- added joint oak_link_center_joint: type fixed, parent tilt_link, child oak_link, origin xyz=-0.03435 -0.01 0 rpy=-1.5707963267948966 0 -1.5707963267948966
- added joint oak_link_left_camera_joint: type fixed, parent oak_link, child oak_link_left_camera_frame, origin xyz=0 0.0375 0 rpy=0 0 0
- added joint oak_link_left_camera_optical_joint: type fixed, parent oak_link_left_camera_frame, child oak_link_left_camera_optical_frame, origin xyz=0 0 0 rpy=-1.5707963267948966 0.0 -1.5707963267948966
- added joint oak_link_model_origin_joint: type fixed, parent oak_link, child oak_link_model_origin, origin xyz=0 0 0 rpy=1.5708 0 1.5708
- added joint oak_link_rgb_camera_joint: type fixed, parent oak_link, child oak_link_rgb_camera_frame, origin xyz=0 0 0 rpy=0 0 0
- added joint oak_link_rgb_camera_optical_joint: type fixed, parent oak_link_rgb_camera_frame, child oak_link_rgb_camera_optical_frame, origin xyz=0 0 0 rpy=-1.5707963267948966 0.0 -1.5707963267948966
- added joint oak_link_right_camera_joint: type fixed, parent oak_link, child oak_link_right_camera_frame, origin xyz=0 -0.0375 0 rpy=0 0 0
- added joint oak_link_right_camera_optical_joint: type fixed, parent oak_link_right_camera_frame, child oak_link_right_camera_optical_frame, origin xyz=0 0 0 rpy=-1.5707963267948966 0.0 -1.5707963267948966
- added joint pan_joint: type revolute, parent pantilt_base_link, child pan_link, origin xyz=0.0452 0 0.0165 rpy=0 0 0, axis 0 0 1, limit lower=-2 upper=2 effort=2.942 velocity=4.433204476989503
- added joint pantilt_mount_joint: type fixed, parent base_link, child pantilt_base_link, origin xyz=0.032725 0 0.0525 rpy=0 0 0
- added joint tilt_joint: type revolute, parent pan_link, child tilt_link, origin xyz=0.0306 0 0.1025 rpy=-1.5707963267948966 1.5707963267948966 0, axis 0 0 1, limit lower=-1.5707963267948966 upper=1.5707963267948966 effort=2.942 velocity=4.433204476989503
