Commit message: update pantilt tilt_joint stl and offsets

File: lekiwi_description/urdf/pantilt/pantilt.urdf (robot description, URDF)
Before this commit: robot pantilt, 7 links, 6 joints
Joints:
- joint oak_link_center_joint: origin xyz=-0.03435 -0.01 0 rpy=-1.5707963267948966 0 -1.5707963267948966 -> xyz=-0.0306 -0.012165 0 rpy=-1.5707963267948966 0 -1.5707963267948966
