Commit message: Refactor control & navigation; add twist_switch_node; fix configs
lekiwi_control (ament_cmake -> ament_python):
- Add twist_switch_node: velocity mux with /twist_switch SetBool service,
  watchdog timeout, and no-publisher guard
- Rename lekiwi.launch.py -> control.launch.py; add gated joy_node (joy arg)
- Move bno055 static params to config/bno055_diagnostics.yaml
- Move pan/tilt xacro args to config/{k2,pantilt}/urdf_config.yaml
- Rename serial_port -> sts_serial_port; remove teleop_config arg (derived inline)
- Add config/twist_switch.yaml; update teleop.yaml for /twist_switch service

lekiwi_bringup:
- Add control_diagnostics, control_mock, sts_serial_port args; forward to control

lekiwi_navigation (ament_cmake -> ament_python):
- Rename nav.launch.py -> navigation.launch.py
- Extract EKF into ekf.launch.py (fusion_mode: base/imu/odom)
- Extract nav2/AMCL logic into nav2.launch.py
- Add map_saver_node; fix map save button X -> R1 (button 5)
- Add os.path.realpath comment in nav2.launch.py

lekiwi_description:
- Regenerate base.urdf, k2.urdf, pantilt.urdf from xacro with default args

.gitignore: ignore lekiwi_navigation/maps/* subdirectories

File: lekiwi_description/urdf/base/base.urdf (robot description, URDF)
Before this commit: robot lekiwi, 11 links, 10 joints
Links:
- link back_wheel_link: geometry collision mesh filename=../meshes/base/omni_wheel.stl; visual mesh filename=../meshes/base/omni_wheel.stl
- link base_link: geometry collision mesh filename=../meshes/base/lekiwi_base.stl; visual mesh filename=../meshes/base/lekiwi_base.stl
- link camera_link: geometry collision mesh filename=../meshes/base/hd_webcam.stl; visual mesh filename=../meshes/base/hd_webcam.stl
- link imu_link: geometry collision mesh filename=../meshes/base/bno055_imu.stl; visual mesh filename=../meshes/base/bno055_imu.stl
- link laser_link: geometry collision mesh filename=../meshes/base/ld06_lidar.stl; visual mesh filename=../meshes/base/ld06_lidar.stl
- link left_wheel_link: geometry collision mesh filename=../meshes/base/omni_wheel.stl; visual mesh filename=../meshes/base/omni_wheel.stl
- link right_wheel_link: geometry collision mesh filename=../meshes/base/omni_wheel.stl; visual mesh filename=../meshes/base/omni_wheel.stl

File: lekiwi_description/urdf/k2.urdf (robot description, URDF)
Before this commit: robot k2, 17 links, 16 joints
Joints:
- joint oak_link_center_joint: origin xyz=-0.03435 -0.01 0 rpy=-1.5707963267948966 0 -1.5707963267948966 -> xyz=-0.0306 -0.012165 0 rpy=-1.5707963267948966 0 -1.5707963267948966

File: lekiwi_description/urdf/pantilt/pantilt.control.xacro (robot description, xacro)
@@ -22,5 +22,5 @@
   <xacro:property name="tilt_joint_upper" value="${pi/2}"/>
   <!-- ROS 2 CONTROL -->
-  <ros2_control name="pt100_control" type="system">
+  <ros2_control name="pantilt_control" type="system">
     <hardware>
       <plugin>sts_hardware_interface/STSHardwareInterface</plugin>

File: lekiwi_description/urdf/pantilt/pantilt.urdf (robot description, URDF)
Before this commit: robot pantilt, 7 links, 6 joints
Links:
- link oak_link_model_origin: geometry visual mesh filename=../meshes/pantilt/oakd_s2.stl
- link pan_link: geometry collision mesh filename=../meshes/pantilt/pan_joint.stl; visual mesh filename=../meshes/pantilt/pan_joint.stl
- link pantilt_base_link: geometry collision mesh filename=../meshes/pantilt/pantilt_base.stl; visual mesh filename=../meshes/pantilt/pan_motor.stl
- link tilt_link: geometry collision mesh filename=../meshes/pantilt/tilt_joint.stl; visual mesh filename=../meshes/pantilt/tilt_joint.stl

Commit message: update package.xmls, setup.py and generated URDF mesh paths

File: lekiwi_description/urdf/base/base.urdf (robot description, URDF)
Before this commit: robot lekiwi, 9 links, 8 joints
Links:
- link back_wheel_link: geometry collision mesh filename=../../meshes/base/omni_wheel.stl; visual mesh filename=../../meshes/base/omni_wheel.stl
- link base_link: geometry collision mesh filename=../../meshes/base/lekiwi_base.stl; visual mesh filename=../../meshes/base/lekiwi_base.stl
- link imu_link: geometry collision mesh filename=../../meshes/base/bno055_imu.stl; visual mesh filename=../../meshes/base/bno055_imu.stl
- link laser_link: geometry collision mesh filename=../../meshes/base/ld06_lidar.stl; visual mesh filename=../../meshes/base/ld06_lidar.stl
- link left_wheel_link: geometry collision mesh filename=../../meshes/base/omni_wheel.stl; visual mesh filename=../../meshes/base/omni_wheel.stl
- link right_wheel_link: geometry collision mesh filename=../../meshes/base/omni_wheel.stl; visual mesh filename=../../meshes/base/omni_wheel.stl

File: lekiwi_description/urdf/pantilt/pantilt.urdf (robot description, URDF)
Before this commit: robot pantilt, 7 links, 6 joints
Links:
- link oak_link_model_origin: geometry visual mesh filename=../../meshes/pantilt/oakd_s2.stl
- link pan_link: geometry collision mesh filename=../../meshes/pantilt/pan_joint.stl; visual mesh filename=../../meshes/pantilt/pan_joint.stl
- link pantilt_base_link: geometry collision mesh filename=../../meshes/pantilt/pantilt_base.stl; visual mesh filename=../../meshes/pantilt/pan_motor.stl
- link tilt_link: geometry collision mesh filename=../../meshes/pantilt/tilt_joint.stl; visual mesh filename=../../meshes/pantilt/tilt_joint.stl
