Commit message: feat: add package test suites, reorganize payload configs, enable service introspection
- Add pytest suites for lekiwi_control, lekiwi_navigation, lekiwi_description, lekiwi_bringup
- Move laser_filter.yaml under config/payloads/pantilt/, split toggles.yaml out of teleop.yaml
- Enable service introspection (configure_introspection) on /twist_switch, /record_waypoint,
  /waypoint_follow, /reset_waypoints, /save_map, matching the existing /emergency_stop setup -
  lets a listener observe every call's request+response regardless of caller (prep for an
  upcoming audio status-indicator node, not yet included in this commit)

Co-Authored-By: Claude Sonnet 5 <noreply@anthropic.com>

File: lekiwi_description/urdf/base/base.urdf (robot description, URDF)
Before this commit: robot lekiwi, 10 links, 9 joints
Links:
- link back_wheel_link: geometry collision mesh filename=package://lekiwi_description/meshes/omni_wheel.stl; visual mesh filename=package://lekiwi_description/meshes/omni_wheel.stl
- link base_link: geometry collision mesh filename=package://lekiwi_description/meshes/lekiwi_base.stl; visual mesh filename=package://lekiwi_description/meshes/lekiwi_base.stl
- link imu_link: geometry collision mesh filename=package://lekiwi_description/meshes/bno055_imu.stl; visual mesh filename=package://lekiwi_description/meshes/bno055_imu.stl
- link laser_link: geometry collision mesh filename=package://lekiwi_description/meshes/ld06_lidar.stl; visual mesh filename=package://lekiwi_description/meshes/ld06_lidar.stl
- link left_wheel_link: geometry collision mesh filename=package://lekiwi_description/meshes/omni_wheel.stl; visual mesh filename=package://lekiwi_description/meshes/omni_wheel.stl
- link mic_link: geometry collision mesh filename=package://lekiwi_description/meshes/respeaker_flex_mic.stl; visual mesh filename=package://lekiwi_description/meshes/respeaker_flex_mic.stl
- link right_wheel_link: geometry collision mesh filename=package://lekiwi_description/meshes/omni_wheel.stl; visual mesh filename=package://lekiwi_description/meshes/omni_wheel.stl

File: lekiwi_description/urdf/base_pantilt/base_pantilt.urdf (robot description, URDF)
Before this commit: robot lekiwi, 16 links, 15 joints
Links:
- link back_wheel_link: geometry collision mesh filename=package://lekiwi_description/meshes/omni_wheel.stl; visual mesh filename=package://lekiwi_description/meshes/omni_wheel.stl
- link base_link: geometry collision mesh filename=package://lekiwi_description/meshes/lekiwi_base.stl; visual mesh filename=package://lekiwi_description/meshes/lekiwi_base.stl
- link imu_link: geometry collision mesh filename=package://lekiwi_description/meshes/bno055_imu.stl; visual mesh filename=package://lekiwi_description/meshes/bno055_imu.stl
- link laser_link: geometry collision mesh filename=package://lekiwi_description/meshes/ld06_lidar.stl; visual mesh filename=package://lekiwi_description/meshes/ld06_lidar.stl
- link left_wheel_link: geometry collision mesh filename=package://lekiwi_description/meshes/omni_wheel.stl; visual mesh filename=package://lekiwi_description/meshes/omni_wheel.stl
- link mic_link: geometry collision mesh filename=package://lekiwi_description/meshes/respeaker_flex_mic.stl; visual mesh filename=package://lekiwi_description/meshes/respeaker_flex_mic.stl
- link oak_link_model_origin: geometry visual mesh filename=package://pt_description/meshes/oakd_s2.stl
- link pan_link: geometry collision mesh filename=package://pt_description/meshes/pan_joint_101.stl; visual mesh filename=package://pt_description/meshes/pan_joint_101.stl
- link pantilt_base_link: geometry collision mesh filename=package://pt_description/meshes/pantilt_base_101.stl; visual mesh filename=package://pt_description/meshes/pan_motor.stl
- link right_wheel_link: geometry collision mesh filename=package://lekiwi_description/meshes/omni_wheel.stl; visual mesh filename=package://lekiwi_description/meshes/omni_wheel.stl
- link tilt_link: geometry collision mesh filename=package://pt_description/meshes/tilt_joint_oakd_s2.stl; visual mesh filename=package://pt_description/meshes/tilt_joint_oakd_s2.stl

Commit message: Fix stale prebuilt URDFs; drop pantilt's own internal_control_period
TestPrebuiltUrdfConsistency was failing in CI: the committed base.urdf and
base_pantilt.urdf no longer matched their xacro sources. base.urdf had
plain relative mesh paths instead of package:// URIs (regenerated wrong by
the previous urdf_config.yaml commit), and base_pantilt.urdf still carried
years-stale raw.githubusercontent.com/.../pantilt100/... mesh URLs from
before that submodule was renamed to pantilt_ros2 and switched to
package://. Regenerated both from source with xacro, matching the test's
exact args.

Also drops the pantilt-specific internal_control_period override (20) -
pantilt now shares the base's value (10) rather than diverging from it.
Updated TestUrdfConfigPantilt accordingly.

Co-Authored-By: Claude Sonnet 5 <noreply@anthropic.com>

File: lekiwi_description/urdf/base/base.urdf (robot description, URDF)
Before this commit: robot lekiwi, 10 links, 9 joints
Links:
- link back_wheel_link: geometry collision mesh filename=package://lekiwi_description/meshes/omni_wheel.stl; visual mesh filename=package://lekiwi_description/meshes/omni_wheel.stl
- link base_link: geometry collision mesh filename=package://lekiwi_description/meshes/lekiwi_base.stl; visual mesh filename=package://lekiwi_description/meshes/lekiwi_base.stl
- link imu_link: geometry collision mesh filename=package://lekiwi_description/meshes/bno055_imu.stl; visual mesh filename=package://lekiwi_description/meshes/bno055_imu.stl
- link laser_link: geometry collision mesh filename=package://lekiwi_description/meshes/ld06_lidar.stl; visual mesh filename=package://lekiwi_description/meshes/ld06_lidar.stl
- link left_wheel_link: geometry collision mesh filename=package://lekiwi_description/meshes/omni_wheel.stl; visual mesh filename=package://lekiwi_description/meshes/omni_wheel.stl
- link mic_link: geometry collision mesh filename=package://lekiwi_description/meshes/respeaker_flex_mic.stl; visual mesh filename=package://lekiwi_description/meshes/respeaker_flex_mic.stl
- link right_wheel_link: geometry collision mesh filename=package://lekiwi_description/meshes/omni_wheel.stl; visual mesh filename=package://lekiwi_description/meshes/omni_wheel.stl

File: lekiwi_description/urdf/base_pantilt/base_pantilt.urdf (robot description, URDF)
Before this commit: robot lekiwi, 16 links, 15 joints
Links:
- link back_wheel_link: geometry collision mesh filename=package://lekiwi_description/meshes/omni_wheel.stl; visual mesh filename=package://lekiwi_description/meshes/omni_wheel.stl
- link base_link: geometry collision mesh filename=package://lekiwi_description/meshes/lekiwi_base.stl; visual mesh filename=package://lekiwi_description/meshes/lekiwi_base.stl
- link imu_link: geometry collision mesh filename=package://lekiwi_description/meshes/bno055_imu.stl; visual mesh filename=package://lekiwi_description/meshes/bno055_imu.stl
- link laser_link: geometry collision mesh filename=package://lekiwi_description/meshes/ld06_lidar.stl; visual mesh filename=package://lekiwi_description/meshes/ld06_lidar.stl
- link left_wheel_link: geometry collision mesh filename=package://lekiwi_description/meshes/omni_wheel.stl; visual mesh filename=package://lekiwi_description/meshes/omni_wheel.stl
- link mic_link: geometry collision mesh filename=package://lekiwi_description/meshes/respeaker_flex_mic.stl; visual mesh filename=package://lekiwi_description/meshes/respeaker_flex_mic.stl
- link oak_link_model_origin: geometry visual mesh filename=package://pt_description/meshes/oakd_s2.stl
- link pantilt_base_link: geometry collision mesh filename=package://pt_description/meshes/pantilt_base_101.stl; visual mesh filename=package://pt_description/meshes/pan_motor.stl
- link right_wheel_link: geometry collision mesh filename=package://lekiwi_description/meshes/omni_wheel.stl; visual mesh filename=package://lekiwi_description/meshes/omni_wheel.stl
- link shoulder_link: geometry collision mesh filename=package://pt_description/meshes/pan_joint_101.stl; visual mesh filename=package://pt_description/meshes/pan_joint_101.stl
- link tilt_link: geometry collision mesh filename=package://pt_description/meshes/tilt_joint_oakd_s2.stl; visual mesh filename=package://pt_description/meshes/tilt_joint_oakd_s2.stl

Commit message: Regenerate the pre-built URDFs with portable mesh paths; drop test_without_ros and the Windows CI job
Local meshes use relative paths, the pan-tilt meshes use raw GitHub URLs, and the staleness test applies the same rewrite. Regenerate with python3 lekiwi_description/test/test_urdf_xacro.py --write.

Co-Authored-By: Claude Sonnet 5 <noreply@anthropic.com>

File: lekiwi_description/urdf/base/base.urdf (robot description, URDF)
Before this commit: robot lekiwi, 10 links, 9 joints
Links:
- link back_wheel_link: geometry collision mesh filename=../../meshes/omni_wheel.stl scale=1.0 1.0 1.0; visual mesh filename=../../meshes/omni_wheel.stl scale=1.0 1.0 1.0
- link base_link: geometry collision mesh filename=../../meshes/lekiwi_base.stl; visual mesh filename=../../meshes/lekiwi_base.stl
- link imu_link: geometry collision mesh filename=../../meshes/bno055_imu.stl; visual mesh filename=../../meshes/bno055_imu.stl
- link laser_link: geometry collision mesh filename=../../meshes/ld06_lidar.stl; visual mesh filename=../../meshes/ld06_lidar.stl
- link left_wheel_link: geometry collision mesh filename=../../meshes/omni_wheel.stl scale=1.0 1.0 1.0; visual mesh filename=../../meshes/omni_wheel.stl scale=1.0 1.0 1.0
- link mic_link: geometry collision mesh filename=../../meshes/respeaker_flex_mic.stl; visual mesh filename=../../meshes/respeaker_flex_mic.stl
- link right_wheel_link: geometry collision mesh filename=../../meshes/omni_wheel.stl scale=1.0 1.0 1.0; visual mesh filename=../../meshes/omni_wheel.stl scale=1.0 1.0 1.0

File: lekiwi_description/urdf/base_pantilt/base_pantilt.urdf (robot description, URDF)
Before this commit: robot lekiwi, 16 links, 15 joints
Links:
- link back_wheel_link: geometry collision mesh filename=../../meshes/omni_wheel.stl scale=1.0 1.0 1.0; visual mesh filename=../../meshes/omni_wheel.stl scale=1.0 1.0 1.0
- link base_link: geometry collision mesh filename=../../meshes/lekiwi_base.stl; visual mesh filename=../../meshes/lekiwi_base.stl
- link imu_link: geometry collision mesh filename=../../meshes/bno055_imu.stl; visual mesh filename=../../meshes/bno055_imu.stl
- link laser_link: geometry collision mesh filename=../../meshes/ld06_lidar.stl; visual mesh filename=../../meshes/ld06_lidar.stl
- link left_wheel_link: geometry collision mesh filename=../../meshes/omni_wheel.stl scale=1.0 1.0 1.0; visual mesh filename=../../meshes/omni_wheel.stl scale=1.0 1.0 1.0
- link mic_link: geometry collision mesh filename=../../meshes/respeaker_flex_mic.stl; visual mesh filename=../../meshes/respeaker_flex_mic.stl
- link oak_link_model_origin: geometry visual mesh filename=https://raw.githubusercontent.com/adityakamath/pantilt_ros2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
- link pantilt_base_link: geometry collision mesh filename=https://raw.githubusercontent.com/adityakamath/pantilt_ros2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; visual mesh filename=https://raw.githubusercontent.com/adityakamath/pantilt_ros2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
- link right_wheel_link: geometry collision mesh filename=../../meshes/omni_wheel.stl scale=1.0 1.0 1.0; visual mesh filename=../../meshes/omni_wheel.stl scale=1.0 1.0 1.0
- link shoulder_link: geometry collision mesh filename=https://raw.githubusercontent.com/adityakamath/pantilt_ros2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; visual mesh filename=https://raw.githubusercontent.com/adityakamath/pantilt_ros2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
- link tilt_link: geometry collision mesh filename=https://raw.githubusercontent.com/adityakamath/pantilt_ros2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; visual mesh filename=https://raw.githubusercontent.com/adityakamath/pantilt_ros2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
