Commit message: expose xacro args as parameters, add to yaml config files

File: lekiwi_description/urdf/base/base.control.xacro (robot description, xacro)
@@ -14,14 +14,16 @@
   <xacro:arg name="imu_axis_remap" default="P1"/>      <!-- Mounting orientation P0-P7, see BNO055 datasheet Table 3-4 -->
   <xacro:arg name="imu_sensor_mode" default="NDOF"/>   <!-- Fusion mode: NDOF, NDOF_FMC_OFF, IMUPLUS -->
+  <!-- Configurable hardware parameters (STS3215 defaults) -->
+  <xacro:arg name="sts_max_velocity_steps" default="3400"/>  <!-- STS3215=3400, STS3032=2900, STS3235=3400 -->
+  <xacro:arg name="proportional_acc_max"   default="25"/>    <!-- [0-254]; 0 = disable proportional ACC -->
   <!-- Base operating mode -->
   <xacro:property name="base_operating_mode" value="1"/>  <!-- Velocity mode -->
-  <!-- Motor-specific parameter (STS3215 default) -->
-  <!-- Adjust for other motor models: STS3032 max=2900, STS3235 max=3400 -->
-  <xacro:property name="sts_max_velocity_steps" value="3400"/>  <!-- Max hardware velocity in steps/s (absolute motor limit, do not exceed) -->
+  <!-- Motor-specific parameter — sourced from arg, STS3215 default -->
+  <xacro:property name="sts_max_velocity_steps" value="$(arg sts_max_velocity_steps)"/>  <!-- Max hardware velocity in steps/s -->
   <!-- Proportional ACC parameters (SyncWriteSpe velocity path only) -->
   <!-- ACC given to the wheel with the largest |target - current| velocity delta. -->
   <!-- All others scaled proportionally so every wheel finishes ramping in equal time. -->
   <!-- Set proportional_acc_max to 0 to disable (ACC=0 for all wheels). -->
-  <xacro:property name="proportional_acc_max" value="25"/>        <!-- [0-254] -->
+  <xacro:property name="proportional_acc_max" value="$(arg proportional_acc_max)"/>        <!-- [0-254] -->
   <!-- Wheel geometry for omnidirectional control -->
   <xacro:property name="wheel_radius" value="0.051"/>  <!-- meters -->

File: lekiwi_description/urdf/k2.control.xacro (robot description, xacro)
@@ -18,14 +18,22 @@
   <xacro:arg name="imu_axis_remap"  default="P1"/>      <!-- Mounting orientation P0-P7, see BNO055 datasheet Table 3-4 -->
   <xacro:arg name="imu_sensor_mode" default="NDOF"/>    <!-- Fusion mode: NDOF, NDOF_FMC_OFF, IMUPLUS -->
+  <!-- Configurable hardware parameters (STS3215 defaults) -->
+  <xacro:arg name="sts_max_velocity_steps" default="3400"/>  <!-- STS3215=3400, STS3032=2900, STS3235=3400 -->
+  <xacro:arg name="proportional_acc_max"   default="25"/>    <!-- [0-254]; 0 = disable proportional ACC -->
+  <xacro:arg name="proportional_vel_max"   default="0"/>     <!-- [0-max_velocity_steps]; 0 = each joint uses commanded velocity -->
+  <!-- Pan and Tilt joint limits (configurable, symmetric ±π/2 defaults) -->
+  <xacro:arg name="pan_joint_lower"        default="-1.5708"/>  <!-- rad, default -π/2 -->
+  <xacro:arg name="pan_joint_upper"        default="1.5708"/>   <!-- rad, default +π/2 -->
+  <xacro:arg name="tilt_joint_lower"       default="-1.5708"/>  <!-- rad, default -π/2 -->
+  <xacro:arg name="tilt_joint_upper"       default="1.5708"/>   <!-- rad, default +π/2 -->
   <!-- Base operating mode -->
   <xacro:property name="base_operating_mode" value="1"/>  <!-- Velocity mode -->
-  <!-- Motor-specific parameter (STS3215 default) -->
-  <!-- Adjust for other motor models: STS3032 max=2900, STS3235 max=3400 -->
-  <xacro:property name="sts_max_velocity_steps" value="3400"/>  <!-- Max hardware velocity in steps/s (absolute motor limit, do not exceed) -->
+  <!-- Motor-specific parameter — sourced from arg, STS3215 default -->
+  <xacro:property name="sts_max_velocity_steps" value="$(arg sts_max_velocity_steps)"/>  <!-- Max hardware velocity in steps/s -->
   <!-- Proportional ACC parameters (SyncWriteSpe velocity path only) -->
   <!-- ACC given to the wheel with the largest |target - current| velocity delta. -->
   <!-- All others scaled proportionally so every wheel finishes ramping in equal time. -->
   <!-- Set proportional_acc_max to 0 to disable (ACC=0 for all wheels). -->
-  <xacro:property name="proportional_acc_max" value="25"/>        <!-- [0-254] -->
+  <xacro:property name="proportional_acc_max" value="$(arg proportional_acc_max)"/>        <!-- [0-254] -->
   <!-- Wheel geometry for omnidirectional control -->
   <xacro:property name="wheel_radius" value="0.051"/>  <!-- meters -->
@@ -42,9 +50,9 @@
   <xacro:property name="max_linear_velocity_y" value="${wheel_radius * max_velocity_rads / 1.0}"/>
   <xacro:property name="max_angular_velocity_z" value="${wheel_radius * max_velocity_rads / wheel_base_radius}"/>
-  <!-- Pan and tilt joint limits -->
-  <xacro:property name="pan_joint_lower"  value="${-pi/2}"/>
-  <xacro:property name="pan_joint_upper"  value="${pi/2}"/>
-  <xacro:property name="tilt_joint_lower" value="${-pi/2}"/>
-  <xacro:property name="tilt_joint_upper" value="${pi/2}"/>
+  <!-- Pan and tilt joint limits — properties sourced from args for use in pantilt.module.xacro -->
+  <xacro:property name="pan_joint_lower"  value="$(arg pan_joint_lower)"/>
+  <xacro:property name="pan_joint_upper"  value="$(arg pan_joint_upper)"/>
+  <xacro:property name="tilt_joint_lower" value="$(arg tilt_joint_lower)"/>
+  <xacro:property name="tilt_joint_upper" value="$(arg tilt_joint_upper)"/>
   <!-- ROS 2 CONTROL -->
   <!-- System interface — all STS3215 joints on a single serial bus -->
@@ -61,4 +69,6 @@
       <!-- Proportional ACC: scale per-wheel acceleration so all wheels finish ramping in equal time -->
       <param name="proportional_acc_max">${proportional_acc_max}</param>
+      <!-- Proportional VEL: scale per-joint speed so all position joints arrive simultaneously -->
+      <param name="proportional_vel_max">$(arg proportional_vel_max)</param>
     </hardware>
     <!-- Left wheel joint (Motor ID 7) -->

File: lekiwi_description/urdf/pantilt/pantilt.control.xacro (robot description, xacro)
@@ -10,15 +10,23 @@
   <xacro:arg name="pan_center_steps"  default="2048"/>
   <xacro:arg name="tilt_center_steps" default="2048"/>
+  <!-- Configurable hardware parameters (STS3215 defaults) -->
+  <xacro:arg name="sts_max_velocity_steps" default="3400"/>  <!-- STS3215=3400, STS3032=2900, STS3235=3400 -->
+  <xacro:arg name="proportional_vel_max"   default="0"/>     <!-- [0-max_velocity_steps]; 0 = each joint uses commanded velocity -->
+  <!-- Pan and Tilt joint limits (configurable, symmetric ±π/2 defaults) -->
+  <xacro:arg name="pan_joint_lower"        default="-1.5708"/>  <!-- rad, default -π/2 -->
+  <xacro:arg name="pan_joint_upper"        default="1.5708"/>   <!-- rad, default +π/2 -->
+  <xacro:arg name="tilt_joint_lower"       default="-1.5708"/>  <!-- rad, default -π/2 -->
+  <xacro:arg name="tilt_joint_upper"       default="1.5708"/>   <!-- rad, default +π/2 -->
   <!-- Motor-specific parameter (STS3215 default) -->
   <xacro:property name="pantilt_operating_mode" default="0"/>  <!-- Position mode -->
-  <xacro:property name="sts_max_velocity_steps" value="3400"/>  <!-- Max hardware velocity in steps/s (absolute motor limit, do not exceed) -->
+  <xacro:property name="sts_max_velocity_steps" value="$(arg sts_max_velocity_steps)"/>  <!-- Max hardware velocity in steps/s -->
   <xacro:property name="max_velocity_steps" value="${int(sts_max_velocity_steps * 0.85)}"/> <!-- steps/second (85% of hardware max, 15% safety margin) -->
   <xacro:property name="max_velocity_rads" value="${max_velocity_steps*2*pi/4096}"/> <!-- rad/s -->
   <xacro:property name="max_torque_nm" value="2.942"/>  <!-- N⋅m (30 kgf⋅cm for STS3215) -->
-  <!-- Pan and Tilt joint limits -->
-  <xacro:property name="pan_joint_lower" value="${-pi/2}"/>
-  <xacro:property name="pan_joint_upper" value="${pi/2}"/>
-  <xacro:property name="tilt_joint_lower" value="${-pi/2}"/>
-  <xacro:property name="tilt_joint_upper" value="${pi/2}"/>
+  <!-- Pan and Tilt joint limits — properties sourced from args for use in module.xacro -->
+  <xacro:property name="pan_joint_lower"  value="$(arg pan_joint_lower)"/>
+  <xacro:property name="pan_joint_upper"  value="$(arg pan_joint_upper)"/>
+  <xacro:property name="tilt_joint_lower" value="$(arg tilt_joint_lower)"/>
+  <xacro:property name="tilt_joint_upper" value="$(arg tilt_joint_upper)"/>
   <!-- ROS 2 CONTROL -->
   <ros2_control name="pantilt_control" type="system">
@@ -31,4 +39,5 @@
       <param name="enable_mock_mode">$(arg use_mock)</param>
       <param name="max_velocity_steps">${sts_max_velocity_steps}</param>
+      <param name="proportional_vel_max">$(arg proportional_vel_max)</param>
       <param name="reset_states_on_activate">true</param>
     </hardware>
