Commit message: Add Gazebo simulation: base drive, LiDAR, IMU, and pantilt payload
sim:=true on lekiwi.launch.py runs the whole real control/nav stack (control.launch.py,
navigation.launch.py, teleop, twist_switch_node, collision_monitor) against Gazebo
instead of real hardware - only the ros2_control hardware layer differs
(ros2_control_hardware_type: real -> gz_ros2_control/GazeboSimSystem), everything above
it is unchanged code.

- base.control.xacro/base.urdf.xacro, base_pantilt equivalents: hardware plugin swap,
  drop STS-only telemetry interfaces GazeboSimSystem can't back, <gazebo> plugin block
  spawning controller_manager embedded in gz_sim (two <parameters> tags for
  base+payload in the pantilt case - gz_ros2_control supports multiple, same as the
  real standalone ros2_control_node already merges those two yaml files).
- base.module.xacro: native Gazebo LD19 lidar and BNO055 IMU sensors, values measured
  directly off the real robot (update rate, angular resolution, noise stddevs from
  imu_sensor_broadcaster's covariances) rather than guessed. gz_frame_id overrides
  gz-sim's default scoped sensor frame_id so TF resolves the same as on hardware.
  IMU publishes directly onto imu_sensor_broadcaster's own topic name so EKF needs no
  reconfiguration between sim and real; imu_sensor_broadcaster itself isn't spawned in
  gazebo mode to avoid a duplicate publisher.
- worlds/empty.sdf: gz-sim's bundled empty world doesn't load the Sensors system
  plugin, so <sensor> elements never produce data - own copy with it added.
- control.launch.py: skips its own controller_manager in gazebo mode (gz_sim's
  embedded one takes over); payload no longer forces hardware_type back to "real".
- lekiwi.launch.py: also fixes a real crash - FindPackageShare('lekiwi_audio') ran
  unconditionally regardless of sim mode, so any fresh clone without lekiwi_audio
  (not committed to this repo) would crash on launch. Now resolved lazily with a
  graceful skip if the package isn't present.
- payloads/pantilt100 bumped to f03b95d (same gz_ros2_control support, upstream).

Verified via full xacro re-renders (real-mode output confirmed byte-identical) and a
mocked launch_setup() run with lekiwi_audio's install hidden, matching a real fresh
clone. Gazebo itself hasn't been run end-to-end yet - this machine's GPU driver
doesn't support the rendering pipeline gz-sim needs.

Co-Authored-By: Claude Sonnet 5 <noreply@anthropic.com>

File: lekiwi_description/urdf/base/base.control.xacro (robot description, xacro)
@@ -9,4 +9,13 @@
   <xacro:arg name="back_motor_id" default="8"/>
   <xacro:arg name="right_motor_id" default="9"/>
+  <!-- Gazebo simulation -->
+  <!-- "real" (default) keeps the STS3215 serial hardware plugin below unchanged.
+       "gazebo" swaps the base's <hardware> plugin for gz_ros2_control/GazeboSimSystem,
+       which implements the same SystemInterface contract - the joints, controllers,
+       and control.yaml stay identical either way. -->
+  <xacro:arg name="ros2_control_hardware_type" default="real"/>
+  <!-- Path to the controllers YAML the embedded controller_manager should load; only
+       used when the <gazebo> plugin below is actually instantiated (i.e. in sim). -->
+  <xacro:arg name="simulation_controllers" default=""/>
   <!-- BNO055 IMU parameters (externally settable) -->
   <xacro:arg name="imu_i2c_bus"    default="1"/>       <!-- I2C bus number (/dev/i2c-1) -->
@@ -44,14 +53,19 @@
   <ros2_control name="lekiwi_base" type="system">
     <hardware>
-      <plugin>sts_hardware_interface/STSHardwareInterface</plugin>
-      <!-- Serial communication parameters -->
-      <param name="serial_port">$(arg serial_port)</param>
-      <param name="baud_rate">$(arg baud_rate)</param>
-      <param name="use_sync_write">$(arg use_sync_write)</param>
-      <param name="enable_mock_mode">$(arg use_mock)</param>
-      <!-- Motor-specific parameter (adjust for different STS motor models) -->
-      <param name="max_velocity_steps">${sts_max_velocity_steps}</param>
-      <!-- Proportional ACC: scale per-wheel acceleration so all wheels finish ramping in equal time -->
-      <param name="proportional_acc_max">${proportional_acc_max}</param>
+      <xacro:if value="${'$(arg ros2_control_hardware_type)' == 'gazebo'}">
+        <plugin>gz_ros2_control/GazeboSimSystem</plugin>
+      </xacro:if>
+      <xacro:unless value="${'$(arg ros2_control_hardware_type)' == 'gazebo'}">
+        <plugin>sts_hardware_interface/STSHardwareInterface</plugin>
+        <!-- Serial communication parameters -->
+        <param name="serial_port">$(arg serial_port)</param>
+        <param name="baud_rate">$(arg baud_rate)</param>
+        <param name="use_sync_write">$(arg use_sync_write)</param>
+        <param name="enable_mock_mode">$(arg use_mock)</param>
+        <!-- Motor-specific parameter (adjust for different STS motor models) -->
+        <param name="max_velocity_steps">${sts_max_velocity_steps}</param>
+        <!-- Proportional ACC: scale per-wheel acceleration so all wheels finish ramping in equal time -->
+        <param name="proportional_acc_max">${proportional_acc_max}</param>
+      </xacro:unless>
     </hardware>
     <!-- Left wheel joint (Motor ID 7) -->
@@ -63,8 +77,12 @@
       <state_interface name="velocity"/>
       <state_interface name="effort"/>
-      <state_interface name="voltage"/>
-      <state_interface name="temperature"/>
-      <state_interface name="current"/>
-      <state_interface name="is_moving"/>
+      <!-- Real-hardware-only telemetry: gz_ros2_control/GazeboSimSystem only knows
+           position/velocity/effort, and simulated wheels have no real telemetry for these. -->
+      <xacro:unless value="${'$(arg ros2_control_hardware_type)' == 'gazebo'}">
+        <state_interface name="voltage"/>
+        <state_interface name="temperature"/>
+        <state_interface name="current"/>
+        <state_interface name="is_moving"/>
+      </xacro:unless>
     </joint>
     <!-- Back wheel joint (Motor ID 8) -->
@@ -76,8 +94,12 @@
       <state_interface name="velocity"/>
       <state_interface name="effort"/>
-      <state_interface name="voltage"/>
-      <state_interface name="temperature"/>
-      <state_interface name="current"/>
-      <state_interface name="is_moving"/>
+      <!-- Real-hardware-only telemetry: gz_ros2_control/GazeboSimSystem only knows
+           position/velocity/effort, and simulated wheels have no real telemetry for these. -->
+      <xacro:unless value="${'$(arg ros2_control_hardware_type)' == 'gazebo'}">
+        <state_interface name="voltage"/>
+        <state_interface name="temperature"/>
+        <state_interface name="current"/>
+        <state_interface name="is_moving"/>
+      </xacro:unless>
     </joint>
     <!-- Right wheel joint (Motor ID 9) -->
@@ -89,36 +111,46 @@
       <state_interface name="velocity"/>
       <state_interface name="effort"/>
-      <state_interface name="voltage"/>
-      <state_interface name="temperature"/>
-      <state_interface name="current"/>
-      <state_interface name="is_moving"/>
+      <!-- Real-hardware-only telemetry: gz_ros2_control/GazeboSimSystem only knows
+           position/velocity/effort, and simulated wheels have no real telemetry for these. -->
+      <xacro:unless value="${'$(arg ros2_control_hardware_type)' == 'gazebo'}">
+        <state_interface name="voltage"/>
+        <state_interface name="temperature"/>
+        <state_interface name="current"/>
+        <state_interface name="is_moving"/>
+      </xacro:unless>
     </joint>
   </ros2_control>
   <!-- ROS 2 CONTROL -->
-  <!-- Sensor interface (BNO055 IMU) -->
-  <ros2_control name="lekiwi_imu" type="sensor">
-    <hardware>
-      <plugin>bno055_hardware_interface/BNO055HardwareInterface</plugin>
-      <param name="i2c_bus">$(arg imu_i2c_bus)</param>       <!-- I2C bus number (default: 1 → /dev/i2c-1) -->
-      <param name="i2c_addr">$(arg imu_i2c_addr)</param>     <!-- I2C address in hex, no 0x prefix (default: 28 = 0x28) -->
-      <param name="axis_remap">$(arg imu_axis_remap)</param> <!-- Axis placement config: P0-P7 (default: P1) -->
-      <param name="sensor_mode">$(arg imu_sensor_mode)</param> <!-- Fusion mode: NDOF, NDOF_FMC_OFF, IMUPLUS (default: NDOF) -->
-      <param name="enable_mock_mode">$(arg use_mock)</param>  <!-- Reuse the system-level mock flag -->
-    </hardware>
-    <sensor name="bno055">
-      <!-- Orientation (quaternion, unit norm) -->
-      <state_interface name="orientation.x"/>
-      <state_interface name="orientation.y"/>
-      <state_interface name="orientation.z"/>
-      <state_interface name="orientation.w"/>
-      <!-- Angular velocity (rad/s) -->
-      <state_interface name="angular_velocity.x"/>
-      <state_interface name="angular_velocity.y"/>
-      <state_interface name="angular_velocity.z"/>
-      <!-- Linear acceleration (m/s²), gravity-compensated -->
-      <state_interface name="linear_acceleration.x"/>
-      <state_interface name="linear_acceleration.y"/>
-      <state_interface name="linear_acceleration.z"/>
-    </sensor>
-  </ros2_control>
+  <!-- Sensor interface (BNO055 IMU). Omitted entirely in gazebo mode: base.module.xacro's
+       native Gazebo IMU sensor + ros_gz_bridge supplies /imu_sensor_broadcaster/imu
+       directly instead (see the comment there), so there's nothing for this mock
+       hardware component to usefully do in sim - and imu_sensor_broadcaster itself isn't
+       spawned in gazebo mode either (control.launch.py), so it would go unclaimed anyway. -->
+  <xacro:unless value="${'$(arg ros2_control_hardware_type)' == 'gazebo'}">
+    <ros2_control name="lekiwi_imu" type="sensor">
+      <hardware>
+        <plugin>bno055_hardware_interface/BNO055HardwareInterface</plugin>
+        <param name="i2c_bus">$(arg imu_i2c_bus)</param>       <!-- I2C bus number (default: 1 → /dev/i2c-1) -->
+        <param name="i2c_addr">$(arg imu_i2c_addr)</param>     <!-- I2C address in hex, no 0x prefix (default: 28 = 0x28) -->
+        <param name="axis_remap">$(arg imu_axis_remap)</param> <!-- Axis placement config: P0-P7 (default: P1) -->
+        <param name="sensor_mode">$(arg imu_sensor_mode)</param> <!-- Fusion mode: NDOF, NDOF_FMC_OFF, IMUPLUS (default: NDOF) -->
+        <param name="enable_mock_mode">$(arg use_mock)</param>  <!-- Reuse the system-level mock flag -->
+      </hardware>
+      <sensor name="bno055">
+        <!-- Orientation (quaternion, unit norm) -->
+        <state_interface name="orientation.x"/>
+        <state_interface name="orientation.y"/>
+        <state_interface name="orientation.z"/>
+        <state_interface name="orientation.w"/>
+        <!-- Angular velocity (rad/s) -->
+        <state_interface name="angular_velocity.x"/>
+        <state_interface name="angular_velocity.y"/>
+        <state_interface name="angular_velocity.z"/>
+        <!-- Linear acceleration (m/s²), gravity-compensated -->
+        <state_interface name="linear_acceleration.x"/>
+        <state_interface name="linear_acceleration.y"/>
+        <state_interface name="linear_acceleration.z"/>
+      </sensor>
+    </ros2_control>
+  </xacro:unless>
 </robot>

File: lekiwi_description/urdf/base/base.module.xacro (robot description, xacro)
@@ -58,4 +58,49 @@
     <!-- Laser frame -->
     <link name="laser_frame"/>
+    <!-- Gazebo simulation: LD19 lidar, values measured directly off the real robot
+         (ros2 launch lekiwi_bringup laser.launch.py, then `ros2 topic hz /scan` and
+         echoing individual messages) rather than the datasheet:
+           - update_rate=10: measured /scan rate was a steady 10.00-10.01 Hz.
+           - samples=452: angle_increment measured ~0.0139 rad/point average across
+             several messages; 2*pi/0.0139 ~= 452. (The real driver actually publishes
+             partial ~129-point slices per message rather than one full 452-point sweep -
+             that's a chunking quirk of ldlidar_ros2_node's publishing, not something
+             SLAM/Nav2 depend on, so it's not replicated here; a clean full sweep at the
+             same angular resolution is the right target.)
+           - min_angle/max_angle=0..2pi and range 0.02-12m: read directly off the real
+             /scan message fields (angle_min/angle_max/range_min/range_max).
+         gz_frame_id overrides gz-sim's default scoped sensor frame_id
+         (e.g. lekiwi/laser_frame/lidar) to the plain "laser_frame" the real
+         ldlidar_ros2_node publishes (lekiwi_bringup/config/laser.yaml), so TF lookups
+         resolve the same way in sim as on hardware - unofficial SDF tag (emits a
+         "not defined in SDF" warning) but functional: gazebosim/gz-sensors#306.
+         nav2/slam_toolbox's own range caps (obstacle_max_range: 5.5, max_laser_range:
+         8.0) are intentionally below this sensor's 12m max, same as with the real LD19.
+         Inert outside Gazebo, like the <gazebo> control plugin in base.urdf.xacro. -->
+    <gazebo reference="laser_frame">
+      <sensor name="lidar" type="gpu_lidar">
+        <pose>0 0 0 0 0 0</pose>
+        <topic>scan</topic>
+        <gz_frame_id>laser_frame</gz_frame_id>
+        <update_rate>10</update_rate>
+        <always_on>true</always_on>
+        <visualize>false</visualize>
+        <lidar>
+          <scan>
+            <horizontal>
+              <samples>452</samples>
+              <resolution>1</resolution>
+              <min_angle>0.0</min_angle>
+              <max_angle>6.283185307179586</max_angle>
+            </horizontal>
+          </scan>
+          <range>
+            <min>0.02</min>
+            <max>12.0</max>
+            <resolution>0.01</resolution>
+          </range>
+        </lidar>
+      </sensor>
+    </gazebo>
     <!-- BNO055 IMU link -->
     <link name="imu_link">
@@ -80,4 +125,42 @@
     <!-- IMU frame -->
     <link name="imu_frame"/>
+    <!-- Gazebo simulation: BNO055 IMU. Matches imu_sensor_broadcaster's frame_id
+         (lekiwi_control/config/base/control.yaml: frame_id=imu_frame) by attaching
+         directly to the imu_frame link, and topic is set to the exact topic name
+         imu_sensor_broadcaster would publish on (/imu_sensor_broadcaster/imu) so EKF
+         (lekiwi_navigation/config/robot_localization/ekf*.yaml: imu0) needs no
+         reconfiguration between real and sim. Because of this, imu_sensor_broadcaster
+         itself is NOT spawned in gazebo mode (control.launch.py) - it would otherwise
+         publish the mock bno055_hardware_interface's fake static data onto the same
+         topic, racing with this bridged one. update_rate=50 matches controller_manager's
+         update_rate (lekiwi_control/config/base/control.yaml) - the effective rate
+         imu_sensor_broadcaster publishes at on real hardware regardless of the BNO055's
+         own internal fusion rate. angular_velocity/linear_acceleration noise stddev
+         values are sqrt() of imu_sensor_broadcaster's static_covariance_* parameters
+         (same yaml file) - gz's IMU sensor has no equivalent independent orientation
+         noise parameter, so orientation comes out physics-consistent/noise-free instead.
+         gz_frame_id and inertness outside Gazebo: see the lidar sensor above. -->
+    <gazebo reference="imu_frame">
+      <sensor name="imu" type="imu">
+        <pose>0 0 0 0 0 0</pose>
+        <topic>imu_sensor_broadcaster/imu</topic>
+        <gz_frame_id>imu_frame</gz_frame_id>
+        <update_rate>50</update_rate>
+        <always_on>true</always_on>
+        <visualize>false</visualize>
+        <imu>
+          <angular_velocity>
+            <x><noise type="gaussian"><mean>0.0</mean><stddev>0.00316</stddev></noise></x>
+            <y><noise type="gaussian"><mean>0.0</mean><stddev>0.00316</stddev></noise></y>
+            <z><noise type="gaussian"><mean>0.0</mean><stddev>0.00316</stddev></noise></z>
+          </angular_velocity>
+          <linear_acceleration>
+            <x><noise type="gaussian"><mean>0.0</mean><stddev>0.01414</stddev></noise></x>
+            <y><noise type="gaussian"><mean>0.0</mean><stddev>0.01414</stddev></noise></y>
+            <z><noise type="gaussian"><mean>0.0</mean><stddev>0.01414</stddev></noise></z>
+          </linear_acceleration>
+        </imu>
+      </sensor>
+    </gazebo>
     <!-- Respeaker flex mic link -->
     <link name="mic_link">

File: lekiwi_description/urdf/base/base.urdf.xacro (robot description, xacro)
@@ -9,3 +9,11 @@
     <origin xyz="0 0 ${wheel_radius - wheel_base_offset_z}" rpy="0 0 0"/>
   </xacro:lekiwi_base_module>
+  <!-- Gazebo simulation: spawns controller_manager inside the gz_sim process, loading
+       $(arg simulation_controllers). Inert (ignored) outside Gazebo, so this is safe to
+       leave in place regardless of ros2_control_hardware_type. -->
+  <gazebo>
+    <plugin filename="gz_ros2_control-system" name="gz_ros2_control::GazeboSimROS2ControlPlugin">
+      <parameters>$(arg simulation_controllers)</parameters>
+    </plugin>
+  </gazebo>
 </robot>
