Commit message: Add MuJoCo simulation, lekiwi_audio, and repo restructuring
MuJoCo simulation support (replacing the never-launch-wired Gazebo
path): parametric MJCF templates under lekiwi_description/mjcf/,
mirroring the URDF side's one-file-per-payload structure, xacro-
processed at launch time by control.launch.py. Wired into both
base.control.xacro and base_pantilt.control.xacro via
ros2_control_hardware_type:="mujoco", exposing IMU/lidar through
mujoco_ros2_control's built-in sensor registration. Gazebo support
remains at the xacro level only, not wired into any launch file.

Repo restructuring: renamed the pantilt100 submodule to pantilt_ros2
(matching its GitHub rename), and vendored sts_hardware_interface,
bno055_hardware_interface, and ldlidar_ros2 as git submodules under
a new modules/ directory instead of requiring them to be cloned
separately alongside this workspace.

Added lekiwi_audio: spoken status announcements for e-stop, mode
switching, and waypoint actions, watching service introspection so
announcements fire regardless of what triggered the call. Kokoro TTS
model files aren't committed (116 MB) - render_phrases.py downloads
them from the upstream GitHub release on demand, only when a phrase
actually needs (re-)rendering; the common case ships pre-rendered
sounds/*.wav and never touches them.

Also: removed the now-orphaned Gazebo world file and its CMakeLists
entry; fixed several stale/incorrect comments found while auditing
(wrong launch-arg descriptions, a dangling reference to a renamed
launch arg, hardware-plugin-wiring claims that predated this same
change); trimmed comments across the MuJoCo/xacro files and the
README that had grown into implementation narratives rather than the
facts needed to use or modify the code; reworked the README into a
proper project guide (Packages/Dependencies, concise launch args and
controls) instead of a design document.

Co-Authored-By: Claude Sonnet 5 <noreply@anthropic.com>

File: lekiwi_description/urdf/base/base.control.xacro (robot description, xacro)
@@ -9,13 +9,18 @@
   <xacro:arg name="back_motor_id" default="8"/>
   <xacro:arg name="right_motor_id" default="9"/>
-  <!-- Gazebo simulation -->
-  <!-- "real" (default) keeps the STS3215 serial hardware plugin below unchanged.
-       "gazebo" swaps the base's <hardware> plugin for gz_ros2_control/GazeboSimSystem,
-       which implements the same SystemInterface contract - the joints, controllers,
-       and control.yaml stay identical either way. -->
+  <!-- Simulation -->
+  <!-- "real" (default) keeps the STS3215 serial hardware plugin below unchanged. "mujoco"
+       swaps it for mujoco_ros2_control/MujocoSystemInterface, which also natively hosts the
+       IMU and lidar sensors below (mujoco_type="imu"/the laser_frame <sensor> block) - wired
+       into control.launch.py. "gazebo" swaps it for gz_ros2_control/GazeboSimSystem; the
+       joints/controllers/control.yaml stay identical, but this option exists at the
+       xacro level only, not wired into any launch file yet. -->
   <xacro:arg name="ros2_control_hardware_type" default="real"/>
   <!-- Path to the controllers YAML the embedded controller_manager should load; only
        used when the <gazebo> plugin below is actually instantiated (i.e. in sim). -->
   <xacro:arg name="simulation_controllers" default=""/>
+  <!-- MJCF scene path and headless flag; only used when ros2_control_hardware_type:="mujoco". -->
+  <xacro:arg name="mujoco_model" default=""/>
+  <xacro:arg name="mujoco_headless" default="false"/>
   <!-- BNO055 IMU parameters (externally settable) -->
   <xacro:arg name="imu_i2c_bus"    default="1"/>       <!-- I2C bus number (/dev/i2c-1) -->
@@ -56,5 +61,10 @@
         <plugin>gz_ros2_control/GazeboSimSystem</plugin>
       </xacro:if>
-      <xacro:unless value="${'$(arg ros2_control_hardware_type)' == 'gazebo'}">
+      <xacro:if value="${'$(arg ros2_control_hardware_type)' == 'mujoco'}">
+        <plugin>mujoco_ros2_control/MujocoSystemInterface</plugin>
+        <param name="mujoco_model">$(arg mujoco_model)</param>
+        <param name="headless">$(arg mujoco_headless)</param>
+      </xacro:if>
+      <xacro:if value="${'$(arg ros2_control_hardware_type)' == 'real'}">
         <plugin>sts_hardware_interface/STSHardwareInterface</plugin>
         <!-- Serial communication parameters -->
@@ -67,5 +77,5 @@
         <!-- Proportional ACC: scale per-wheel acceleration so all wheels finish ramping in equal time -->
         <param name="proportional_acc_max">${proportional_acc_max}</param>
-      </xacro:unless>
+      </xacro:if>
     </hardware>
     <!-- Left wheel joint (Motor ID 7) -->
@@ -77,12 +87,13 @@
       <state_interface name="velocity"/>
       <state_interface name="effort"/>
-      <!-- Real-hardware-only telemetry: gz_ros2_control/GazeboSimSystem only knows
+      <!-- Real-hardware-only telemetry: neither gz_ros2_control/GazeboSimSystem nor
+           mujoco_ros2_control/MujocoSystemInterface know anything beyond
            position/velocity/effort, and simulated wheels have no real telemetry for these. -->
-      <xacro:unless value="${'$(arg ros2_control_hardware_type)' == 'gazebo'}">
+      <xacro:if value="${'$(arg ros2_control_hardware_type)' == 'real'}">
         <state_interface name="voltage"/>
         <state_interface name="temperature"/>
         <state_interface name="current"/>
         <state_interface name="is_moving"/>
-      </xacro:unless>
+      </xacro:if>
     </joint>
     <!-- Back wheel joint (Motor ID 8) -->
@@ -94,12 +105,13 @@
       <state_interface name="velocity"/>
       <state_interface name="effort"/>
-      <!-- Real-hardware-only telemetry: gz_ros2_control/GazeboSimSystem only knows
+      <!-- Real-hardware-only telemetry: neither gz_ros2_control/GazeboSimSystem nor
+           mujoco_ros2_control/MujocoSystemInterface know anything beyond
            position/velocity/effort, and simulated wheels have no real telemetry for these. -->
-      <xacro:unless value="${'$(arg ros2_control_hardware_type)' == 'gazebo'}">
+      <xacro:if value="${'$(arg ros2_control_hardware_type)' == 'real'}">
         <state_interface name="voltage"/>
         <state_interface name="temperature"/>
         <state_interface name="current"/>
         <state_interface name="is_moving"/>
-      </xacro:unless>
+      </xacro:if>
     </joint>
     <!-- Right wheel joint (Motor ID 9) -->
@@ -111,21 +123,69 @@
       <state_interface name="velocity"/>
       <state_interface name="effort"/>
-      <!-- Real-hardware-only telemetry: gz_ros2_control/GazeboSimSystem only knows
+      <!-- Real-hardware-only telemetry: neither gz_ros2_control/GazeboSimSystem nor
+           mujoco_ros2_control/MujocoSystemInterface know anything beyond
            position/velocity/effort, and simulated wheels have no real telemetry for these. -->
-      <xacro:unless value="${'$(arg ros2_control_hardware_type)' == 'gazebo'}">
+      <xacro:if value="${'$(arg ros2_control_hardware_type)' == 'real'}">
         <state_interface name="voltage"/>
         <state_interface name="temperature"/>
         <state_interface name="current"/>
         <state_interface name="is_moving"/>
-      </xacro:unless>
+      </xacro:if>
     </joint>
+    <!-- mujoco_ros2_control's IMU/lidar sensors must live inside the SAME <ros2_control>
+         block as the MujocoSystemInterface <hardware><plugin> above - each ros2_control
+         block is a separate hardware-plugin instance with its own isolated HardwareInfo,
+         so a sensor declared in a different block (like lekiwi_imu below) would never be
+         seen by this one. These map to lekiwi_description/mjcf/base_subtree.xml's MJCF
+         sensors. -->
+    <xacro:if value="${'$(arg ros2_control_hardware_type)' == 'mujoco'}">
+      <!-- BNO055 IMU - mujoco_type="imu" tells MujocoSystemInterface::register_sensors to
+           look for MJCF sensors named bno055_quat/bno055_gyro/bno055_accel (the fixed
+           _quat/_gyro/_accel suffix convention), attached to base_subtree.xml's imu_site. Same
+           state_interface list as the real-hardware lekiwi_imu block below - duplicated,
+           not shared via a macro, to keep both branches readable independently. -->
+      <sensor name="bno055">
+        <param name="mujoco_type">imu</param>
+        <state_interface name="orientation.x"/>
+        <state_interface name="orientation.y"/>
+        <state_interface name="orientation.z"/>
+        <state_interface name="orientation.w"/>
+        <state_interface name="angular_velocity.x"/>
+        <state_interface name="angular_velocity.y"/>
+        <state_interface name="angular_velocity.z"/>
+        <state_interface name="linear_acceleration.x"/>
+        <state_interface name="linear_acceleration.y"/>
+        <state_interface name="linear_acceleration.z"/>
+      </sensor>
+      <!-- LD19 lidar - matched to base_subtree.xml's 360 "lidar-<i>" MJCF rangefinder sensors by
+           this <sensor> block's own name ("lidar" - matching the part of "lidar-<i>" before
+           the last hyphen, per mujoco_lidar.cpp's parse_lidar_name - NOT the frame_name
+           param below, easy to mix up), not by a mujoco_type param (the lidar registration
+           path is separate from register_sensors).
+           angle_increment/min_angle/max_angle intentionally don't match the real LD19's
+           452-sample resolution - see base_subtree.xml's lidar comment for why. laserscan_topic
+           matches the real ldlidar_ros2_node's /scan topic (lekiwi_bringup/config/laser.yaml)
+           so downstream consumers (SLAM, Nav2) don't need to know whether they're talking to
+           real or simulated lidar. -->
+      <sensor name="lidar">
+        <param name="frame_name">laser_frame</param>
+        <param name="min_angle">0.0</param>
+        <param name="max_angle">6.274458660919615</param>
+        <param name="angle_increment">0.017453292519943295</param>
+        <param name="range_min">0.02</param>
+        <param name="range_max">12.0</param>
+        <param name="laserscan_topic">/scan</param>
+      </sensor>
+    </xacro:if>
   </ros2_control>
   <!-- ROS 2 CONTROL -->
-  <!-- Sensor interface (BNO055 IMU). Omitted entirely in gazebo mode: base.module.xacro's
-       native Gazebo IMU sensor + ros_gz_bridge supplies /imu_sensor_broadcaster/imu
-       directly instead (see the comment there), so there's nothing for this mock
-       hardware component to usefully do in sim - and imu_sensor_broadcaster itself isn't
-       spawned in gazebo mode either (control.launch.py), so it would go unclaimed anyway. -->
-  <xacro:unless value="${'$(arg ros2_control_hardware_type)' == 'gazebo'}">
+  <!-- Sensor interface (BNO055 IMU) for real hardware. Omitted in gazebo mode:
+       base.module.xacro's native Gazebo IMU sensor + ros_gz_bridge supplies
+       /imu_sensor_broadcaster/imu directly instead (see the comment there). Omitted in
+       mujoco mode too: the equivalent sensor lives inside the lekiwi_base system block
+       above instead (mujoco_ros2_control requires it in the same <ros2_control> block as
+       the plugin declaration). imu_sensor_broadcaster itself isn't spawned in gazebo mode
+       either (control.launch.py), so a lekiwi_imu block would go unclaimed there anyway. -->
+  <xacro:if value="${'$(arg ros2_control_hardware_type)' == 'real'}">
     <ros2_control name="lekiwi_imu" type="sensor">
       <hardware>
@@ -153,4 +213,4 @@
       </sensor>
     </ros2_control>
-  </xacro:unless>
+  </xacro:if>
 </robot>

File: lekiwi_description/urdf/base/base.module.xacro (robot description, xacro)
@@ -58,24 +58,9 @@
     <!-- Laser frame -->
     <link name="laser_frame"/>
-    <!-- Gazebo simulation: LD19 lidar, values measured directly off the real robot
-         (ros2 launch lekiwi_bringup laser.launch.py, then `ros2 topic hz /scan` and
-         echoing individual messages) rather than the datasheet:
-           - update_rate=10: measured /scan rate was a steady 10.00-10.01 Hz.
-           - samples=452: angle_increment measured ~0.0139 rad/point average across
-             several messages; 2*pi/0.0139 ~= 452. (The real driver actually publishes
-             partial ~129-point slices per message rather than one full 452-point sweep -
-             that's a chunking quirk of ldlidar_ros2_node's publishing, not something
-             SLAM/Nav2 depend on, so it's not replicated here; a clean full sweep at the
-             same angular resolution is the right target.)
-           - min_angle/max_angle=0..2pi and range 0.02-12m: read directly off the real
-             /scan message fields (angle_min/angle_max/range_min/range_max).
-         gz_frame_id overrides gz-sim's default scoped sensor frame_id
-         (e.g. lekiwi/laser_frame/lidar) to the plain "laser_frame" the real
-         ldlidar_ros2_node publishes (lekiwi_bringup/config/laser.yaml), so TF lookups
-         resolve the same way in sim as on hardware - unofficial SDF tag (emits a
-         "not defined in SDF" warning) but functional: gazebosim/gz-sensors#306.
-         nav2/slam_toolbox's own range caps (obstacle_max_range: 5.5, max_laser_range:
-         8.0) are intentionally below this sensor's 12m max, same as with the real LD19.
-         Inert outside Gazebo, like the <gazebo> control plugin in base.urdf.xacro. -->
+    <!-- Gazebo simulation: LD19 lidar. update_rate/samples/angle/range values measured
+         directly off the real robot's /scan topic, not the datasheet. gz_frame_id overrides
+         gz-sim's default scoped sensor frame_id to the plain "laser_frame" the real
+         ldlidar_ros2_node publishes, so TF resolves the same in sim as on hardware
+         (unofficial SDF tag - gazebosim/gz-sensors#306). Inert outside Gazebo. -->
     <gazebo reference="laser_frame">
       <sensor name="lidar" type="gpu_lidar">
@@ -125,20 +110,11 @@
     <!-- IMU frame -->
     <link name="imu_frame"/>
-    <!-- Gazebo simulation: BNO055 IMU. Matches imu_sensor_broadcaster's frame_id
-         (lekiwi_control/config/base/control.yaml: frame_id=imu_frame) by attaching
-         directly to the imu_frame link, and topic is set to the exact topic name
-         imu_sensor_broadcaster would publish on (/imu_sensor_broadcaster/imu) so EKF
-         (lekiwi_navigation/config/robot_localization/ekf*.yaml: imu0) needs no
-         reconfiguration between real and sim. Because of this, imu_sensor_broadcaster
-         itself is NOT spawned in gazebo mode (control.launch.py) - it would otherwise
-         publish the mock bno055_hardware_interface's fake static data onto the same
-         topic, racing with this bridged one. update_rate=50 matches controller_manager's
-         update_rate (lekiwi_control/config/base/control.yaml) - the effective rate
-         imu_sensor_broadcaster publishes at on real hardware regardless of the BNO055's
-         own internal fusion rate. angular_velocity/linear_acceleration noise stddev
-         values are sqrt() of imu_sensor_broadcaster's static_covariance_* parameters
-         (same yaml file) - gz's IMU sensor has no equivalent independent orientation
-         noise parameter, so orientation comes out physics-consistent/noise-free instead.
-         gz_frame_id and inertness outside Gazebo: see the lidar sensor above. -->
+    <!-- Gazebo simulation: BNO055 IMU. Attached to imu_frame and published on
+         /imu_sensor_broadcaster/imu (imu_sensor_broadcaster's own topic/frame_id) so EKF
+         needs no reconfiguration between real and sim; imu_sensor_broadcaster itself isn't
+         spawned in gazebo mode to avoid racing with this bridged topic. update_rate=50
+         matches controller_manager's rate. Noise stddevs are sqrt() of
+         imu_sensor_broadcaster's static_covariance_* params (gz has no separate orientation
+         noise, so orientation comes out noise-free). gz_frame_id/inertness: see lidar above. -->
     <gazebo reference="imu_frame">
       <sensor name="imu" type="imu">
