Commit message: Add teleop.launch.py split, race-safety fixes, and comment/README cleanup
teleop.launch.py splits joystick-specific launch surface out of control.launch.py,
matching the so_arm_ros2 core/teleop launch pattern. nav2.launch.py/slam.launch.py
gain the same strict-bool launch-argument coercion control.launch.py already used,
fixing a real type-coercion bug on their use_sim_time/autostart/diagnostics args.

map_saver_node.py and waypoint_recorder_node.py each gain a generation/state guard
against a stale async callback racing a newer one. Bumps modules/ldlidar_ros2 to
pick up a fix for a real shutdown-time crash (FD_SETSIZE abort from closing a
serial fd out from under its still-running read thread), reproduced and verified
fixed on real hardware.

Comment blocks trimmed to house style across the touched files, and README
brought back in sync with the new imu/laser/audio/battery_monitor launch args
and the ina260_ros2 battery integration.

File: lekiwi_description/urdf/base/base.control.xacro (robot description, xacro)
@@ -10,10 +10,6 @@
   <xacro:arg name="right_motor_id" default="9"/>
   <!-- Simulation -->
-  <!-- "real" (default) keeps the STS3215 serial hardware plugin below unchanged. "mujoco"
-       swaps it for mujoco_ros2_control/MujocoSystemInterface, which also natively hosts the
-       IMU and lidar sensors below (mujoco_type="imu"/the laser_frame <sensor> block) - wired
-       into control.launch.py. "gazebo" swaps it for gz_ros2_control/GazeboSimSystem; the
-       joints/controllers/control.yaml stay identical, but this option exists at the
-       xacro level only, not wired into any launch file yet. -->
+  <!-- "real" (default): STS3215 serial plugin. "mujoco": MujocoSystemInterface (also hosts
+       IMU/lidar below), wired into control.launch.py. "gazebo": GazeboSimSystem, xacro-only. -->
   <xacro:arg name="ros2_control_hardware_type" default="real"/>
   <!-- Path to the controllers YAML the embedded controller_manager should load; only
@@ -24,4 +20,5 @@
   <xacro:arg name="mujoco_headless" default="false"/>
   <!-- BNO055 IMU parameters (externally settable) -->
+  <xacro:arg name="imu"             default="true"/>   <!-- false = no physical IMU; omits the lekiwi_imu sensor block below (real hardware only) -->
   <xacro:arg name="imu_i2c_bus"    default="1"/>       <!-- I2C bus number (/dev/i2c-1) -->
   <xacro:arg name="imu_i2c_addr"   default="28"/>      <!-- I2C address: 28 = 0x28 (ADR pin low) -->
@@ -29,10 +26,10 @@
   <xacro:arg name="imu_sensor_mode" default="NDOF"/>   <!-- Fusion mode: NDOF, NDOF_FMC_OFF, IMUPLUS -->
   <!-- Configurable hardware parameters (STS3215 defaults) -->
-  <xacro:arg name="sts_max_velocity_steps" default="3400"/>  <!-- STS3215=3400, STS3032=2900, STS3235=3400 -->
+  <xacro:arg name="sts3215_max_vel_steps" default="3400"/>  <!-- STS3215=3400, STS3032=2900, STS3235=3400 -->
   <xacro:arg name="proportional_acc_max"   default="25"/>    <!-- [0-254]; 0 = disable proportional ACC -->
   <!-- Base operating mode -->
   <xacro:property name="base_operating_mode" value="1"/>  <!-- Velocity mode -->
   <!-- Motor-specific parameter — sourced from arg, STS3215 default -->
-  <xacro:property name="sts_max_velocity_steps" value="$(arg sts_max_velocity_steps)"/>  <!-- Max hardware velocity in steps/s -->
+  <xacro:property name="sts3215_max_vel_steps" value="$(arg sts3215_max_vel_steps)"/>  <!-- Max hardware velocity in steps/s -->
   <!-- Proportional ACC parameters (SyncWriteSpe velocity path only) -->
   <!-- ACC given to the wheel with the largest |target - current| velocity delta. -->
@@ -45,5 +42,5 @@
   <xacro:property name="theta" value="${2*pi/3}"/>  <!-- 120° between wheels -->
   <!-- Maximum allowable speed/acceleration/torque for each motor -->
-  <xacro:property name="max_velocity_steps" value="${int(sts_max_velocity_steps * 0.85)}"/> <!-- steps/second (85% of hardware max, 15% safety margin) -->
+  <xacro:property name="max_velocity_steps" value="${int(sts3215_max_vel_steps * 0.85)}"/> <!-- steps/second (85% of hardware max, 15% safety margin) -->
   <xacro:property name="max_velocity_rads" value="${max_velocity_steps*2*pi/4096}"/> <!-- rad/s -->
   <xacro:property name="max_torque_nm" value="2.942"/> <!-- N⋅m (30 kgf⋅cm for STS3215) -->
@@ -73,6 +70,4 @@
         <param name="use_sync_write">$(arg use_sync_write)</param>
         <param name="enable_mock_mode">$(arg use_mock)</param>
-        <!-- Motor-specific parameter (adjust for different STS motor models) -->
-        <param name="max_velocity_steps">${sts_max_velocity_steps}</param>
         <!-- Proportional ACC: scale per-wheel acceleration so all wheels finish ramping in equal time -->
         <param name="proportional_acc_max">${proportional_acc_max}</param>
@@ -83,11 +78,11 @@
       <param name="motor_id">$(arg left_motor_id)</param>
       <param name="operating_mode">${base_operating_mode}</param>
+      <!-- Motor-specific, model-dependent parameter (per joint so different STS models can share this bus) -->
+      <param name="max_velocity_steps">${sts3215_max_vel_steps}</param>
       <command_interface name="velocity"/>
       <state_interface name="position"/>
       <state_interface name="velocity"/>
       <state_interface name="effort"/>
-      <!-- Real-hardware-only telemetry: neither gz_ros2_control/GazeboSimSystem nor
-           mujoco_ros2_control/MujocoSystemInterface know anything beyond
-           position/velocity/effort, and simulated wheels have no real telemetry for these. -->
+      <!-- Real-hardware-only telemetry - sim plugins have nothing beyond position/velocity/effort. -->
       <xacro:if value="${'$(arg ros2_control_hardware_type)' == 'real'}">
         <state_interface name="voltage"/>
@@ -101,11 +96,11 @@
       <param name="motor_id">$(arg back_motor_id)</param>
       <param name="operating_mode">${base_operating_mode}</param>
+      <!-- Motor-specific, model-dependent parameter (per joint so different STS models can share this bus) -->
+      <param name="max_velocity_steps">${sts3215_max_vel_steps}</param>
       <command_interface name="velocity"/>
       <state_interface name="position"/>
       <state_interface name="velocity"/>
       <state_interface name="effort"/>
-      <!-- Real-hardware-only telemetry: neither gz_ros2_control/GazeboSimSystem nor
-           mujoco_ros2_control/MujocoSystemInterface know anything beyond
-           position/velocity/effort, and simulated wheels have no real telemetry for these. -->
+      <!-- Real-hardware-only telemetry - sim plugins have nothing beyond position/velocity/effort. -->
       <xacro:if value="${'$(arg ros2_control_hardware_type)' == 'real'}">
         <state_interface name="voltage"/>
@@ -119,11 +114,11 @@
       <param name="motor_id">$(arg right_motor_id)</param>
       <param name="operating_mode">${base_operating_mode}</param>
+      <!-- Motor-specific, model-dependent parameter (per joint so different STS models can share this bus) -->
+      <param name="max_velocity_steps">${sts3215_max_vel_steps}</param>
       <command_interface name="velocity"/>
       <state_interface name="position"/>
       <state_interface name="velocity"/>
       <state_interface name="effort"/>
-      <!-- Real-hardware-only telemetry: neither gz_ros2_control/GazeboSimSystem nor
-           mujoco_ros2_control/MujocoSystemInterface know anything beyond
-           position/velocity/effort, and simulated wheels have no real telemetry for these. -->
+      <!-- Real-hardware-only telemetry - sim plugins have nothing beyond position/velocity/effort. -->
       <xacro:if value="${'$(arg ros2_control_hardware_type)' == 'real'}">
         <state_interface name="voltage"/>
@@ -133,39 +128,26 @@
       </xacro:if>
     </joint>
-    <!-- mujoco_ros2_control's IMU/lidar sensors must live inside the SAME <ros2_control>
-         block as the MujocoSystemInterface <hardware><plugin> above - each ros2_control
-         block is a separate hardware-plugin instance with its own isolated HardwareInfo,
-         so a sensor declared in a different block (like lekiwi_imu below) would never be
-         seen by this one. These map to lekiwi_description/mjcf/base_subtree.xml's MJCF
-         sensors. -->
+    <!-- IMU/lidar sensors must live in this SAME <ros2_control> block as the plugin above -
+         each block is an isolated HardwareInfo, so lekiwi_imu below couldn't see them. -->
     <xacro:if value="${'$(arg ros2_control_hardware_type)' == 'mujoco'}">
-      <!-- BNO055 IMU - mujoco_type="imu" tells MujocoSystemInterface::register_sensors to
-           look for MJCF sensors named bno055_quat/bno055_gyro/bno055_accel (the fixed
-           _quat/_gyro/_accel suffix convention), attached to base_subtree.xml's imu_site. Same
-           state_interface list as the real-hardware lekiwi_imu block below - duplicated,
-           not shared via a macro, to keep both branches readable independently. -->
-      <sensor name="bno055">
-        <param name="mujoco_type">imu</param>
-        <state_interface name="orientation.x"/>
-        <state_interface name="orientation.y"/>
-        <state_interface name="orientation.z"/>
-        <state_interface name="orientation.w"/>
-        <state_interface name="angular_velocity.x"/>
-        <state_interface name="angular_velocity.y"/>
-        <state_interface name="angular_velocity.z"/>
-        <state_interface name="linear_acceleration.x"/>
-        <state_interface name="linear_acceleration.y"/>
-        <state_interface name="linear_acceleration.z"/>
-      </sensor>
-      <!-- LD19 lidar - matched to base_subtree.xml's 360 "lidar-<i>" MJCF rangefinder sensors by
-           this <sensor> block's own name ("lidar" - matching the part of "lidar-<i>" before
-           the last hyphen, per mujoco_lidar.cpp's parse_lidar_name - NOT the frame_name
-           param below, easy to mix up), not by a mujoco_type param (the lidar registration
-           path is separate from register_sensors).
-           angle_increment/min_angle/max_angle intentionally don't match the real LD19's
-           452-sample resolution - see base_subtree.xml's lidar comment for why. laserscan_topic
-           matches the real ldlidar_ros2_node's /scan topic (lekiwi_bringup/config/laser.yaml)
-           so downstream consumers (SLAM, Nav2) don't need to know whether they're talking to
-           real or simulated lidar. -->
+      <!-- mujoco_type=imu maps to base_subtree.xml's bno055_quat/gyro/accel MJCF sensors -
+           same state_interfaces as the real block below (duplicated), gated on imu:=true. -->
+      <xacro:if value="${'$(arg imu)' == 'true'}">
+        <sensor name="bno055">
+          <param name="mujoco_type">imu</param>
+          <state_interface name="orientation.x"/>
+          <state_interface name="orientation.y"/>
+          <state_interface name="orientation.z"/>
+          <state_interface name="orientation.w"/>
+          <state_interface name="angular_velocity.x"/>
+          <state_interface name="angular_velocity.y"/>
+          <state_interface name="angular_velocity.z"/>
+          <state_interface name="linear_acceleration.x"/>
+          <state_interface name="linear_acceleration.y"/>
+          <state_interface name="linear_acceleration.z"/>
+        </sensor>
+      </xacro:if>
+      <!-- Matched to base_subtree.xml's MJCF sensors by this block's name ("lidar"), not
+           frame_name. Resolution intentionally differs from the real LD19 - see base_subtree.xml. -->
       <sensor name="lidar">
         <param name="frame_name">laser_frame</param>
@@ -180,12 +162,7 @@
   </ros2_control>
   <!-- ROS 2 CONTROL -->
-  <!-- Sensor interface (BNO055 IMU) for real hardware. Omitted in gazebo mode:
-       base.module.xacro's native Gazebo IMU sensor + ros_gz_bridge supplies
-       /imu_sensor_broadcaster/imu directly instead (see the comment there). Omitted in
-       mujoco mode too: the equivalent sensor lives inside the lekiwi_base system block
-       above instead (mujoco_ros2_control requires it in the same <ros2_control> block as
-       the plugin declaration). imu_sensor_broadcaster itself isn't spawned in gazebo mode
-       either (control.launch.py), so a lekiwi_imu block would go unclaimed there anyway. -->
-  <xacro:if value="${'$(arg ros2_control_hardware_type)' == 'real'}">
+  <!-- Real hardware only - gazebo bridges its own IMU sensor instead (base.module.xacro),
+       mujoco hosts its sensor inside lekiwi_base above; also omitted when imu:=false. -->
+  <xacro:if value="${'$(arg ros2_control_hardware_type)' == 'real' and '$(arg imu)' == 'true'}">
     <ros2_control name="lekiwi_imu" type="sensor">
       <hardware>

File: lekiwi_description/urdf/base/base.module.xacro (robot description, xacro)
@@ -58,9 +58,6 @@
     <!-- Laser frame -->
     <link name="laser_frame"/>
-    <!-- Gazebo simulation: LD19 lidar. update_rate/samples/angle/range values measured
-         directly off the real robot's /scan topic, not the datasheet. gz_frame_id overrides
-         gz-sim's default scoped sensor frame_id to the plain "laser_frame" the real
-         ldlidar_ros2_node publishes, so TF resolves the same in sim as on hardware
-         (unofficial SDF tag - gazebosim/gz-sensors#306). Inert outside Gazebo. -->
+    <!-- Values measured off the real /scan topic, not the datasheet. gz_frame_id matches
+         ldlidar_ros2_node's real "laser_frame" so TF resolves the same in sim (gz-sensors#306). -->
     <gazebo reference="laser_frame">
       <sensor name="lidar" type="gpu_lidar">
@@ -110,33 +107,30 @@
     <!-- IMU frame -->
     <link name="imu_frame"/>
-    <!-- Gazebo simulation: BNO055 IMU. Attached to imu_frame and published on
-         /imu_sensor_broadcaster/imu (imu_sensor_broadcaster's own topic/frame_id) so EKF
-         needs no reconfiguration between real and sim; imu_sensor_broadcaster itself isn't
-         spawned in gazebo mode to avoid racing with this bridged topic. update_rate=50
-         matches controller_manager's rate. Noise stddevs are sqrt() of
-         imu_sensor_broadcaster's static_covariance_* params (gz has no separate orientation
-         noise, so orientation comes out noise-free). gz_frame_id/inertness: see lidar above. -->
-    <gazebo reference="imu_frame">
-      <sensor name="imu" type="imu">
-        <pose>0 0 0 0 0 0</pose>
-        <topic>imu_sensor_broadcaster/imu</topic>
-        <gz_frame_id>imu_frame</gz_frame_id>
-        <update_rate>50</update_rate>
-        <always_on>true</always_on>
-        <visualize>false</visualize>
-        <imu>
-          <angular_velocity>
-            <x><noise type="gaussian"><mean>0.0</mean><stddev>0.00316</stddev></noise></x>
-            <y><noise type="gaussian"><mean>0.0</mean><stddev>0.00316</stddev></noise></y>
-            <z><noise type="gaussian"><mean>0.0</mean><stddev>0.00316</stddev></noise></z>
-          </angular_velocity>
-          <linear_acceleration>
-            <x><noise type="gaussian"><mean>0.0</mean><stddev>0.01414</stddev></noise></x>
-            <y><noise type="gaussian"><mean>0.0</mean><stddev>0.01414</stddev></noise></y>
-            <z><noise type="gaussian"><mean>0.0</mean><stddev>0.01414</stddev></noise></z>
-          </linear_acceleration>
-        </imu>
-      </sensor>
-    </gazebo>
+    <!-- Bridges to imu_sensor_broadcaster's own topic so EKF needs no sim/real reconfig;
+         imu_sensor_broadcaster itself isn't spawned in gazebo mode, to avoid racing this. -->
+    <xacro:if value="${'$(arg imu)' == 'true'}">
+      <gazebo reference="imu_frame">
+        <sensor name="imu" type="imu">
+          <pose>0 0 0 0 0 0</pose>
+          <topic>imu_sensor_broadcaster/imu</topic>
+          <gz_frame_id>imu_frame</gz_frame_id>
+          <update_rate>50</update_rate>
+          <always_on>true</always_on>
+          <visualize>false</visualize>
+          <imu>
+            <angular_velocity>
+              <x><noise type="gaussian"><mean>0.0</mean><stddev>0.00316</stddev></noise></x>
+              <y><noise type="gaussian"><mean>0.0</mean><stddev>0.00316</stddev></noise></y>
+              <z><noise type="gaussian"><mean>0.0</mean><stddev>0.00316</stddev></noise></z>
+            </angular_velocity>
+            <linear_acceleration>
+              <x><noise type="gaussian"><mean>0.0</mean><stddev>0.01414</stddev></noise></x>
+              <y><noise type="gaussian"><mean>0.0</mean><stddev>0.01414</stddev></noise></y>
+              <z><noise type="gaussian"><mean>0.0</mean><stddev>0.01414</stddev></noise></z>
+            </linear_acceleration>
+          </imu>
+        </sensor>
+      </gazebo>
+    </xacro:if>
     <!-- Respeaker flex mic link -->
     <link name="mic_link">
