Commit message: removed webcam

File: lekiwi_description/urdf/base/base.common.xacro (robot description, xacro)
@@ -13,9 +13,4 @@
   <xacro:property name="laser_base_offset_z" value="0.0915"/>
   <xacro:property name="laser_offset_rx" value="${pi/2}"/>
-  <!-- HD camera offsets from base_link -->
-  <xacro:property name="camera_base_offset_x" value="0.114"/>
-  <xacro:property name="camera_base_offset_z" value="0.026"/>
-  <xacro:property name="camera_offset_ry" value="${pi/2}"/>
-  <xacro:property name="camera_frame_offset_rz" value="${3*pi/2}"/>
   <!-- LDLidar frame offsets from laser_link -->
   <xacro:property name="laser_frame_offset_z" value="0.027"/>

File: lekiwi_description/urdf/base/base.module.xacro (robot description, xacro)
@@ -80,26 +80,4 @@
     <!-- IMU frame -->
     <link name="imu_frame"/>
-    <!-- Camera link -->
-    <link name="camera_link">
-      <visual>
-        <origin xyz="0 0 0" rpy="0 0 0"/>
-        <geometry>
-          <mesh filename="package://lekiwi_description/meshes/base/hd_webcam.stl"/>
-        </geometry>
-        <material name="base_charcoal"/>
-      </visual>
-      <collision>
-        <origin xyz="0 0 0" rpy="0 0 0"/>
-        <geometry>
-          <mesh filename="package://lekiwi_description/meshes/base/hd_webcam.stl"/>
-        </geometry>
-      </collision>
-      <inertial>
-        <mass value="0.05"/>
-        <inertia ixx="0.00001" ixy="0.0" ixz="0.0" iyy="0.00001" iyz="0.0" izz="0.00001"/>
-      </inertial>
-    </link>
-    <!-- Camera frame -->
-    <link name="camera"/>
     <!-- Left wheel link -->
     <link name="left_wheel_link">
@@ -187,16 +165,4 @@
       <origin xyz="0 0 0" rpy="0 0 0"/>
     </joint>
-    <!-- camera fixed joint -->
-    <joint name="camera_joint" type="fixed">
-      <parent link="base_link"/>
-      <child link="camera_link"/>
-      <origin xyz="${camera_base_offset_x} 0 ${camera_base_offset_z}" rpy="0 ${camera_offset_ry} 0"/>
-    </joint>
-    <!-- camera_frame fixed joint -->
-    <joint name="camera_frame_joint" type="fixed">
-      <parent link="camera_link"/>
-      <child link="camera"/>
-      <origin xyz="0 0 0" rpy="0 0 ${camera_frame_offset_rz}"/>
-    </joint>
     <!-- left wheel joint: 60 degrees anti-clockwise from +X at radius wheel_base_radius -->
     <joint name="left_wheel_joint" type="continuous">

File: lekiwi_description/urdf/base/base.urdf (robot description, URDF)
Before this commit: robot lekiwi, 11 links, 10 joints
Links:
- removed link camera
- removed link camera_link
Joints:
- removed joint camera_frame_joint
- removed joint camera_joint

File: lekiwi_description/urdf/k2.urdf (robot description, URDF)
Before this commit: robot k2, 17 links, 16 joints
Links:
- removed link camera
- removed link camera_link
Joints:
- removed joint camera_frame_joint
- removed joint camera_joint

Commit message: added respeaker URDF, integrated cloudini for pointcloud compression

File: lekiwi_description/urdf/base/base.common.xacro (robot description, xacro)
@@ -18,3 +18,6 @@
   <xacro:property name="imu_base_offset_x" value="-0.044"/>
   <xacro:property name="imu_base_offset_z" value="0.08"/>
+  <!-- Respeaker flex mic offsets from base_link -->
+  <xacro:property name="mic_base_offset_x" value="-0.045042"/>
+  <xacro:property name="mic_base_offset_z" value="0.10901"/>
 </robot>

File: lekiwi_description/urdf/base/base.module.xacro (robot description, xacro)
@@ -80,4 +80,24 @@
     <!-- IMU frame -->
     <link name="imu_frame"/>
+    <!-- Respeaker flex mic link -->
+    <link name="mic_link">
+      <visual>
+        <origin xyz="0 0 0" rpy="0 0 0"/>
+        <geometry>
+          <mesh filename="package://lekiwi_description/meshes/base/respeaker_flex_mic.stl"/>
+        </geometry>
+        <material name="base_charcoal"/>
+      </visual>
+      <collision>
+        <origin xyz="0 0 0" rpy="0 0 0"/>
+        <geometry>
+          <mesh filename="package://lekiwi_description/meshes/base/respeaker_flex_mic.stl"/>
+        </geometry>
+      </collision>
+      <inertial>
+        <mass value="0.05"/>
+        <inertia ixx="0.00001" ixy="0.0" ixz="0.0" iyy="0.00001" iyz="0.0" izz="0.00001"/>
+      </inertial>
+    </link>
     <!-- Left wheel link -->
     <link name="left_wheel_link">
@@ -165,4 +185,10 @@
       <origin xyz="0 0 0" rpy="0 0 0"/>
     </joint>
+    <!-- Respeaker flex mic fixed joint -->
+    <joint name="mic_joint" type="fixed">
+      <parent link="base_link"/>
+      <child link="mic_link"/>
+      <origin xyz="${mic_base_offset_x} 0 ${mic_base_offset_z}" rpy="0 0 0"/>
+    </joint>
     <!-- left wheel joint: 60 degrees anti-clockwise from +X at radius wheel_base_radius -->
     <joint name="left_wheel_joint" type="continuous">

File: lekiwi_description/urdf/base/base.urdf (robot description, URDF)
Before this commit: robot lekiwi, 9 links, 8 joints
Links:
- added link mic_link, mass 0.05; collision mesh filename=../../meshes/base/respeaker_flex_mic.stl; visual mesh filename=../../meshes/base/respeaker_flex_mic.stl
Joints:
- added joint mic_joint: type fixed, parent base_link, child mic_link, origin xyz=-0.045042 0 0.10901 rpy=0 0 0

File: lekiwi_description/urdf/k2.urdf (robot description, URDF)
Before this commit: robot k2, 15 links, 14 joints
Links:
- added link mic_link, mass 0.05; collision mesh filename=../meshes/base/respeaker_flex_mic.stl; visual mesh filename=../meshes/base/respeaker_flex_mic.stl
Joints:
- added joint mic_joint: type fixed, parent base_link, child mic_link, origin xyz=-0.045042 0 0.10901 rpy=0 0 0
- joint pan_joint: limit lower=-1.5707963267948966 upper=1.5707963267948966 effort=2.942 velocity=1e6 -> lower=-1.5708 upper=1.5708 effort=2.942 velocity=1e6
- joint tilt_joint: limit lower=-1.5707963267948966 upper=1.5707963267948966 effort=2.942 velocity=1e6 -> lower=-1.5708 upper=1.5708 effort=2.942 velocity=1e6
