Commit message: Add lekiwi_mujoco sim core; derive wheel geometry from control.yaml
Stage 2 of the mujoco-branch migration: the pure-Python MjSpec-based
simulation core (model building, Gymnasium env, keyboard preview,
benchmarking), plus the MJCF rewrite it depends on (16-roller-per-wheel
omni-wheel contact model in base_subtree.xml) and the URDF/xacro changes
that make wheel_radius/wheel_offset/wheel_base_radius derive from
lekiwi_control's control.yaml instead of being duplicated as hardcoded
xacro literals. Prebuilt base.urdf/base_pantilt.urdf and the three
lekiwi_mujoco snapshot MJCFs are regenerated from these sources.

control.launch.py now passes base_controller_config through to xacro,
matching the new required arg.

Co-Authored-By: Claude Sonnet 5 <noreply@anthropic.com>

File: lekiwi_description/urdf/base/base.common.xacro (robot description, xacro)
@@ -6,6 +6,15 @@
   <!-- Base mesh rotation about Z (rad) -->
   <xacro:property name="base_offset_rz" value="${3*pi/2}"/>
+  <!-- Common wheel geometry: used by ROS controllers, URDF and MuJoCo. -->
+  <!-- Required input: base_controller_config:=/path/to/base/control.yaml.
+       The launch/integration layer supplies it; description does not depend on control. -->
+  <xacro:property name="base_geometry" value="${xacro.load_yaml('$(arg base_controller_config)')['base_controller']['ros__parameters']}"/>
+  <xacro:property name="wheel_radius" value="${base_geometry['wheel_radius']}"/>
+  <xacro:property name="offset" value="${base_geometry['wheel_offset']}"/>
+  <!-- CAD wheel mesh radius in metres; a mesh reference measurement, not an operating parameter. -->
+  <xacro:property name="wheel_mesh_radius" value="0.051"/>
+  <xacro:property name="wheel_mesh_scale" value="${wheel_radius / wheel_mesh_radius}"/>
   <!-- Wheel mount offsets -->
-  <xacro:property name="wheel_base_radius" value="0.132239"/>
+  <xacro:property name="wheel_base_radius" value="${base_geometry['robot_radius']}"/>
   <xacro:property name="wheel_base_offset_z" value="0.01036"/>
   <!-- LD06 laser offsets from base_link -->

File: lekiwi_description/urdf/base/base.control.xacro (robot description, xacro)
@@ -42,6 +42,4 @@
   <xacro:property name="proportional_acc_max" value="$(arg proportional_acc_max)"/>        <!-- [0-254] -->
   <!-- Wheel geometry for omnidirectional control -->
-  <xacro:property name="wheel_radius" value="0.051"/>  <!-- meters -->
-  <xacro:property name="offset" value="${pi/3}"/>  <!-- 60° -->
   <xacro:property name="theta" value="${2*pi/3}"/>  <!-- 120° between wheels -->
   <!-- Maximum allowable speed/acceleration/torque for each motor -->

File: lekiwi_description/urdf/base/base.module.xacro (robot description, xacro)
@@ -158,12 +158,12 @@
         <origin xyz="0 0 0" rpy="0 0 0"/>
         <geometry>
-          <mesh filename="package://lekiwi_description/meshes/omni_wheel.stl"/>
-        </geometry>
-        <material name="base_charcoal"/>
-      </visual>
-      <collision>
-        <origin xyz="0 0 0" rpy="0 0 0"/>
-        <geometry>
-          <mesh filename="package://lekiwi_description/meshes/omni_wheel.stl"/>
+          <mesh filename="package://lekiwi_description/meshes/omni_wheel.stl" scale="${wheel_mesh_scale} ${wheel_mesh_scale} ${wheel_mesh_scale}"/>
+        </geometry>
+        <material name="base_charcoal"/>
+      </visual>
+      <collision>
+        <origin xyz="0 0 0" rpy="0 0 0"/>
+        <geometry>
+          <mesh filename="package://lekiwi_description/meshes/omni_wheel.stl" scale="${wheel_mesh_scale} ${wheel_mesh_scale} ${wheel_mesh_scale}"/>
         </geometry>
       </collision>
@@ -178,12 +178,12 @@
         <origin xyz="0 0 0" rpy="0 0 0"/>
         <geometry>
-          <mesh filename="package://lekiwi_description/meshes/omni_wheel.stl"/>
-        </geometry>
-        <material name="base_charcoal"/>
-      </visual>
-      <collision>
-        <origin xyz="0 0 0" rpy="0 0 0"/>
-        <geometry>
-          <mesh filename="package://lekiwi_description/meshes/omni_wheel.stl"/>
+          <mesh filename="package://lekiwi_description/meshes/omni_wheel.stl" scale="${wheel_mesh_scale} ${wheel_mesh_scale} ${wheel_mesh_scale}"/>
+        </geometry>
+        <material name="base_charcoal"/>
+      </visual>
+      <collision>
+        <origin xyz="0 0 0" rpy="0 0 0"/>
+        <geometry>
+          <mesh filename="package://lekiwi_description/meshes/omni_wheel.stl" scale="${wheel_mesh_scale} ${wheel_mesh_scale} ${wheel_mesh_scale}"/>
         </geometry>
       </collision>
@@ -198,12 +198,12 @@
         <origin xyz="0 0 0" rpy="0 0 0"/>
         <geometry>
-          <mesh filename="package://lekiwi_description/meshes/omni_wheel.stl"/>
-        </geometry>
-        <material name="base_charcoal"/>
-      </visual>
-      <collision>
-        <origin xyz="0 0 0" rpy="0 0 0"/>
-        <geometry>
-          <mesh filename="package://lekiwi_description/meshes/omni_wheel.stl"/>
+          <mesh filename="package://lekiwi_description/meshes/omni_wheel.stl" scale="${wheel_mesh_scale} ${wheel_mesh_scale} ${wheel_mesh_scale}"/>
+        </geometry>
+        <material name="base_charcoal"/>
+      </visual>
+      <collision>
+        <origin xyz="0 0 0" rpy="0 0 0"/>
+        <geometry>
+          <mesh filename="package://lekiwi_description/meshes/omni_wheel.stl" scale="${wheel_mesh_scale} ${wheel_mesh_scale} ${wheel_mesh_scale}"/>
         </geometry>
       </collision>

File: lekiwi_description/urdf/base/base.urdf (robot description, URDF)
Before this commit: robot lekiwi, 10 links, 9 joints
Links:
- link back_wheel_link: geometry collision mesh filename=package://lekiwi_description/meshes/omni_wheel.stl scale=1.0 1.0 1.0; visual mesh filename=package://lekiwi_description/meshes/omni_wheel.stl scale=1.0 1.0 1.0
- link left_wheel_link: geometry collision mesh filename=package://lekiwi_description/meshes/omni_wheel.stl scale=1.0 1.0 1.0; visual mesh filename=package://lekiwi_description/meshes/omni_wheel.stl scale=1.0 1.0 1.0
- link right_wheel_link: geometry collision mesh filename=package://lekiwi_description/meshes/omni_wheel.stl scale=1.0 1.0 1.0; visual mesh filename=package://lekiwi_description/meshes/omni_wheel.stl scale=1.0 1.0 1.0

File: lekiwi_description/urdf/base_pantilt/base_pantilt.control.xacro (robot description, xacro)
@@ -57,6 +57,4 @@
   <xacro:property name="proportional_acc_max" value="$(arg proportional_acc_max)"/>        <!-- [0-254] -->
   <!-- Wheel geometry for omnidirectional control -->
-  <xacro:property name="wheel_radius" value="0.051"/>  <!-- meters -->
-  <xacro:property name="offset" value="${pi/3}"/>  <!-- 60° -->
   <xacro:property name="theta" value="${2*pi/3}"/>  <!-- 120° between wheels -->
   <!-- Maximum allowable speed/acceleration/torque for each motor -->

File: lekiwi_description/urdf/base_pantilt/base_pantilt.urdf (robot description, URDF)
Before this commit: robot lekiwi, 16 links, 15 joints
Links:
- link back_wheel_link: geometry collision mesh filename=package://lekiwi_description/meshes/omni_wheel.stl scale=1.0 1.0 1.0; visual mesh filename=package://lekiwi_description/meshes/omni_wheel.stl scale=1.0 1.0 1.0
- link left_wheel_link: geometry collision mesh filename=package://lekiwi_description/meshes/omni_wheel.stl scale=1.0 1.0 1.0; visual mesh filename=package://lekiwi_description/meshes/omni_wheel.stl scale=1.0 1.0 1.0
- link right_wheel_link: geometry collision mesh filename=package://lekiwi_description/meshes/omni_wheel.stl scale=1.0 1.0 1.0; visual mesh filename=package://lekiwi_description/meshes/omni_wheel.stl scale=1.0 1.0 1.0

File: lekiwi_mujoco/mjcf/base.mjcf.xacro (robot description, xacro)
@@ -4,11 +4,10 @@
      base_pantilt.mjcf.xacro for base+payload, add base_<payload>.mjcf.xacro for new payloads
      rather than an arg-driven branch here. Geometry lives in base_shared.xml/base_subtree.xml.
-     Standalone: xacro base.mjcf.xacro > /tmp/lekiwi_base.xml
-     control.launch.py runs the same command at launch time and passes the result as
+     Generate runnable models with scripts/build_mujoco_models.py.
+     control.launch.py uses this MjSpec generator and passes the result as
      mujoco_model. Uses $(find package), not relative paths - relative paths resolve against
      the output file's location at launch time, not this file's own directory. -->
 <mujoco xmlns:xacro="http://www.ros.org/wiki/xacro" model="lekiwi">
-  <xacro:arg name="scene" default="true"/>
-  <!-- xacro:include, not a plain <include> - base_shared.xml needs $(arg scene) resolved. -->
+  <!-- Robot assets only; build_mujoco_models.py composes a separate scene. -->
   <xacro:include filename="$(find lekiwi_mujoco)/mjcf/base_shared.xml"/>
   <worldbody>

File: lekiwi_mujoco/mjcf/base_pantilt.mjcf.xacro (robot description, xacro)
@@ -5,14 +5,13 @@
      mounts at base_pantilt.common.xacro's pantilt_base_offset_x/z, matching
      base_pantilt.urdf.xacro's fixed joint.
-     Standalone: xacro base_pantilt.mjcf.xacro pantilt_config:=pt101 > /tmp/lekiwi_pt101.xml
-     control.launch.py runs the same command at launch time when payload:=pantilt. -->
+     Use scripts/build_mujoco_models.py to synchronize URDF parameters and compose
+     the scene. control.launch.py uses that same generator at launch time. -->
 <mujoco xmlns:xacro="http://www.ros.org/wiki/xacro" model="lekiwi_pantilt">
   <xacro:arg name="pantilt_config" default="pt101"/>
-  <xacro:arg name="scene" default="true"/>
   <!-- Declared here BEFORE including pantilt.mjcf.xacro (which defaults standalone to true)
        so this default wins - xacro uses the first <xacro:arg> declaration seen. Suppresses
        pantilt.mjcf.xacro's own worldbody/scene emission. -->
   <xacro:arg name="standalone" default="false"/>
-  <!-- xacro:include, not a plain <include> - base_shared.xml needs $(arg scene) resolved. -->
+  <!-- Robot assets only; build_mujoco_models.py composes a separate scene. -->
   <xacro:include filename="$(find lekiwi_mujoco)/mjcf/base_shared.xml"/>
   <xacro:include filename="$(find pt_description)/mjcf/pantilt.mjcf.xacro"/>
