Commit message: Add the MuJoCo simulation, simulated e-stop, payload config ownership and README restructure (#10)
* Create lekiwi_mujoco package, move MJCF assets out of lekiwi_description

Stage 1 of the mujoco-branch migration: a bare ament_python package
skeleton hosting the MJCF models, repointing lekiwi_control's mujoco
xacro processing and the models' own internal includes at it.

Co-Authored-By: Claude Sonnet 5 <noreply@anthropic.com>

* Add lekiwi_mujoco sim core; derive wheel geometry from control.yaml

Stage 2 of the mujoco-branch migration: the pure-Python MjSpec-based
simulation core (model building, Gymnasium env, keyboard preview,
benchmarking), plus the MJCF rewrite it depends on (16-roller-per-wheel
omni-wheel contact model in base_subtree.xml) and the URDF/xacro changes
that make wheel_radius/wheel_offset/wheel_base_radius derive from
lekiwi_control's control.yaml instead of being duplicated as hardcoded
xacro literals. Prebuilt base.urdf/base_pantilt.urdf and the three
lekiwi_mujoco snapshot MJCFs are regenerated from these sources.

control.launch.py now passes base_controller_config through to xacro,
matching the new required arg.

Co-Authored-By: Claude Sonnet 5 <noreply@anthropic.com>

* Generate MJCF via lekiwi_mujoco.build_mujoco_models in control.launch.py

Stage 4 of the mujoco-branch migration: replace the raw xacro-subprocess
MJCF generation with the MjSpec-based build_mujoco_models module, which
also syncs velocity/position limits and payload optical-frame conventions
that a plain xacro pass didn't handle. Adds the mujoco_scene launch arg
(flat/none/custom scene path) alongside the existing mujoco_model override.

Co-Authored-By: Claude Sonnet 5 <noreply@anthropic.com>

* Rename sim gui arg to mujoco_gui, default to false (headless by default)

gui:=true was the actual cause of the "MuJoCo camera GLFW" crash, not a
hard headless-rendering limitation: it forced mujoco_headless:=false,
so MujocoSystemInterface tried to open a real GLFW window on a
display-less Pi and took the whole ros2_control_node down with it.
With mujoco_headless:=true (the new default), the plugin's own
HeadlessAdapter path runs with no display/GPU/OpenGL needed at all,
and the camera-init failure degrades to a warning instead of a crash.

Co-Authored-By: Claude Sonnet 5 <noreply@anthropic.com>

* Update sim docs: mujoco_gui rename, camera GLFW no longer a hard limit

Reflects the root-cause fix in the previous commit: sim:=true is
headless by default now, and the OAK-D camera-init failure is a
graceful warning, not a crash, in either repo.

Co-Authored-By: Claude Sonnet 5 <noreply@anthropic.com>

* Wire BAM-identified STS3215 params; drop instance.py, redundant scripts

Copies so_arm_mujoco/mjcf/sts3215.mjcf.xacro verbatim (minus its unused
visual/collision sub-classes, which collide with pt_description's own
same-named classes when payload variants compose) and wires it into the
wheel joints via class="sts3215". Only damping actually applies from the
MJCF class - armature/frictionloss get overwritten by config/mujoco.yaml's
actuators.wheel block regardless, which now carries the BAM values
directly. Wheel joints override damping="0" locally: BAM identified it
for a small-range position-controlled arm joint, not a continuously
spinning velocity-controlled wheel, and it measurably fights the
velocity actuator at speed (confirmed via test_measured_motion_in_all_payloads
regressing before this override).

Also, matching so_arm_mujoco's file layout:
- Removed the 3 scripts/*.py shims (sys.path.insert + import + main()) -
  setup.py's console_scripts already point directly at the package
  modules; standalone `python3 -m lekiwi_mujoco.<module>` invocation is
  now documented in each module's own docstring instead.
- Removed instance.py's RobotInstance/multi-instance-prefix/spawn-transform
  support - lekiwi only ever runs one robot today. Its named-element
  resolution (RobotBindings) is still needed and used by every consumer,
  so it's inlined into simulation.py instead, minus prefix handling.
  world.attach() needs prefix='' passed explicitly now - its own default
  isn't empty string, unlike the value RobotInstance used to supply.

Co-Authored-By: Claude Sonnet 5 <noreply@anthropic.com>

* CI: build/test lekiwi_mujoco and add cross-platform mujoco job

Recording-related additions from the mujoco branch (rosbag2 apt packages,
test_recording.py) are intentionally left out; basedpyright step kept.

Co-Authored-By: Claude Sonnet 5 <noreply@anthropic.com>

* Add lekiwi_mujoco docs, viewer travel trail and no-ROS regression test

Docs from the mujoco branch, adapted to this migration: standalone use is
`python3 -m lekiwi_mujoco.<module>` (scripts/ shims removed), multi-instance
and prefix/spawn sections dropped with instance.py, rosbag2/MCAP mentions
reworded since recording isn't part of lekiwi yet. Adds the bounded
visual-only XY trail in mujoco_preview.py (+ test_trail.py) and
test_without_ros.py, which needs mujoco and xacro pip-installed (as CI
does) since it runs in isolated mode.

Co-Authored-By: Claude Sonnet 5 <noreply@anthropic.com>

* Consolidate docs: package details in lekiwi_mujoco/README, overview in top-level README

lekiwi_mujoco/README.md now carries usage, ROS integration, parameter
ownership, STS3215 notes, model limitations, API, testing and open items
(absorbing mjcf/README.md, mjcf/PARAMETERS.md, architecture-review.md and
the durable parts of ros-parity.md, all removed). docs/ keeps only the
observation contract and the remote-viewer plan, updated with current
status. Top-level README gains the lekiwi_mujoco package, its Python
dependencies, a pointer in Simulation, and the structure entry.

Co-Authored-By: Claude Sonnet 5 <noreply@anthropic.com>

* Remove the Gymnasium adapter and the mujoco docs folder

Nothing in the robot used LeKiwiEnv (it defined no reward or task), so drop
mujoco_env.py, observations.py, their tests, the [gym] extra and the
gymnasium installs in CI. A future RL setup would be a separate lekiwi_gym
package built on lekiwi_mujoco's build() and Simulation. Also remove the
remote-viewer plan (superseded by Foxglove) and the observation contract doc.

Co-Authored-By: Claude Sonnet 5 <noreply@anthropic.com>

* Native lidar, camera plugin and arena scene for the MuJoCo sim

The 360 per-ray rangefinders cost about 9 ms per 2 ms physics step (99% of
the step), holding the sim to ~0.17x real time on the Pi. The lidar is now a
native mujoco.plugin.lidar sensor cast at 5 Hz (~1.0x), published by
Mujoco3dLidarPlugin as /scan_raw and filtered to /scan with laser_filters
(no-hit to inf, pan-tilt self-occlusion mask). The plugin excludes no bodies,
so plugin models drop the LD06 mesh around the ray origin; standalone tools
keep rangefinders (--lidar plugin|rangefinder).

Also: CameraPlugin (headless EGL, oak_rgb_camera_optical_frame, image
upside down like the inverted real mount), FreeJointStatePublisherPlugin
ground truth, an arena scene, control.launch.py enable_odom_tf (default
true; lekiwi.launch.py passes false because the EKF publishes it).

Base speed limits: the controller has no limit parameters, so remove the
dead linear/angular blocks from control.yaml; the ROS sim follows teleop and
Nav2 directly, and standalone tools use command.base_velocity in
mujoco.yaml. Tests for the moved limits and removed legacy lidar block are
updated; READMEs rewritten for replication.

Co-Authored-By: Claude Sonnet 5 <noreply@anthropic.com>

* Bump pantilt_ros2 submodule pointer to its README cleanup

Co-Authored-By: Claude Sonnet 5 <noreply@anthropic.com>

* Add mujoco_scene argument to lekiwi.launch.py (sim only)

Passed through to control.launch.py only when sim:=true, so the full stack
can run in the walled arena scene; ignored on real hardware.

Co-Authored-By: Claude Sonnet 5 <noreply@anthropic.com>

* Sim: synchronous lidar, compressed camera topic, 5 Hz camera, rename laser filter configs

- Native lidar runs synchronously so scans carry current timestamps
- Republish /oak/rgb/image_raw as compressed via image_transport
- Camera at 5 Hz: headless software rendering cannot sustain more on the Pi
- Rename sim_laser_filter*.yaml to mujoco_laser_filter*.yaml

Co-Authored-By: Claude Sonnet 5 <noreply@anthropic.com>

* lekiwi_mujoco: take the pan-tilt MJCF from pt_mujoco; regenerate snapshots with relative mesh paths

Co-Authored-By: Claude Sonnet 5 <noreply@anthropic.com>

* lekiwi_mujoco: mount the pan-tilt payload from pt_mujoco instead of embedding its MJCF

The builder expands the robot URDF, has pt_mujoco build the payload from it and attaches it at
the URDF's pantilt_mount_joint. Payload servo parameters, limits, camera and its plugin config now
belong to pt_mujoco; lekiwi keeps only a 5 Hz camera-rate override for the Pi. The generated models
are numerically identical to before (world poses and 3 s of simulated motion match exactly).

Co-Authored-By: Claude Sonnet 5 <noreply@anthropic.com>

* Document the pt_mujoco payload split; select pt_mujoco in CI

Co-Authored-By: Claude Sonnet 5 <noreply@anthropic.com>

* Bump pantilt_ros2 to the version that provides pt_mujoco

Co-Authored-By: Claude Sonnet 5 <noreply@anthropic.com>

* lekiwi_mujoco: regenerate pan-tilt models with pt_mujoco's BAM servo profile

Co-Authored-By: Claude Sonnet 5 <noreply@anthropic.com>

* lekiwi_bringup: move the pantilt laser filter to config/pantilt_laser_filter.yaml

The filter is looked up as config/<payload>_laser_filter.yaml, so the empty payloads/pantilt
folders are gone. A test covers the lookup and is added to CI.

Co-Authored-By: Claude Sonnet 5 <noreply@anthropic.com>

* README: keep the focus on the base and describe how payloads are wired in

Co-Authored-By: Claude Sonnet 5 <noreply@anthropic.com>

* Rename the teleop configs to base_teleop.yaml and <payload>_teleop.yaml

config/base/teleop.yaml -> base_teleop.yaml and config/payloads/pantilt/teleop.yaml ->
pantilt_teleop.yaml. teleop.launch.py loads config/payloads/<payload>/<payload>_teleop.yaml, and a
test covers the wiring for the base-only and pantilt cases.

Co-Authored-By: Claude Sonnet 5 <noreply@anthropic.com>

* lekiwi: read the pan-tilt servo profile from pt_control; drop the payload urdf_config.yaml

The pan-tilt's internal_* values now come from pt_control's urdf_config.yaml (defaults 65/50/0),
so they are tuned in one place for standalone and lekiwi. proportional_vel_max, a bus-level setting,
moves to the base urdf_config.yaml. The wheels keep 254/254/100. The real-mode ros2_control block is
identical to before for both the base and base + pan-tilt. Prebuilt URDF regenerated.

Co-Authored-By: Claude Sonnet 5 <noreply@anthropic.com>

* Add estop_mujoco_plugin and let payloads own their controller config

Simulated /emergency_stop as a robot-agnostic mujoco_ros2_control plugin, ExternalWrench plugin, depth-to-scan for the pan-tilt in sim, payload controller taken from pt_control, and CI/README updates.

Co-Authored-By: Claude Sonnet 5 <noreply@anthropic.com>

* Rename estop_mujoco_plugin to mujoco_ros2_plugins with one shared header

One library and one header (mujoco_ros2_plugins.hpp) so more simulation plugins can be added next to the emergency stop.

Co-Authored-By: Claude Sonnet 5 <noreply@anthropic.com>

* Make mujoco_ros2_plugins a submodule

It now lives in github.com/adityakamath/mujoco_ros2_plugins.

Co-Authored-By: Claude Sonnet 5 <noreply@anthropic.com>

* Bump mujoco_ros2_plugins

Co-Authored-By: Claude Sonnet 5 <noreply@anthropic.com>

* Bump mujoco_ros2_plugins

Co-Authored-By: Claude Sonnet 5 <noreply@anthropic.com>

* Bump mujoco_ros2_plugins

Co-Authored-By: Claude Sonnet 5 <noreply@anthropic.com>

* Bump mujoco_ros2_plugins

Co-Authored-By: Claude Sonnet 5 <noreply@anthropic.com>

* Bump mujoco_ros2_plugins

Co-Authored-By: Claude Sonnet 5 <noreply@anthropic.com>

* Bump mujoco_ros2_plugins

Co-Authored-By: Claude Sonnet 5 <noreply@anthropic.com>

* Shorten mujoco config comments

Co-Authored-By: Claude Sonnet 5 <noreply@anthropic.com>

* Bump pantilt_ros2 and mujoco_ros2_plugins

Co-Authored-By: Claude Sonnet 5 <noreply@anthropic.com>

* Refresh package.xml metadata and dependencies

Add author and URLs, align versions, declare rcl_interfaces (audio) and pt_control plus the plugin package (mujoco), drop the unused pt_description from control, and describe the navigation package correctly.

Co-Authored-By: Claude Sonnet 5 <noreply@anthropic.com>

* Flatten lekiwi_control/config: drop the base and payloads folders

Co-Authored-By: Claude Sonnet 5 <noreply@anthropic.com>

* README: point the payload teleop wiring at the flattened config folder

Co-Authored-By: Claude Sonnet 5 <noreply@anthropic.com>

* Regenerate the pre-built URDFs with portable mesh paths; drop test_without_ros and the Windows CI job

Local meshes use relative paths, the pan-tilt meshes use raw GitHub URLs, and the staleness test applies the same rewrite. Regenerate with python3 lekiwi_description/test/test_urdf_xacro.py --write.

Co-Authored-By: Claude Sonnet 5 <noreply@anthropic.com>

* Restructure the top-level and lekiwi_mujoco READMEs to the pantilt_ros2 pattern

Co-Authored-By: Claude Sonnet 5 <noreply@anthropic.com>

* Add READMEs for lekiwi_audio, lekiwi_description, lekiwi_control and lekiwi_bringup

Co-Authored-By: Claude Sonnet 5 <noreply@anthropic.com>

* Add a lekiwi_navigation README; write the IMU address as 0x28

Co-Authored-By: Claude Sonnet 5 <noreply@anthropic.com>

* Address review: credentials in the MuJoCo CI job, forward --lidar, guard the URDF joint lookup, defer the pt_mujoco import for the base

Co-Authored-By: Claude Sonnet 5 <noreply@anthropic.com>

---------

Co-authored-by: Claude Sonnet 5 <noreply@anthropic.com>

File: lekiwi_description/urdf/base/base.common.xacro (robot description, xacro)
@@ -6,6 +6,15 @@
   <!-- Base mesh rotation about Z (rad) -->
   <xacro:property name="base_offset_rz" value="${3*pi/2}"/>
+  <!-- Common wheel geometry: used by ROS controllers, URDF and MuJoCo. -->
+  <!-- Required input: base_controller_config:=/path/to/lekiwi_control/config/control.yaml.
+       The launch/integration layer supplies it; description does not depend on control. -->
+  <xacro:property name="base_geometry" value="${xacro.load_yaml('$(arg base_controller_config)')['base_controller']['ros__parameters']}"/>
+  <xacro:property name="wheel_radius" value="${base_geometry['wheel_radius']}"/>
+  <xacro:property name="offset" value="${base_geometry['wheel_offset']}"/>
+  <!-- CAD wheel mesh radius in metres; a mesh reference measurement, not an operating parameter. -->
+  <xacro:property name="wheel_mesh_radius" value="0.051"/>
+  <xacro:property name="wheel_mesh_scale" value="${wheel_radius / wheel_mesh_radius}"/>
   <!-- Wheel mount offsets -->
-  <xacro:property name="wheel_base_radius" value="0.132239"/>
+  <xacro:property name="wheel_base_radius" value="${base_geometry['robot_radius']}"/>
   <xacro:property name="wheel_base_offset_z" value="0.01036"/>
   <!-- LD06 laser offsets from base_link -->

File: lekiwi_description/urdf/base/base.control.xacro (robot description, xacro)
@@ -42,6 +42,4 @@
   <xacro:property name="proportional_acc_max" value="$(arg proportional_acc_max)"/>        <!-- [0-254] -->
   <!-- Wheel geometry for omnidirectional control -->
-  <xacro:property name="wheel_radius" value="0.051"/>  <!-- meters -->
-  <xacro:property name="offset" value="${pi/3}"/>  <!-- 60° -->
   <xacro:property name="theta" value="${2*pi/3}"/>  <!-- 120° between wheels -->
   <!-- Maximum allowable speed/acceleration/torque for each motor -->
@@ -164,15 +162,8 @@
         </sensor>
       </xacro:if>
-      <!-- Matched to base_subtree.xml's MJCF sensors by this block's name ("lidar"), not
-           frame_name. Resolution intentionally differs from the real LD19 - see base_subtree.xml. -->
-      <sensor name="lidar">
-        <param name="frame_name">laser_frame</param>
-        <param name="min_angle">0.0</param>
-        <param name="max_angle">6.274458660919615</param>
-        <param name="angle_increment">0.017453292519943295</param>
-        <param name="range_min">0.02</param>
-        <param name="range_max">12.0</param>
-        <param name="laserscan_topic">/scan</param>
-      </sensor>
+      <!-- No <sensor name="lidar"> here: that legacy rangefinder path is deprecated and costs
+           ~9 ms per physics step. The lidar is a native mujoco.plugin.lidar sensor (see
+           lekiwi_mujoco build option lidar=plugin) published by Mujoco3dLidarPlugin as /scan, configured in
+           lekiwi_mujoco/config/mujoco_ros2_control_plugins.yaml. -->
     </xacro:if>
   </ros2_control>

File: lekiwi_description/urdf/base/base.urdf (robot description, URDF)
Before this commit: robot lekiwi, 10 links, 9 joints
Links:
- link back_wheel_link: geometry collision mesh filename=../../meshes/omni_wheel.stl scale=1.0 1.0 1.0; visual mesh filename=../../meshes/omni_wheel.stl scale=1.0 1.0 1.0
- link base_link: geometry collision mesh filename=../../meshes/lekiwi_base.stl; visual mesh filename=../../meshes/lekiwi_base.stl
- link imu_link: geometry collision mesh filename=../../meshes/bno055_imu.stl; visual mesh filename=../../meshes/bno055_imu.stl
- link laser_link: geometry collision mesh filename=../../meshes/ld06_lidar.stl; visual mesh filename=../../meshes/ld06_lidar.stl
- link left_wheel_link: geometry collision mesh filename=../../meshes/omni_wheel.stl scale=1.0 1.0 1.0; visual mesh filename=../../meshes/omni_wheel.stl scale=1.0 1.0 1.0
- link mic_link: geometry collision mesh filename=../../meshes/respeaker_flex_mic.stl; visual mesh filename=../../meshes/respeaker_flex_mic.stl
- link right_wheel_link: geometry collision mesh filename=../../meshes/omni_wheel.stl scale=1.0 1.0 1.0; visual mesh filename=../../meshes/omni_wheel.stl scale=1.0 1.0 1.0

File: lekiwi_description/urdf/base_pantilt/base_pantilt.control.xacro (robot description, xacro)
@@ -13,11 +13,11 @@
   <xacro:arg name="internal_acc_coeff" default="100"/>
   <xacro:arg name="internal_control_period" default="20"/>
-  <!-- Pan/tilt-specific EEPROM tuning, independent from the wheel args above - the pantilt
-       arm accelerates/moves too fast at the wheels' aggressive settings, drawing enough
-       current to crash the Pi. Defaults here match pantilt.joints.xacro's own macro
-       defaults; override via urdf_config.yaml's pantilt_internal_* keys. -->
-  <xacro:arg name="pantilt_internal_max_vel" default="254"/>
-  <xacro:arg name="pantilt_internal_max_acc" default="254"/>
-  <xacro:arg name="pantilt_internal_acc_coeff" default="100"/>
+  <!-- Pan/tilt EEPROM tuning, independent of the wheel args above. Defaults match
+       pantilt.joints.xacro's own macro defaults (the slow, smooth profile: the wheels' 254/254/100
+       makes the pan-tilt accelerate fast enough to crash the Pi); the launch file passes the values
+       from pt_control's urdf_config.yaml so they can be tuned there. -->
+  <xacro:arg name="pantilt_internal_max_vel" default="65"/>
+  <xacro:arg name="pantilt_internal_max_acc" default="50"/>
+  <xacro:arg name="pantilt_internal_acc_coeff" default="0"/>
   <!-- Pan/tilt motor IDs, step-centering, and joint limits are NOT args here - they're
        pt_description's own physical-calibration constants, baked into pantilt.joints.xacro's
@@ -57,6 +57,4 @@
   <xacro:property name="proportional_acc_max" value="$(arg proportional_acc_max)"/>        <!-- [0-254] -->
   <!-- Wheel geometry for omnidirectional control -->
-  <xacro:property name="wheel_radius" value="0.051"/>  <!-- meters -->
-  <xacro:property name="offset" value="${pi/3}"/>  <!-- 60° -->
   <xacro:property name="theta" value="${2*pi/3}"/>  <!-- 120° between wheels -->
   <!-- Maximum allowable speed/acceleration/torque for each motor -->
@@ -192,14 +190,8 @@
         </sensor>
       </xacro:if>
-      <!-- Matched to base_subtree.xml's MJCF sensors by name ("lidar") - see base.control.xacro. -->
-      <sensor name="lidar">
-        <param name="frame_name">laser_frame</param>
-        <param name="min_angle">0.0</param>
-        <param name="max_angle">6.274458660919615</param>
-        <param name="angle_increment">0.017453292519943295</param>
-        <param name="range_min">0.02</param>
-        <param name="range_max">12.0</param>
-        <param name="laserscan_topic">/scan</param>
-      </sensor>
+      <!-- No <sensor name="lidar"> here: that legacy rangefinder path is deprecated and costs
+           ~9 ms per physics step. The lidar is a native mujoco.plugin.lidar sensor (see
+           lekiwi_mujoco build option lidar=plugin) published by Mujoco3dLidarPlugin as /scan, configured in
+           lekiwi_mujoco/config/mujoco_ros2_control_plugins.yaml. -->
     </xacro:if>
   </ros2_control>

File: lekiwi_description/urdf/base_pantilt/base_pantilt.urdf (robot description, URDF)
Before this commit: robot lekiwi, 16 links, 15 joints
Links:
- link back_wheel_link: geometry collision mesh filename=../../meshes/omni_wheel.stl scale=1.0 1.0 1.0; visual mesh filename=../../meshes/omni_wheel.stl scale=1.0 1.0 1.0
- link base_link: geometry collision mesh filename=../../meshes/lekiwi_base.stl; visual mesh filename=../../meshes/lekiwi_base.stl
- link imu_link: geometry collision mesh filename=../../meshes/bno055_imu.stl; visual mesh filename=../../meshes/bno055_imu.stl
- link laser_link: geometry collision mesh filename=../../meshes/ld06_lidar.stl; visual mesh filename=../../meshes/ld06_lidar.stl
- link left_wheel_link: geometry collision mesh filename=../../meshes/omni_wheel.stl scale=1.0 1.0 1.0; visual mesh filename=../../meshes/omni_wheel.stl scale=1.0 1.0 1.0
- link mic_link: geometry collision mesh filename=../../meshes/respeaker_flex_mic.stl; visual mesh filename=../../meshes/respeaker_flex_mic.stl
- link oak_link_model_origin: geometry visual mesh filename=https://raw.githubusercontent.com/adityakamath/pantilt_ros2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
- link pantilt_base_link: geometry collision mesh filename=https://raw.githubusercontent.com/adityakamath/pantilt_ros2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; visual mesh filename=https://raw.githubusercontent.com/adityakamath/pantilt_ros2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
- link right_wheel_link: geometry collision mesh filename=../../meshes/omni_wheel.stl scale=1.0 1.0 1.0; visual mesh filename=../../meshes/omni_wheel.stl scale=1.0 1.0 1.0
- link shoulder_link: geometry collision mesh filename=https://raw.githubusercontent.com/adityakamath/pantilt_ros2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; visual mesh filename=https://raw.githubusercontent.com/adityakamath/pantilt_ros2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
- link tilt_link: geometry collision mesh filename=https://raw.githubusercontent.com/adityakamath/pantilt_ros2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; visual mesh filename=https://raw.githubusercontent.com/adityakamath/pantilt_ros2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
