Commit message: refactor: integrate pantilt100, rename addon→payload, restructure packages
lekiwi_bringup:
- Convert to launch-only package (no C++ — remove pcl_compressor_node, cloudini deps)
- Remove oakd.launch.py, oakd_vio.yaml, oakd_vio_pcl.yaml (moved to pt100_bringup)
- Rename laser_filter_k2.yaml → laser_filter.yaml
- Rename config arg: addon → payload (lekiwi.launch.py, laser.launch.py)
- lekiwi.launch.py: delegate OAK-D to pt100_bringup/oakd.launch.py when payload=pantilt

lekiwi_control:
- Remove pantilt/ config dir (urdf_config.yaml, control.yaml, teleop.yaml)
- control.launch.py: adopt urdf_config.yaml pattern (yaml.safe_load + CLI overrides)
- Rename config arg: addon → payload

lekiwi_description:
- Replace lekiwi pantilt xacros with pt100_description includes/macros
- Move base STLs from meshes/base/* to meshes/* (flat structure)
- Remove pantilt/ urdf and mesh directories (now in pt100_description)
- Add exec_depend on pt100_description

Co-Authored-By: Claude Sonnet 4.6 <noreply@anthropic.com>

File: lekiwi_description/urdf/base/base.module.xacro (robot description, xacro)
@@ -21,5 +21,5 @@
         <origin xyz="0 0 0" rpy="0 0 ${base_offset_rz}"/>
         <geometry>
-          <mesh filename="package://lekiwi_description/meshes/base/lekiwi_base.stl"/>
+          <mesh filename="package://lekiwi_description/meshes/lekiwi_base.stl"/>
         </geometry>
         <material name="base_light_grey"/>
@@ -28,5 +28,5 @@
         <origin xyz="0 0 0" rpy="0 0 ${base_offset_rz}"/>
         <geometry>
-          <mesh filename="package://lekiwi_description/meshes/base/lekiwi_base.stl"/>
+          <mesh filename="package://lekiwi_description/meshes/lekiwi_base.stl"/>
         </geometry>
       </collision>
@@ -41,5 +41,5 @@
         <origin xyz="0 0 0" rpy="${laser_offset_rx} 0 0"/>
         <geometry>
-          <mesh filename="package://lekiwi_description/meshes/base/ld06_lidar.stl"/>
+          <mesh filename="package://lekiwi_description/meshes/ld06_lidar.stl"/>
         </geometry>
         <material name="base_charcoal"/>
@@ -48,5 +48,5 @@
         <origin xyz="0 0 0" rpy="${laser_offset_rx} 0 0"/>
         <geometry>
-          <mesh filename="package://lekiwi_description/meshes/base/ld06_lidar.stl"/>
+          <mesh filename="package://lekiwi_description/meshes/ld06_lidar.stl"/>
         </geometry>
       </collision>
@@ -63,12 +63,12 @@
         <origin xyz="0 0 0" rpy="0 0 0"/>
         <geometry>
-          <mesh filename="package://lekiwi_description/meshes/base/bno055_imu.stl"/>
-        </geometry>
-        <material name="base_charcoal"/>
-      </visual>
-      <collision>
-        <origin xyz="0 0 0" rpy="0 0 0"/>
-        <geometry>
-          <mesh filename="package://lekiwi_description/meshes/base/bno055_imu.stl"/>
+          <mesh filename="package://lekiwi_description/meshes/bno055_imu.stl"/>
+        </geometry>
+        <material name="base_charcoal"/>
+      </visual>
+      <collision>
+        <origin xyz="0 0 0" rpy="0 0 0"/>
+        <geometry>
+          <mesh filename="package://lekiwi_description/meshes/bno055_imu.stl"/>
         </geometry>
       </collision>
@@ -85,12 +85,12 @@
         <origin xyz="0 0 0" rpy="0 0 0"/>
         <geometry>
-          <mesh filename="package://lekiwi_description/meshes/base/respeaker_flex_mic.stl"/>
-        </geometry>
-        <material name="base_charcoal"/>
-      </visual>
-      <collision>
-        <origin xyz="0 0 0" rpy="0 0 0"/>
-        <geometry>
-          <mesh filename="package://lekiwi_description/meshes/base/respeaker_flex_mic.stl"/>
+          <mesh filename="package://lekiwi_description/meshes/respeaker_flex_mic.stl"/>
+        </geometry>
+        <material name="base_charcoal"/>
+      </visual>
+      <collision>
+        <origin xyz="0 0 0" rpy="0 0 0"/>
+        <geometry>
+          <mesh filename="package://lekiwi_description/meshes/respeaker_flex_mic.stl"/>
         </geometry>
       </collision>
@@ -105,12 +105,12 @@
         <origin xyz="0 0 0" rpy="0 0 0"/>
         <geometry>
-          <mesh filename="package://lekiwi_description/meshes/base/omni_wheel.stl"/>
-        </geometry>
-        <material name="base_charcoal"/>
-      </visual>
-      <collision>
-        <origin xyz="0 0 0" rpy="0 0 0"/>
-        <geometry>
-          <mesh filename="package://lekiwi_description/meshes/base/omni_wheel.stl"/>
+          <mesh filename="package://lekiwi_description/meshes/omni_wheel.stl"/>
+        </geometry>
+        <material name="base_charcoal"/>
+      </visual>
+      <collision>
+        <origin xyz="0 0 0" rpy="0 0 0"/>
+        <geometry>
+          <mesh filename="package://lekiwi_description/meshes/omni_wheel.stl"/>
         </geometry>
       </collision>
@@ -125,12 +125,12 @@
         <origin xyz="0 0 0" rpy="0 0 0"/>
         <geometry>
-          <mesh filename="package://lekiwi_description/meshes/base/omni_wheel.stl"/>
-        </geometry>
-        <material name="base_charcoal"/>
-      </visual>
-      <collision>
-        <origin xyz="0 0 0" rpy="0 0 0"/>
-        <geometry>
-          <mesh filename="package://lekiwi_description/meshes/base/omni_wheel.stl"/>
+          <mesh filename="package://lekiwi_description/meshes/omni_wheel.stl"/>
+        </geometry>
+        <material name="base_charcoal"/>
+      </visual>
+      <collision>
+        <origin xyz="0 0 0" rpy="0 0 0"/>
+        <geometry>
+          <mesh filename="package://lekiwi_description/meshes/omni_wheel.stl"/>
         </geometry>
       </collision>
@@ -145,12 +145,12 @@
         <origin xyz="0 0 0" rpy="0 0 0"/>
         <geometry>
-          <mesh filename="package://lekiwi_description/meshes/base/omni_wheel.stl"/>
-        </geometry>
-        <material name="base_charcoal"/>
-      </visual>
-      <collision>
-        <origin xyz="0 0 0" rpy="0 0 0"/>
-        <geometry>
-          <mesh filename="package://lekiwi_description/meshes/base/omni_wheel.stl"/>
+          <mesh filename="package://lekiwi_description/meshes/omni_wheel.stl"/>
+        </geometry>
+        <material name="base_charcoal"/>
+      </visual>
+      <collision>
+        <origin xyz="0 0 0" rpy="0 0 0"/>
+        <geometry>
+          <mesh filename="package://lekiwi_description/meshes/omni_wheel.stl"/>
         </geometry>
       </collision>

File: lekiwi_description/urdf/base/base.urdf (robot description, URDF)
Before this commit: robot lekiwi, 10 links, 9 joints
Links:
- link back_wheel_link: geometry collision mesh filename=../../meshes/omni_wheel.stl; visual mesh filename=../../meshes/omni_wheel.stl
- link base_link: geometry collision mesh filename=../../meshes/lekiwi_base.stl; visual mesh filename=../../meshes/lekiwi_base.stl
- link imu_link: geometry collision mesh filename=../../meshes/bno055_imu.stl; visual mesh filename=../../meshes/bno055_imu.stl
- link laser_link: geometry collision mesh filename=../../meshes/ld06_lidar.stl; visual mesh filename=../../meshes/ld06_lidar.stl
- link left_wheel_link: geometry collision mesh filename=../../meshes/omni_wheel.stl; visual mesh filename=../../meshes/omni_wheel.stl
- link mic_link: geometry collision mesh filename=../../meshes/respeaker_flex_mic.stl; visual mesh filename=../../meshes/respeaker_flex_mic.stl
- link right_wheel_link: geometry collision mesh filename=../../meshes/omni_wheel.stl; visual mesh filename=../../meshes/omni_wheel.stl

File: lekiwi_description/urdf/k2.common.xacro (robot description, xacro)
@@ -2,5 +2,5 @@
 <robot xmlns:xacro="http://www.ros.org/wiki/xacro">
   <xacro:include filename="$(find lekiwi_description)/urdf/base/base.common.xacro"/>
-  <xacro:include filename="$(find lekiwi_description)/urdf/pantilt/pantilt.common.xacro"/>
+  <xacro:include filename="$(find pt100_description)/urdf/pantilt.common.xacro"/>
   <!-- Pantilt mount point on base_link (integration-specific offsets) -->
   <xacro:property name="pantilt_base_offset_x" value="0.032725"/>

File: lekiwi_description/urdf/k2.control.xacro (robot description, xacro)
@@ -50,9 +50,10 @@
   <xacro:property name="max_linear_velocity_y" value="${wheel_radius * max_velocity_rads / 1.0}"/>
   <xacro:property name="max_angular_velocity_z" value="${wheel_radius * max_velocity_rads / wheel_base_radius}"/>
-  <!-- Pan and tilt joint limits — properties sourced from args for use in pantilt.module.xacro -->
+  <!-- Pan and tilt joint limits — properties sourced from args for use in pt100.module.xacro -->
   <xacro:property name="pan_joint_lower"  value="$(arg pan_joint_lower)"/>
   <xacro:property name="pan_joint_upper"  value="$(arg pan_joint_upper)"/>
   <xacro:property name="tilt_joint_lower" value="$(arg tilt_joint_lower)"/>
   <xacro:property name="tilt_joint_upper" value="$(arg tilt_joint_upper)"/>
+  <xacro:include filename="$(find pt100_description)/urdf/pantilt.joints.xacro"/>
   <!-- ROS 2 CONTROL -->
   <!-- System interface — all STS3215 joints on a single serial bus -->
@@ -111,38 +112,14 @@
       <state_interface name="is_moving"/>
     </joint>
-    <!-- Pan joint (Motor ID 1, position mode) -->
-    <joint name="pan_joint">
-      <param name="motor_id">$(arg pan_motor_id)</param>
-      <param name="operating_mode">0</param>
-      <param name="min_position">${pan_joint_lower}</param>
-      <param name="max_position">${pan_joint_upper}</param>
-      <param name="max_velocity">${max_velocity_rads}</param>
-      <param name="position_center_steps">$(arg pan_center_steps)</param>
-      <command_interface name="position"/>
-      <state_interface name="position"/>
-      <state_interface name="velocity"/>
-      <state_interface name="effort"/>
-      <state_interface name="voltage"/>
-      <state_interface name="temperature"/>
-      <state_interface name="current"/>
-      <state_interface name="is_moving"/>
-    </joint>
-    <!-- Tilt joint (Motor ID 2, position mode) -->
-    <joint name="tilt_joint">
-      <param name="motor_id">$(arg tilt_motor_id)</param>
-      <param name="operating_mode">0</param>
-      <param name="min_position">${tilt_joint_lower}</param>
-      <param name="max_position">${tilt_joint_upper}</param>
-      <param name="max_velocity">${max_velocity_rads}</param>
-      <param name="position_center_steps">$(arg tilt_center_steps)</param>
-      <command_interface name="position"/>
-      <state_interface name="position"/>
-      <state_interface name="velocity"/>
-      <state_interface name="effort"/>
-      <state_interface name="voltage"/>
-      <state_interface name="temperature"/>
-      <state_interface name="current"/>
-      <state_interface name="is_moving"/>
-    </joint>
+    <xacro:pt100_joints
+        pan_motor_id="$(arg pan_motor_id)"
+        tilt_motor_id="$(arg tilt_motor_id)"
+        pan_center_steps="$(arg pan_center_steps)"
+        tilt_center_steps="$(arg tilt_center_steps)"
+        sts_max_velocity_steps="${sts_max_velocity_steps}"
+        pan_joint_lower="${pan_joint_lower}"
+        pan_joint_upper="${pan_joint_upper}"
+        tilt_joint_lower="${tilt_joint_lower}"
+        tilt_joint_upper="${tilt_joint_upper}"/>
   </ros2_control>
   <!-- ROS 2 CONTROL -->

File: lekiwi_description/urdf/k2.urdf (robot description, URDF)
Before this commit: robot k2, 16 links, 15 joints
Links:
- link back_wheel_link: geometry collision mesh filename=../meshes/omni_wheel.stl; visual mesh filename=../meshes/omni_wheel.stl
- link base_link: geometry collision mesh filename=../meshes/lekiwi_base.stl; visual mesh filename=../meshes/lekiwi_base.stl
- link imu_link: geometry collision mesh filename=../meshes/bno055_imu.stl; visual mesh filename=../meshes/bno055_imu.stl
- link laser_link: geometry collision mesh filename=../meshes/ld06_lidar.stl; visual mesh filename=../meshes/ld06_lidar.stl
- link left_wheel_link: geometry collision mesh filename=../meshes/omni_wheel.stl; visual mesh filename=../meshes/omni_wheel.stl
- link mic_link: geometry collision mesh filename=../meshes/respeaker_flex_mic.stl; visual mesh filename=../meshes/respeaker_flex_mic.stl
- link right_wheel_link: geometry collision mesh filename=../meshes/omni_wheel.stl; visual mesh filename=../meshes/omni_wheel.stl

File: lekiwi_description/urdf/k2.urdf.xacro (robot description, xacro)
@@ -4,11 +4,11 @@
   <xacro:include filename="$(find lekiwi_description)/urdf/k2.control.xacro"/>
   <xacro:include filename="$(find lekiwi_description)/urdf/base/base.module.xacro"/>
-  <xacro:include filename="$(find lekiwi_description)/urdf/pantilt/pantilt.module.xacro"/>
+  <xacro:include filename="$(find pt100_description)/urdf/pt100.module.xacro"/>
   <link name="base_footprint"/>
   <xacro:lekiwi_base_module parent="base_footprint">
     <origin xyz="0 0 ${wheel_radius - wheel_base_offset_z}" rpy="0 0 0"/>
   </xacro:lekiwi_base_module>
-  <xacro:pantilt_module parent="base_link">
+  <xacro:pt100_module parent="base_link">
     <origin xyz="${pantilt_base_offset_x} 0 ${pantilt_base_offset_z}" rpy="0 0 0"/>
-  </xacro:pantilt_module>
+  </xacro:pt100_module>
 </robot>
