Commit message: Update pantilt_ros2 submodule, matching lekiwi-side integration to shoulder_pan_joint rename
Bumps payloads/pantilt_ros2 to d49e2ba (pan_joint/pan_link renamed to
shoulder_pan_joint/shoulder_link to match so101/so100's own naming, plus the
pan_joint origin-to-mesh alignment fix and single-source-of-truth motor ID/joint
limit config - see that commit for detail).

Updates the lekiwi-side integration to match:
- base_pantilt.control.xacro: drop the duplicated pan/tilt motor ID, step-centering,
  and joint limit xacro:args - pantilt.joints.xacro's macro defaults are now their
  single source of truth (lekiwi_control/config/payloads/pantilt/urdf_config.yaml
  shrinks to just proportional_vel_max accordingly).
- lekiwi_control/config/payloads/pantilt/control.yaml: pan_joint -> shoulder_pan_joint
  in the joint_limits/joint_state_broadcaster/pantilt_controller joint lists.
- lekiwi_control/launch/control.launch.py: drop the now-removed urdf_config.yaml keys
  from the xacro_cmd construction.
- base_pantilt.urdf and lekiwi_pt100/101_oakd_s2.xml MJCF snapshots regenerated to
  match.
- test_control_config.py / test_urdf_xacro.py updated for the rename and the shrunk
  urdf_config.yaml.

Co-Authored-By: Claude Sonnet 5 <noreply@anthropic.com>

File: lekiwi_description/urdf/base_pantilt/base_pantilt.control.xacro (robot description, xacro)
@@ -9,8 +9,10 @@
   <xacro:arg name="back_motor_id" default="8"/>
   <xacro:arg name="right_motor_id" default="9"/>
-  <xacro:arg name="pan_motor_id"      default="1"/>
-  <xacro:arg name="tilt_motor_id"     default="2"/>
-  <xacro:arg name="pan_center_steps"  default="2048"/>
-  <xacro:arg name="tilt_center_steps" default="2048"/>
+  <!-- Pan/tilt motor IDs, step-centering, and joint limits are NOT args here - they're
+       pt_description's own physical-calibration constants, baked into pantilt.joints.xacro's
+       macro defaults (single source of truth - see that file and pantilt.control.xacro's
+       matching comment). Override them explicitly on the <xacro:pantilt_joints> call below
+       only if this specific unit is ever calibrated differently from pt_description's
+       defaults. -->
   <!-- BNO055 IMU parameters (externally settable) -->
   <xacro:arg name="imu"             default="true"/>    <!-- false = no physical IMU; omits the lekiwi_imu sensor block below (real hardware only) -->
@@ -23,9 +25,4 @@
   <xacro:arg name="proportional_acc_max"   default="25"/>    <!-- [0-254]; 0 = disable proportional ACC -->
   <xacro:arg name="proportional_vel_max"   default="0"/>     <!-- [0-max_velocity_steps]; 0 = each joint uses commanded velocity -->
-  <!-- Pan and Tilt joint limits (configurable, symmetric ±π/2 defaults) -->
-  <xacro:arg name="pan_joint_lower"        default="-1.5708"/>  <!-- rad, default -π/2 -->
-  <xacro:arg name="pan_joint_upper"        default="1.5708"/>   <!-- rad, default +π/2 -->
-  <xacro:arg name="tilt_joint_lower"       default="-1.5708"/>  <!-- rad, default -π/2 -->
-  <xacro:arg name="tilt_joint_upper"       default="1.5708"/>   <!-- rad, default +π/2 -->
   <!-- Simulation -->
   <!-- "real" (default): STS3215 serial plugin. "mujoco": MujocoSystemInterface, driving
@@ -62,9 +59,4 @@
   <xacro:property name="max_linear_velocity_y" value="${wheel_radius * max_velocity_rads / 1.0}"/>
   <xacro:property name="max_angular_velocity_z" value="${wheel_radius * max_velocity_rads / wheel_base_radius}"/>
-  <!-- Pan and tilt joint limits — properties sourced from args for use in pantilt.module.xacro -->
-  <xacro:property name="pan_joint_lower"  value="$(arg pan_joint_lower)"/>
-  <xacro:property name="pan_joint_upper"  value="$(arg pan_joint_upper)"/>
-  <xacro:property name="tilt_joint_lower" value="$(arg tilt_joint_lower)"/>
-  <xacro:property name="tilt_joint_upper" value="$(arg tilt_joint_upper)"/>
   <!-- Duplicates pt_description's own promoted property (not included here - base_pantilt
        uses its own copy of the pantilt control block) for pantilt.module.xacro's gazebo limit. -->
@@ -152,13 +144,5 @@
     </joint>
     <xacro:pantilt_joints
-        pan_motor_id="$(arg pan_motor_id)"
-        tilt_motor_id="$(arg tilt_motor_id)"
-        pan_center_steps="$(arg pan_center_steps)"
-        tilt_center_steps="$(arg tilt_center_steps)"
         sts3215_max_vel_steps="${sts3215_max_vel_steps}"
-        pan_joint_lower="${pan_joint_lower}"
-        pan_joint_upper="${pan_joint_upper}"
-        tilt_joint_lower="${tilt_joint_lower}"
-        tilt_joint_upper="${tilt_joint_upper}"
         ros2_control_hardware_type="$(arg ros2_control_hardware_type)"/>
     <!-- IMU/lidar sensors must live in this SAME <ros2_control> block as the plugin above -

File: lekiwi_description/urdf/base_pantilt/base_pantilt.urdf (robot description, URDF)
Before this commit: robot lekiwi, 16 links, 15 joints
Links:
- removed link pan_link
- added link shoulder_link, mass 0.119226; collision mesh filename=package://pt_description/meshes/pan_joint_101.stl; visual mesh filename=package://pt_description/meshes/pan_joint_101.stl
Joints:
- removed joint pan_joint
- added joint shoulder_pan_joint: type revolute, parent pantilt_base_link, child shoulder_link, origin xyz=0.0452 0 0.0648559 rpy=0 0 0, axis 0 0 1, limit lower=-1.5708 upper=1.5708 effort=2.942 velocity=1000000.0
- joint tilt_joint: origin xyz=0.0306 0 0.1025 rpy=-1.5707963267948966 1.5707963267948966 0 -> xyz=0.0306 0 0.0541441 rpy=-1.5707963267948966 1.5707963267948966 0; parent pan_link -> shoulder_link
