Commit message: Update payload wiring, MuJoCo models and docs
Refactor control and bringup launch files and the pan-tilt xacro, rebuild the
MuJoCo models and tests to match, and bump mujoco_ros2_plugins.

Docs: move the camera notes into proper sections, document nav2_target_node,
the extra xacro arguments and the MuJoCo helper modules, clarify the empty
mission default, and note that the LD06 and LD19 are the same device.

File: lekiwi_description/urdf/base_pantilt/base_pantilt.common.xacro (robot description, xacro)
@@ -2,6 +2,4 @@
 <robot xmlns:xacro="http://www.ros.org/wiki/xacro">
   <xacro:include filename="$(find lekiwi_description)/urdf/base/base.common.xacro"/>
-  <!-- Camera selection is independent of PT100/PT101 and shared with pt_description. -->
-  <xacro:arg name="camera_config" default="gemini2"/>
   <xacro:include filename="$(find pt_description)/urdf/pantilt.common.xacro"/>
   <!-- Pantilt mount point on base_link (integration-specific offsets) -->

File: lekiwi_description/urdf/base_pantilt/base_pantilt.control.xacro (robot description, xacro)
@@ -192,25 +192,8 @@
       </xacro:if>
       <!-- The Gemini camera IMU uses the upstream MuJoCo ros2_control IMU mapping. -->
-      <xacro:if value="${'$(arg camera_config)' == 'gemini2' and '$(arg enable_camera)' == 'true'}">
+      <xacro:if value="${'$(arg enable_camera)' == 'true'}">
         <sensor name="gemini2">
           <param name="mujoco_type">imu</param>
           <param name="mujoco_sensor_name">gemini2</param>
-          <state_interface name="orientation.x"/>
-          <state_interface name="orientation.y"/>
-          <state_interface name="orientation.z"/>
-          <state_interface name="orientation.w"/>
-          <state_interface name="angular_velocity.x"/>
-          <state_interface name="angular_velocity.y"/>
-          <state_interface name="angular_velocity.z"/>
-          <state_interface name="linear_acceleration.x"/>
-          <state_interface name="linear_acceleration.y"/>
-          <state_interface name="linear_acceleration.z"/>
-        </sensor>
-      </xacro:if>
-      <!-- OAK-D S2 uses the same upstream IMU mapping at its URDF mount. -->
-      <xacro:if value="${'$(arg camera_config)' == 'oakd_s2' and '$(arg enable_camera)' == 'true'}">
-        <sensor name="oak">
-          <param name="mujoco_type">imu</param>
-          <param name="mujoco_sensor_name">oak</param>
           <state_interface name="orientation.x"/>
           <state_interface name="orientation.y"/>

File: lekiwi_description/urdf/base_pantilt/base_pantilt_gemini2.urdf (robot description, URDF)
Before this commit: robot lekiwi, 16 links, 15 joints
Links:
- removed link oak_imu_frame
- removed link oak_link
- removed link oak_link_model_origin
- added link gemini2_imu_frame
- added link gemini2_link
- added link gemini2_link_model_origin; visual mesh filename=https://raw.githubusercontent.com/adityakamath/pantilt_ros2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
Joints:
- removed joint oak_imu_frame_joint
- removed joint oak_link_center_joint
- removed joint oak_link_model_origin_joint
- added joint gemini2_imu_frame_joint: type fixed, parent gemini2_link, child gemini2_imu_frame, origin xyz=-0.008 -0.037945 -0.00079 rpy=3.141592653589793 1.5707963267948966 0
- added joint gemini2_link_center_joint: type fixed, parent tilt_link, child gemini2_link, origin xyz=-0.0306 -0.0068941 -0.000225 rpy=1.5707963267948966 0 -1.5707963267948966
- added joint gemini2_link_model_origin_joint: type fixed, parent gemini2_link, child gemini2_link_model_origin, origin xyz=0 0 0 rpy=1.5707963267948966 0 1.5707963267948966
